File: PCB/V1A/Electronic_Load_V1A.sch (EAGLE design)
At the start: 124 parts, among them IC301 MAX743CPE, IC302 7805T, IC303 7805T, J101 +, J102 -, J103 +, J104 -, Q101 SIRC10DP, Q102 SIRC10DP, Q103 SIRC10DP, Q104 IXTK102N65X2, Q105 SIRC10DP, Q106 SIRC10DP, Q107 SIRC10DP, Q108 IXTK102N65X2, U1 LT1014, U101 AD420, U102 AD420, U103 LT1014, U201 LT1014, U202 LTC1865-MSOP, U203 LTC1865-MSOP

Commit message: Changed measurement opamps to OPA77
Parts:
- removed U1: LT1014, SparkFun-Retired:LT1014
- added C501, C502, C503, C504, C505, C506, C508, C510, C511, C512, C513, C514, C516: 0.1µ, rcl:C-EUC0805
- added C507, C509, C515: 1µ, rcl:CPOL-EUSMCC
- added HS401, HS402: HEATSINK-LGA115X, mechanical:HEATSINK-LGA115X
- added IC501, IC502, IC503, IC504, IC505: OPA77P, burr-brown:OPA77P
- added J401, J403: +, SparkFun-Connectors:BANANA_CONN
- added J402, J404: -, SparkFun-Connectors:BANANA_CONN
- added Q401, Q402, Q403, Q405, Q406, Q407: SIRC10DP, transistors:SIRC10DP
- added Q404, Q408: IXTK102N65X2, transistors:IXTK102N65X2
- added R401, R402, R403, R404, R405, R409, R410, R411, R412: 100R, rcl:R-EU_M5923
- added R406, R408, R413, R415: 0R004, rcl:R-EU_R6332
- added R407, R414: 2R, rcl:R-EU_M5923
- added R501, R502, R503, R508, R509, R510, R511, R512, R513, R514, R515, R516, R518, R519, R531, R532, R533, R534: 200k, rcl:R-EU_R0805
- added R504, R505, R506, R507, R527, R528, R529, R530: 5k, rcl:R-EU_R0805
- added R517: 20k, rcl:R-EU_R0805
- added R520, R521, R524, R525: 10k, rcl:R-EU_R0805
- added R522, R523, R526, R535, R536: 20k, rcl:R-TRIMM4G/J
- added S401: (no value), switch:320-938
- added U501, U502, U503: LTC1865-MSOP, adc_dac:LTC1865-MSOP
- renumbered R1 to R124, R10 to R133, R11 to R134, R12 to R136, R13 to R135, R14 to R138, R15 to R137, R2 to R125, R3 to R126, R4 to R127, R5 to R131, R6 to R130, R7 to R129, R8 to R128, R9 to R132
Connections:
- new net DUT_+1: J403.1, Q404.D, Q408.D, S4011.S
- new net MISO: U501.SDO, U502.SDO, U503.SDO
- new net MOSI: U501.SDI, U502.SDI, U503.SDI
- new net N$52: Q404.G, R404.2
- new net N$54: Q408.G, R411.2
- new net N$55: Q403.G, R405.2
- new net N$56: Q402.G, R403.2
- new net N$57: Q407.G, R412.2
- new net N$58: Q406.G, R410.2
- new net N$59: R401.2, R402.1, R403.1, R405.1, R409.1, R410.1, R412.1
- new net N$60: Q401.G, R402.2
- new net N$61: Q405.G, R409.2
- new net N$62: R516.1, R517.2, R520.1
- new net N$63: IC503.TRIM1, R526.A
- new net N$64: IC504.-IN, R528.2, R533.1
- new net N$65: IC504.+IN, R527.2, R531.2
- new net N$66: IC501.-IN, R505.2, R518.1
- new net N$67: IC501.+IN, R504.2, R514.2
- new net N$68: IC504.TRIM1, R535.A
- new net N$69: IC501.TRIM1, R522.A
- new net N$70: IC501.TRIM2, R522.E
- new net N$71: IC504.TRIM2, R535.E
- new net N$72: IC503.TRIM2, R526.E
- new net N$73: R511.2, R516.2
- new net N$74: IC502.-IN, R507.2, R519.1
- new net N$75: IC502.+IN, R506.2, R515.2
- new net N$76: IC502.TRIM1, R523.A
- new net N$77: IC502.TRIM2, R523.E
- new net N$78: R511.1, R512.2
- new net N$79: R512.1, R513.2
- new net N$80: IC505.-IN, R530.2, R534.1
- new net N$81: IC505.+IN, R529.2, R532.2
- new net N$82: IC505.TRIM1, R536.A
- new net N$83: IC505.TRIM2, R536.E
- new net N$84: R510.1, R513.1
- new net N$85: R509.1, R510.2
- new net N$86: R508.1, R509.2
- new net N$87: R501.2, R508.2
- new net N$88: R501.1, R502.2
- new net N$89: R502.1, R503.2
- new net N$91: IC503.+IN, R520.2, R521.2
- new net N$92: IC503.-IN, R524.2, R525.1
- new net REM_VSENSE+1: J401.1, S4011.O
- new net REM_VSENSE-1: J402.1, S401B.O
- new net SCK: U501.SCK, U502.SCK, U503.SCK
- new net SS_ADC_H: U501.CONV
- new net SS_ADC_L: U503.CONV
- new net SS_ADC_V: U502.CONV
- new net VSENSE: IC503.OUT, R525.2, U502.CH0
- net +15V: now also C501.1, C502.1, C505.1, C511.1, C512.1, IC501.V+, IC502.V+, IC503.V+, IC504.V+, IC505.V+, R522.S, R523.S, R526.S, R535.S, R536.S
- net +5V: now also C507.+, C508.1, C509.+, C510.1, C515.+, C516.1, U501.VCC, U502.VCC, U503.VCC
- net -15V: now also C503.1, C504.1, C506.1, C513.1, C514.1, IC501.V-, IC502.V-, IC503.V-, IC504.V-, IC505.V-
- net BYP_G: now also R401.1
- net CSENSE_H1: now also Q401.S, Q402.S, Q403.S, R406.2, R407.1, R408.2, R504.1, R528.1
- net CSENSE_H1_AMP: now also IC501.OUT, R518.2, U501.CH0
- net CSENSE_H2: now also Q405.S, Q406.S, Q407.S, R413.2, R414.1, R415.2, R506.1, R530.1
- net CSENSE_H2_AMP: now also IC502.OUT, R519.2, U501.CH1
- net CSENSE_L1: now also Q401.D, Q402.D, Q403.D, Q404.S, R407.2, R527.1
- net CSENSE_L1_AMP: now also IC504.OUT, R533.2, U503.CH0
- net CSENSE_L2: now also Q405.D, Q406.D, Q407.D, Q408.S, R414.2, R529.1
- net CSENSE_L2_AMP: now also IC505.OUT, R534.2, U503.CH1
- net GND: now also C501.2, C502.2, C503.2, C504.2, C505.2, C506.2, C507.-, C508.2, C509.-, C510.2, C511.2, C512.2, C513.2, C514.2, C515.-, C516.2, J404.1, R406.1, R408.1, R413.1, R415.1, R505.1, R507.1, R514.1, R515.1, R517.1, R521.1, R531.1, R532.1, S401B.S, U501.AGND, U501.DGND, U502.AGND, U502.DGND, U503.AGND, U503.DGND
- net LOAD_G1: now also R404.1
- net LOAD_G2: now also R411.1
- net VREF: now also U501.VREF, U502.VREF, U503.VREF
- net VSENSE+: now also R503.1, S4011.P
- net VSENSE-: now also R524.1, S401B.P
Other:
- note added: "High current"
- note added: "Low current"
- note added: "Voltage"
- note added: "some info here"

Commit message: Created board layout, added info
Parts:
- removed C101, C102, C107, C108, C109, C110: 100n, rcl:C-EUC0805
- removed C103, C104, C105, C106: 10n, rcl:C-EUC0805
- removed C501, C502, C503, C504, C505, C506, C508, C510, C511, C512, C513, C514, C516: 0.1µ, rcl:C-EUC0805
- removed C507, C509, C515: 1µ, rcl:CPOL-EUSMCC
- removed HS401, HS402: HEATSINK-LGA115X, mechanical:HEATSINK-LGA115X
- removed IC501, IC502, IC503, IC504, IC505: OPA77P, burr-brown:OPA77P
- removed J401, J403: +, SparkFun-Connectors:BANANA_CONN
- removed J402, J404: -, SparkFun-Connectors:BANANA_CONN
- removed Q401, Q402, Q403, Q405, Q406, Q407: SIRC10DP, transistors:SIRC10DP
- removed Q404, Q408: IXTK102N65X2, transistors:IXTK102N65X2
- removed R116, R122, R414: 2R, rcl:R-EU_M5923
- removed R117, R123: 0R002, rcl:R-EU_M5923
- removed R118, R119, R120, R121, R411, R412: 100R, rcl:R-EU_M5923
- removed R124, R125, R126, R127, R128, R129, R130, R131, R132, R133: 1M, rcl:R-EU_R2512
- removed R134: (no value), rcl:R-EU_R2512
- removed R135, R136, R137, R138: 5k, rcl:R-EU_M5923
- removed R413, R415: 0R004, rcl:R-EU_R6332
- removed R501, R502, R503, R508, R509, R510, R511, R512, R513, R514, R515, R516, R518, R519, R531, R532, R533, R534: 200k, rcl:R-EU_R0805
- removed R504, R505, R506, R507, R527, R528, R529, R530: 5k, rcl:R-EU_R0805
- removed R517: 20k, rcl:R-EU_R0805
- removed R520, R521, R524, R525: 10k, rcl:R-EU_R0805
- removed R522, R523, R526, R535, R536: 20k, rcl:R-TRIMM4G/J
- removed S401: (no value), switch:320-938
- removed U101, U102: AD420, adc_dac:AD420
- removed U103: LT1014, SparkFun-Retired:LT1014
- removed U501, U502, U503: LTC1865-MSOP, adc_dac:LTC1865-MSOP
- added C201, C202, C203, C204, C205, C206, C208, C210, C211, C212, C213, C214, C216: 0.1µ, rcl:C-EUC0805
- added C207, C209, C215: 1µ, rcl:CPOL-EUSMCC
- added C401, C402, C407, C408, C409, C410: 100n, rcl:C-EUC0805
- added C403, C404, C405, C406: 10n, rcl:C-EUC0805
- added IC201, IC202, IC203, IC204, IC205: OPA77P, burr-brown:OPA77P
- added R229, R230: 5k, rcl:R-EU_R0805
- added R231, R232, R233, R234: 200k, rcl:R-EU_R0805
- added R235, R236: 20k, rcl:R-TRIMM4G/J
- added U401, U402: AD420, adc_dac:AD420
- added U403: LT1014, SparkFun-Retired:LT1014
- Q104: value IXTK102N65X2 -> IXTK102N65X2PADUP-; device transistors:IXTK102N65X2 -> transistors:IXTK102N65X2PADUP-
- Q108: value IXTK102N65X2 -> IXTK102N65X2PADUP; device transistors:IXTK102N65X2 -> transistors:IXTK102N65X2PADUP
- R101, R102: value 20k -> 100R; device rcl:R-TRIMM4G/J -> rcl:R-EU_M5923
- R103, R104: value 200k -> 100R
- R106, R113, R115: value 100R -> 0R004; device rcl:R-EU_M5923 -> rcl:R-EU_R6332
- R107: value 5k -> 2R; device rcl:R-EU_M5923 -> rcl:R-EU_R0805
- R108: value 5k -> 0R004; device rcl:R-EU_M5923 -> rcl:R-EU_R6332
- R109, R110: value 5k -> 100R
- R114: value 100R -> 2R; device rcl:R-EU_M5923 -> rcl:R-EU_R0805
- R201, R202, R203, R215, R216, R218: value 5k -> 200k
- R205, R207: value 200k -> 5k
- R206: value 200 -> 5k
- R208: value 200 -> 200k
- R210, R212: value 20k -> 200k
- R213, R214: value 20k -> 200k; device rcl:R-TRIMM4G/J -> rcl:R-EU_R0805
- R217: value 5k -> 20k
- R220: value 200 -> 10k
- R221, R225: value 200k -> 10k
- R222: value 200 -> 20k; device rcl:R-EU_R0805 -> rcl:R-TRIMM4G/J
- R223: value 200k -> 20k; device rcl:R-EU_R0805 -> rcl:R-TRIMM4G/J
- R224: value 20k -> 10k
- R226: device rcl:R-EU_R0805 -> rcl:R-TRIMM4G/J
- R227, R228: value 20k -> 5k; device rcl:R-TRIMM4G/J -> rcl:R-EU_R0805
- R401, R402: value 100R -> 20k; device rcl:R-EU_M5923 -> rcl:R-TRIMM4G/J
- R403, R404: value 100R -> 200k
- R406: value 0R004 -> 100R; device rcl:R-EU_R6332 -> rcl:R-EU_M5923
- R407: value 2R -> 5k
- R408: value 0R004 -> 5k; device rcl:R-EU_R6332 -> rcl:R-EU_M5923
- R409, R410: value 100R -> 5k
- U201: value LT1014 -> LTC1865-MSOP; device SparkFun-Retired:LT1014 -> adc_dac:LTC1865-MSOP
Connections:
- removed net CENSE_L1_AMP: R211.2, U201G2.OUT
- removed net DUT_+: J103.1, Q104.D, Q108.D, S1011.S
- removed net N$1: Q104.G, R113.2
- removed net N$10: Q102.G, R114.2
- removed net N$11: R204.2, R207.2, U201G2.+IN
- removed net N$12: R207.1, R208.2, R212.1
- removed net N$13: Q107.G, R121.2
- removed net N$14: Q106.G, R120.2
- removed net N$15: R212.2, R214.S
- removed net N$16: R215.2, R223.1, U201G3.-IN
- removed net N$17: R216.2, R219.2, U201G3.+IN
- removed net N$18: R219.1, R220.2, R224.1
- removed net N$19: R224.2, R227.S
- removed net N$2: Q108.G, R119.2
- removed net N$20: R217.2, R225.1, U201G4.-IN
- removed net N$21: R218.2, R221.2, U201G4.+IN
- removed net N$22: R221.1, R222.2, R226.1
- removed net N$23: R226.2, R228.S
- removed net N$3: R201.2, R209.1, U201G1.-IN
- removed net N$30: Q101.G, R112.2
- removed net N$31: Q105.G, R118.2
- removed net N$4: R202.2, R205.2, U201G1.+IN
- removed net N$41: R124.1, R125.2
- removed net N$42: R125.1, R126.2
- removed net N$43: R126.1, R127.2
- removed net N$45: R127.1, R131.1
- removed net N$46: R130.1, R131.2
- removed net N$47: R129.1, R130.2
- removed net N$48: R128.1, R129.2
- removed net N$49: R128.2, R132.2
- removed net N$5: R205.1, R206.2, R210.1
- removed net N$50: R132.1, R133.2
- removed net N$51: R133.1, R134.2
- removed net N$53: R124.2
- removed net N$6: R111.2, R112.1, R114.1, R115.1, R118.1, R120.1, R121.1
- removed net N$7: R210.2, R213.S
- removed net N$8: R203.2, R211.1, U201G2.-IN
- removed net N$9: Q103.G, R115.2
- removed net REM_VSENSE+: J101.1, S1011.O
- removed net REM_VSENSE-: J102.1, S101B.O
- net +12V: now also C403.2, C404.2, C405.2, C406.2, C407.1, C408.1, U401.VCC, U402.VCC; no longer C103.2, C104.2, C105.2, C106.2, C107.1, C108.1, U101.VCC, U102.VCC
- net +15V: now also C201.1, C202.1, C205.1, C211.1, C212.1, C409.1, IC201.V+, IC202.V+, IC203.V+, IC204.V+, IC205.V+, R222.S, R223.S, R226.S, R235.S, R236.S, U403G1.+V; no longer C109.1, C501.1, C502.1, C505.1, C511.1, C512.1, IC501.V+, IC502.V+, IC503.V+, IC504.V+, IC505.V+, R522.S, R523.S, R526.S, R535.S, R536.S, U103G1.+V, U201G1.+V
- net +5V: now also C207.+, C208.1, C209.+, C210.1, C215.+, C216.1, C401.1, C402.1, U201.VCC, U401.VLL, U402.VLL; no longer C101.1, C102.1, C507.+, C508.1, C509.+, C510.1, C515.+, C516.1, U101.VLL, U102.VLL, U501.VCC, U502.VCC, U503.VCC
- net +5V/1: now also R401.E, R402.E; no longer R101.E, R102.E, R213.A, R214.A, R227.A, R228.A
- net -15V: now also C203.1, C204.1, C206.1, C213.1, C214.1, C410.1, IC201.V-, IC202.V-, IC203.V-, IC204.V-, IC205.V-, U403G1.-V; no longer C110.1, C503.1, C504.1, C506.1, C513.1, C514.1, IC501.V-, IC502.V-, IC503.V-, IC504.V-, IC505.V-, U103G1.-V, U201G1.-V
- net -5V: now also R401.A, R402.A; no longer R101.A, R102.A, R213.E, R214.E, R227.E, R228.E
- net BYP_G: now also R101.1; no longer R111.1, R401.1
- net CSENSE_H1: now also R106.2, R107.1, R108.2, R204.1, R228.1; no longer Q401.S, Q402.S, Q403.S, R116.1, R117.2, R202.1, R406.2, R407.1, R408.2, R504.1, R528.1
- net CSENSE_H1_AMP: now also IC201.OUT, R218.2, U201.CH0; no longer IC501.OUT, R209.2, R518.2, U201G1.OUT, U202.CH0, U501.CH0
- net CSENSE_H2: now also R113.2, R114.1, R115.2, R206.1, R230.1; no longer Q405.S, Q406.S, Q407.S, R122.1, R123.2, R216.1, R413.2, R414.1, R415.2, R506.1, R530.1
- net CSENSE_H2_AMP: now also IC202.OUT, R219.2, U201.CH1; no longer IC502.OUT, R223.2, R519.2, U201G3.OUT, U202.CH1, U501.CH1
- net CSENSE_L1: now also R107.2, R227.1; no longer Q401.D, Q402.D, Q403.D, Q404.S, R116.2, R204.1, R407.2, R527.1
- net CSENSE_L1_AMP: now also IC204.OUT, R233.2; no longer IC504.OUT, R533.2, U503.CH0
- net CSENSE_L2: now also R114.2, R229.1; no longer Q405.D, Q406.D, Q407.D, Q408.S, R122.2, R218.1, R414.2, R529.1
- net CSENSE_L2_AMP: now also IC205.OUT, R234.2; no longer IC505.OUT, R225.2, R534.2, U201G4.OUT, U503.CH1
- net DUT_+1: now also J103.1, Q104.D, Q108.D, S1011.S; no longer J403.1, Q404.D, Q408.D, S4011.S
- net GND: now also C201.2, C202.2, C203.2, C204.2, C205.2, C206.2, C207.-, C208.2, C209.-, C210.2, C211.2, C212.2, C213.2, C214.2, C215.-, C216.2, C401.2, C402.2, C407.2, C408.2, C409.2, C410.2, R108.1, R113.1, R115.1, R205.1, R207.1, R214.1, R221.1, R231.1, R232.1, R405.1, U201.AGND, U201.DGND, U202.AGND, U202.DGND, U203.AGND, U203.DGND, U401.GND, U401.RS1, U401.RS2, U402.GND, U402.RS1, U402.RS2; no longer C101.2, C102.2, C107.2, C108.2, C109.2, C110.2, C501.2, C502.2, C503.2, C504.2, C505.2, C506.2, C507.-, C508.2, C509.-, C510.2, C511.2, C512.2, C513.2, C514.2, C515.-, C516.2, J404.1, R105.1, R117.1, R123.1, R134.1, R201.1, R203.1, R206.1, R208.1, R220.1, R222.1, R408.1, R413.1, R415.1, R505.1, R507.1, R514.1, R515.1, R517.1, R521.1, R531.1, R532.1, S401B.S, U101.GND, U101.RS1, U101.RS2, U102.GND, U102.RS1, U102.RS2, U501.AGND, U501.DGND, U502.AGND, U502.DGND, U503.AGND, U503.DGND
- net LOAD_G1: now also R104.1, R409.2, U403G1.OUT; no longer R109.2, R113.1, R404.1, U103G1.OUT
- net LOAD_G2: now also R111.1, R410.2, U403G2.OUT; no longer R110.2, R119.1, R411.1, U103G2.OUT
- net MISO: now also U201.SDO, U202.SDO, U203.SDO; no longer U501.SDO, U502.SDO, U503.SDO
- net MOSI: now also U201.SDI, U202.SDI, U203.SDI; no longer U501.SDI, U502.SDI, U503.SDI
- net N$24: now also C406.1, U402.CAP2; no longer C106.1, U102.CAP2
- net N$25: now also C403.1, U401.CAP1; no longer C103.1, U101.CAP1
- net N$26: now also C404.1, U402.CAP1; no longer C104.1, U102.CAP1
- net N$27: now also C405.1, U401.CAP2; no longer C105.1, U101.CAP2
- net N$28: now also R407.2, R409.1, U403G1.-IN; no longer R107.2, R109.1, U103G1.-IN
- net N$29: now also R408.2, R410.1, U403G2.-IN; no longer R108.2, R110.1, U103G2.-IN
- net N$32: now also R403.2, R405.2, R407.1; no longer R103.2, R105.2, R107.1
- net N$33: now also R401.S, R403.1; no longer R101.S, R103.1
- net N$34: now also R402.S, R404.1; no longer R102.S, R104.1
- net N$35: now also R404.2, R406.2, R408.1; no longer R104.2, R106.2, R108.1
- net N$52: now also Q104.G, R104.2; no longer Q404.G, R404.2
- net N$54: now also Q108.G, R111.2; no longer Q408.G, R411.2
- net N$55: now also Q103.G, R105.2; no longer Q403.G, R405.2
- net N$56: now also Q102.G, R103.2; no longer Q402.G, R403.2
- net N$57: now also Q107.G, R112.2; no longer Q407.G, R412.2
- net N$58: now also Q106.G, R110.2; no longer Q406.G, R410.2
- net N$59: now also R101.2, R102.1, R103.1, R105.1, R109.1, R110.1, R112.1; no longer R401.2, R402.1, R403.1, R405.1, R409.1, R410.1, R412.1
- net N$60: now also Q101.G, R102.2; no longer Q401.G, R402.2
- net N$61: now also Q105.G, R109.2; no longer Q405.G, R409.2
- net N$62: now also R216.1, R217.2, R220.1; no longer R516.1, R517.2, R520.1
- net N$63: now also IC203.TRIM1, R226.A; no longer IC503.TRIM1, R526.A
- net N$64: now also IC204.-IN, R228.2, R233.1; no longer IC504.-IN, R528.2, R533.1
- net N$65: now also IC204.+IN, R227.2, R231.2; no longer IC504.+IN, R527.2, R531.2
- net N$66: now also IC201.-IN, R205.2, R218.1; no longer IC501.-IN, R505.2, R518.1
- net N$67: now also IC201.+IN, R204.2, R214.2; no longer IC501.+IN, R504.2, R514.2
- net N$68: now also IC204.TRIM1, R235.A; no longer IC504.TRIM1, R535.A
- net N$69: now also IC201.TRIM1, R222.A; no longer IC501.TRIM1, R522.A
- net N$70: now also IC201.TRIM2, R222.E; no longer IC501.TRIM2, R522.E
- net N$71: now also IC204.TRIM2, R235.E; no longer IC504.TRIM2, R535.E
- net N$72: now also IC203.TRIM2, R226.E; no longer IC503.TRIM2, R526.E
- net N$73: now also R211.2, R216.2; no longer R511.2, R516.2
- net N$74: now also IC202.-IN, R207.2, R219.1; no longer IC502.-IN, R507.2, R519.1
- net N$75: now also IC202.+IN, R206.2, R215.2; no longer IC502.+IN, R506.2, R515.2
- net N$76: now also IC202.TRIM1, R223.A; no longer IC502.TRIM1, R523.A
- net N$77: now also IC202.TRIM2, R223.E; no longer IC502.TRIM2, R523.E
- net N$78: now also R211.1, R212.2; no longer R511.1, R512.2
- net N$79: now also R212.1, R213.2; no longer R512.1, R513.2
- net N$80: now also IC205.-IN, R230.2, R234.1; no longer IC505.-IN, R530.2, R534.1
- net N$81: now also IC205.+IN, R229.2, R232.2; no longer IC505.+IN, R529.2, R532.2
- net N$82: now also IC205.TRIM1, R236.A; no longer IC505.TRIM1, R536.A
- net N$83: now also IC205.TRIM2, R236.E; no longer IC505.TRIM2, R536.E
- net N$84: now also R210.1, R213.1; no longer R510.1, R513.1
- net N$85: now also R209.1, R210.2; no longer R509.1, R510.2
- net N$86: now also R208.1, R209.2; no longer R508.1, R509.2
- net N$87: now also R201.2, R208.2; no longer R501.2, R508.2
- net N$88: now also R201.1, R202.2; no longer R501.1, R502.2
- net N$89: now also R202.1, R203.2; no longer R502.1, R503.2
- net N$91: now also IC203.+IN, R220.2, R221.2; no longer IC503.+IN, R520.2, R521.2
- net N$92: now also IC203.-IN, R224.2, R225.1; no longer IC503.-IN, R524.2, R525.1
- net REM_VSENSE+1: now also J101.1, S1011.O; no longer J401.1, S4011.O
- net REM_VSENSE-1: now also J102.1, S101B.O; no longer J402.1, S401B.O
- net SCK: now also U201.SCK, U202.SCK, U203.SCK; no longer U501.SCK, U502.SCK, U503.SCK
- net SS_ADC_H: now also U201.CONV; no longer U501.CONV
- net SS_ADC_L: now also U203.CONV; no longer U503.CONV
- net SS_ADC_V: now also U202.CONV; no longer U502.CONV
- net VGATE_1: now also U401.VOUT, U403G1.+IN; no longer U101.VOUT, U103G1.+IN
- net VGATE_2: now also U402.VOUT, U403G2.+IN; no longer U102.VOUT, U103G2.+IN
- net VREF: now also U201.VREF, U202.VREF, U203.VREF, U401.REF_IN, U401.REF_OUT, U402.REF_IN; no longer U101.REF_IN, U101.REF_OUT, U102.REF_IN, U501.VREF, U502.VREF, U503.VREF
- net VSENSE: now also IC203.OUT, R225.2, U202.CH0; no longer IC503.OUT, R525.2, U502.CH0
- net VSENSE+: now also R203.1; no longer R503.1, S4011.P
- net VSENSE-: now also R224.1; no longer R524.1, S401B.P

Commit message: Board layout work
Parts:
- IC304: value (none) -> 7905
- R101, R102, R103, R104, R105, R109, R110, R111, R112: device rcl:R-EU_M5923 -> rcl:R-EU_R1206
- R107, R114: device rcl:R-EU_R0805 -> rcl:R-EU_R1206
- R403, R404, R405, R406, R407, R408, R409, R410: device rcl:R-EU_M5923 -> rcl:R-EU_R0805
Changed lines of the file:
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@@
 <?xml version="1.0" encoding="utf-8"?>
 <!DOCTYPE eagle SYSTEM "eagle.dtd">
-<eagle version="9.0.0">
+<eagle version="9.0.1">
 <drawing>
 <settings>
@@
 <part name="GND410" library="supply1" library_urn="urn:adsk.eagle:library:371" deviceset="GND" device=""/>
 <part name="GND411" library="supply1" library_urn="urn:adsk.eagle:library:371" deviceset="GND" device=""/>
-<part name="R407" library="rcl" library_urn="urn:adsk.eagle:library:334" deviceset="R-EU_" device="M5923" package3d_urn="urn:adsk.eagle:package:23564/1" value="5k"/>
-<part name="R409" library="rcl" library_urn="urn:adsk.eagle:library:334" deviceset="R-EU_" device="M5923" package3d_urn="urn:adsk.eagle:package:23564/1" value="5k"/>
-<part name="R408" library="rcl" library_urn="urn:adsk.eagle:library:334" deviceset="R-EU_" device="M5923" package3d_urn="urn:adsk.eagle:package:23564/1" value="5k"/>
-<part name="R410" library="rcl" library_urn="urn:adsk.eagle:library:334" deviceset="R-EU_" device="M5923" package3d_urn="urn:adsk.eagle:package:23564/1" value="5k"/>
-<part name="R405" library="rcl" library_urn="urn:adsk.eagle:library:334" deviceset="R-EU_" device="M5923" package3d_urn="urn:adsk.eagle:package:23564/1" value="100R"/>
+<part name="R407" library="rcl" library_urn="urn:adsk.eagle:library:334" deviceset="R-EU_" device="R0805" package3d_urn="urn:adsk.eagle:package:23553/2" value="5k"/>
+<part name="R409" library="rcl" library_urn="urn:adsk.eagle:library:334" deviceset="R-EU_" device="R0805" package3d_urn="urn:adsk.eagle:package:23553/2" value="5k"/>
+<part name="R408" library="rcl" library_urn="urn:adsk.eagle:library:334" deviceset="R-EU_" device="R0805" package3d_urn="urn:adsk.eagle:package:23553/2" value="5k"/>
+<part name="R410" library="rcl" library_urn="urn:adsk.eagle:library:334" deviceset="R-EU_" device="R0805" package3d_urn="urn:adsk.eagle:package:23553/2" value="5k"/>
+<part name="R405" library="rcl" library_urn="urn:adsk.eagle:library:334" deviceset="R-EU_" device="R0805" package3d_urn="urn:adsk.eagle:package:23553/2" value="100R"/>
 <part name="R401" library="rcl" library_urn="urn:adsk.eagle:library:334" deviceset="R-TRIMM" device="4G/J" package3d_urn="urn:adsk.eagle:package:23728/1" value="20k"/>
-<part name="R403" library="rcl" library_urn="urn:adsk.eagle:library:334" deviceset="R-EU_" device="M5923" package3d_urn="urn:adsk.eagle:package:23564/1" value="200k"/>
-<part name="R406" library="rcl" library_urn="urn:adsk.eagle:library:334" deviceset="R-EU_" device="M5923" package3d_urn="urn:adsk.eagle:package:23564/1" value="100R"/>
-<part name="R404" library="rcl" library_urn="urn:adsk.eagle:library:334" deviceset="R-EU_" device="M5923" package3d_urn="urn:adsk.eagle:package:23564/1" value="200k"/>
+<part name="R403" library="rcl" library_urn="urn:adsk.eagle:library:334" deviceset="R-EU_" device="R0805" package3d_urn="urn:adsk.eagle:package:23553/2" value="200k"/>
+<part name="R406" library="rcl" library_urn="urn:adsk.eagle:library:334" deviceset="R-EU_" device="R0805" package3d_urn="urn:adsk.eagle:package:23553/2" value="100R"/>
+<part name="R404" library="rcl" library_urn="urn:adsk.eagle:library:334" deviceset="R-EU_" device="R0805" package3d_urn="urn:adsk.eagle:package:23553/2" value="200k"/>
 <part name="R402" library="rcl" library_urn="urn:adsk.eagle:library:334" deviceset="R-TRIMM" device="4G/J" package3d_urn="urn:adsk.eagle:package:23728/1" value="20k"/>
 <part name="GND409" library="supply1" library_urn="urn:adsk.eagle:library:371" deviceset="GND" device=""/>
@@
 <part name="P-401" library="supply1" library_urn="urn:adsk.eagle:library:371" deviceset="-15V" device=""/>
 <part name="IC303" library="linear" library_urn="urn:adsk.eagle:library:262" deviceset="78*" device="T" package3d_urn="urn:adsk.eagle:package:16414/1" technology="05"/>
-<part name="IC304" library="linear" library_urn="urn:adsk.eagle:library:262" deviceset="79*" device="T" package3d_urn="urn:adsk.eagle:package:16414/1" technology="05"/>
+<part name="IC304" library="linear" library_urn="urn:adsk.eagle:library:262" deviceset="79*" device="T" package3d_urn="urn:adsk.eagle:package:16414/1" technology="05" value="7905"/>
 <part name="C307" library="rcl" library_urn="urn:adsk.eagle:library:334" deviceset="C-EU" device="C0805" package3d_urn="urn:adsk.eagle:package:23617/2" value="0.33u"/>
 <part name="C308" library="rcl" library_urn="urn:adsk.eagle:library:334" deviceset="C-EU" device="C0805" package3d_urn="urn:adsk.eagle:package:23617/2" value="0.1u"/>
@@
 <part name="J102" library="SparkFun-Connectors" deviceset="BANANA_CONN" device="" value="-"/>
 <part name="S101" library="switch" library_urn="urn:adsk.eagle:library:380" deviceset="320-938" device="" package3d_urn="urn:adsk.eagle:package:27685/1"/>
-<part name="R104" library="rcl" library_urn="urn:adsk.eagle:library:334" deviceset="R-EU_" device="M5923" package3d_urn="urn:adsk.eagle:package:23564/1" value="100R"/>
-<part name="R111" library="rcl" library_urn="urn:adsk.eagle:library:334" deviceset="R-EU_" device="M5923" package3d_urn="urn:adsk.eagle:package:23564/1" value="100R"/>
-<part name="R101" library="rcl" library_urn="urn:adsk.eagle:library:334" deviceset="R-EU_" device="M5923" package3d_urn="urn:adsk.eagle:package:23564/1" value="100R"/>
-<part name="R103" library="rcl" library_urn="urn:adsk.eagle:library:334" deviceset="R-EU_" device="M5923" package3d_urn="urn:adsk.eagle:package:23564/1" value="100R"/>
-<part name="R105" library="rcl" library_urn="urn:adsk.eagle:library:334" deviceset="R-EU_" device="M5923" package3d_urn="urn:adsk.eagle:package:23564/1" value="100R"/>
-<part name="R107" library="rcl" library_urn="urn:adsk.eagle:library:334" deviceset="R-EU_" device="R0805" package3d_urn="urn:adsk.eagle:package:23553/2" value="2R"/>
+<part name="R104" library="rcl" library_urn="urn:adsk.eagle:library:334" deviceset="R-EU_" device="R1206" package3d_urn="urn:adsk.eagle:package:23540/2" value="100R"/>
+<part name="R111" library="rcl" library_urn="urn:adsk.eagle:library:334" deviceset="R-EU_" device="R1206" package3d_urn="urn:adsk.eagle:package:23540/2" value="100R"/>
+<part name="R101" library="rcl" library_urn="urn:adsk.eagle:library:334" deviceset="R-EU_" device="R1206" package3d_urn="urn:adsk.eagle:package:23540/2" value="100R"/>
+<part name="R103" library="rcl" library_urn="urn:adsk.eagle:library:334" deviceset="R-EU_" device="R1206" package3d_urn="urn:adsk.eagle:package:23540/2" value="100R"/>
+<part name="R105" library="rcl" library_urn="urn:adsk.eagle:library:334" deviceset="R-EU_" device="R1206" package3d_urn="urn:adsk.eagle:package:23540/2" value="100R"/>
+<part name="R107" library="rcl" library_urn="urn:adsk.eagle:library:334" deviceset="R-EU_" device="R1206" package3d_urn="urn:adsk.eagle:package:23540/2" value="2R"/>
 <part name="R106" library="rcl" library_urn="urn:adsk.eagle:library:334" deviceset="R-EU_" device="R6332" package3d_urn="urn:adsk.eagle:package:23559/2" value="0R004"/>
-<part name="R110" library="rcl" library_urn="urn:adsk.eagle:library:334" deviceset="R-EU_" device="M5923" package3d_urn="urn:adsk.eagle:package:23564/1" value="100R"/>
-<part name="R112" library="rcl" library_urn="urn:adsk.eagle:library:334" deviceset="R-EU_" device="M5923" package3d_urn="urn:adsk.eagle:package:23564/1" value="100R"/>
-<part name="R114" library="rcl" library_urn="urn:adsk.eagle:library:334" deviceset="R-EU_" device="R0805" package3d_urn="urn:adsk.eagle:package:23553/2" value="2R"/>
+<part name="R110" library="rcl" library_urn="urn:adsk.eagle:library:334" deviceset="R-EU_" device="R1206" package3d_urn="urn:adsk.eagle:package:23540/2" value="100R"/>
+<part name="R112" library="rcl" library_urn="urn:adsk.eagle:library:334" deviceset="R-EU_" device="R1206" package3d_urn="urn:adsk.eagle:package:23540/2" value="100R"/>
+<part name="R114" library="rcl" library_urn="urn:adsk.eagle:library:334" deviceset="R-EU_" device="R1206" package3d_urn="urn:adsk.eagle:package:23540/2" value="2R"/>
 <part name="R113" library="rcl" library_urn="urn:adsk.eagle:library:334" deviceset="R-EU_" device="R6332" package3d_urn="urn:adsk.eagle:package:23559/2" value="0R004"/>
 <part name="GND101" library="supply1" library_urn="urn:adsk.eagle:library:371" deviceset="GND" device=""/>
@@
 <part name="Q102" library="transistors" deviceset="SIRC10DP" device=""/>
 <part name="Q103" library="transistors" deviceset="SIRC10DP" device=""/>
-<part name="R102" library="rcl" library_urn="urn:adsk.eagle:library:334" deviceset="R-EU_" device="M5923" package3d_urn="urn:adsk.eagle:package:23564/1" value="100R"/>
-<part name="R109" library="rcl" library_urn="urn:adsk.eagle:library:334" deviceset="R-EU_" device="M5923" package3d_urn="urn:adsk.eagle:package:23564/1" value="100R"/>
+<part name="R102" library="rcl" library_urn="urn:adsk.eagle:library:334" deviceset="R-EU_" device="R1206" package3d_urn="urn:adsk.eagle:package:23540/2" value="100R"/>
+<part name="R109" library="rcl" library_urn="urn:adsk.eagle:library:334" deviceset="R-EU_" device="R1206" package3d_urn="urn:adsk.eagle:package:23540/2" value="100R"/>
 <part name="Q105" library="transistors" deviceset="SIRC10DP" device=""/>
 <part name="Q106" library="transistors" deviceset="SIRC10DP" device=""/>
