File: PCB/V1A/Electronic_Load_V1A.sch (EAGLE design)
At the start: 146 parts, among them IC201 OPA77P, IC202 OPA77P, IC203 OPA77P, IC204 OPA77P, IC205 OPA77P, IC301 MAX743CPE, IC302 7805T, IC303 7805T, IC304 7905, J101 +, J102 -, J103 +, J104 -, Q101 SIRC10DP, Q102 SIRC10DP, Q103 SIRC10DP, Q104 IXTK102N65X2PADUP-, Q105 SIRC10DP, Q106 SIRC10DP, Q107 SIRC10DP, Q108 IXTK102N65X2PADUP, U201 LTC1865-MSOP, U202 LTC1865-MSOP, U203 LTC1865-MSOP, U401 AD420, U402 AD420, U403 LT1014

Commit message: Added temp sensors
Parts:
- added C1, C3, C411, C412: 0.1µ, rcl:C-EUC0805
- added C2: 1µ, rcl:C-EUC0805
- added PAD103, PAD104: PAD-5X2, pads:PAD-5X2
- added Q401, Q403: BC817-25SMD, transistor-npn:BC817-25SMD
- added Q402: BC807-25SMD, transistor-pnp:BC807-25SMD
- added R1, R2, R411, R412, R413: 5k, rcl:R-EU_R0805
- added R3, R4, R5: 10k, rcl:R-EU_R0805
- added U1: LTC1865-MSOP, adc_dac:LTC1865-MSOP
- C301, C310, C311, L301, L302: value 100u -> 100µ
- C302, C401, C402, C409, C410: value 100n -> 0.1µ
- C303, C315: value 1u -> 1µ
- C305: value 10u -> 10µ
- C307, C312: value 0.33u -> 0.33µ
- C308, C314: value 0.1u -> 0.1µ
- C309: value 22u -> 22µ
- C313: value 2u2 -> 2µ2
- C403: value 10n -> 0.1µ
- C407: value 100n -> 10n
- C408: value 100n -> 500p
- R401: value 20k -> 1k; device rcl:R-TRIMM4G/J -> rcl:R-EU_R1206
- R402: value 20k -> 10k; device rcl:R-TRIMM4G/J -> rcl:R-EU_R1206
- R403: value 200k -> 1k; device rcl:R-EU_R0805 -> rcl:R-EU_R1206
- R404: value 200k -> 20k; device rcl:R-EU_R0805 -> rcl:R-TRIMM4G/J
- R405: value 100R -> 20k; device rcl:R-EU_R0805 -> rcl:R-TRIMM4G/J
- R406: value 100R -> 200k
- R407: value 5k -> 200k
- R408, R409: value 5k -> 100R
- renumbered PAD3 to PAD101, PAD4 to PAD105, PAD5 to PAD107, PAD6 to PAD106, PAD7 to PAD102
Connections:
- new net BYP_CTRL: C408.2, R403.1
- new net CLR_DAC1: U401.CLEAR
- new net CLR_DAC2: U402.CLEAR
- new net DAC1_OUT: U401.DATA_OUT, U402.DATA_IN
- new net DAC2_OUT: U402.DATA_OUT
- new net DAC_FAULT: R5.1, U401.FAULT, U402.FAULT
- new net N$47: R2.2, R4.1, U403G4.-IN
- new net N$49: R1.2, R3.1, U403G3.-IN
- new net N$93: Q401.B, Q402.B, Q403.C, R401.1
- new net N$94: C403.1, Q401.C, R401.2, R402.2
- new net N$95: C403.2, Q402.C, Q403.E
- new net N$96: C408.1, Q403.B, R402.1, R403.2
- new net SS_ADC_T: U1.CONV
- new net SS_DAC: U401.LATCH, U402.LATCH
- new net TEMP1_AMP: R3.2, U1.CH0, U403G3.OUT
- new net TEMP1_IN: PAD1.P, U403G3.+IN
- new net TEMP2_AMP: R4.2, U1.CH1, U403G4.OUT
- new net TEMP2_IN: PAD2.P, U403G4.+IN
- net +12V: now also C407.2, C409.1, C410.1; no longer C403.2, C407.1, C408.1
- net +15V: now also C411.1; no longer C409.1
- net +5V: now also C1.1, C2.1, R5.2, U1.VCC
- net +5V/1: now also R404.E, R405.E; no longer R401.E, R402.E
- net -15V: now also C412.1; no longer C410.1
- net -5V: now also C3.2, R404.A, R405.A; no longer R401.A, R402.A
- net BYP_G: now also Q401.E, Q402.E
- net GND: now also C1.2, C2.2, C3.1, C411.2, C412.2, R1.1, R2.1, R408.1, R409.1, U1.AGND, U1.DGND; no longer C407.2, C408.2, R405.1, R406.1
- net LOAD_G1: now also R412.2; no longer R409.2
- net LOAD_G2: now also R413.2; no longer R410.2
- net MISO: now also U1.SDO
- net MOSI: now also U1.SDI, U401.DATA_IN
- net N$24: now also C407.1; no longer C406.1
- net N$25: now also C404.1; no longer C403.1
- net N$26: now also C405.1; no longer C404.1
- net N$27: now also C406.1; no longer C405.1
- net N$28: now also R410.2, R412.1; no longer R407.2, R409.1
- net N$29: now also R411.2, R413.1; no longer R408.2, R410.1
- net N$32: now also R406.2, R408.2, R410.1; no longer R403.2, R405.2, R407.1
- net N$33: now also R404.S, R406.1; no longer R401.S, R403.1
- net N$34: now also R405.S, R407.1; no longer R402.S, R404.1
- net N$35: now also R407.2, R409.2, R411.1; no longer R404.2, R406.2, R408.1
- net SCK: now also U1.SCK, U401.CLOCK, U402.CLOCK
- net VREF: now also U1.VREF
- net VSENSE+: now also PAD103.P; no longer PAD1.P
- net VSENSE-: now also PAD104.P; no longer PAD2.P
Other:
- moved on the sheet: C401, C402, C403, C404, C405, C406, C407, C408, C409, C410, D303, D304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

Commit message: Changed packages, board layout
Changed component packages and values to the ones that are available. Moved the heatsink mount back to the PCB,
Parts:
- added PAD3: PAD-10X4, pads:PAD-10X4
- C1, C201, C202, C203, C204, C205, C206, C208, C210, C211, C212, C213, C214, C216, C3, C302, C307, C308, C312, C314, C401, C402, C403, C408, C409, C411, C412: device rcl:C-EUC0805 -> rcl:C-EUC1206
- C2: device rcl:C-EUC0805 -> rcl:CPOL-EUSMCA
- C207, C209, C215: device rcl:CPOL-EUSMCC -> rcl:CPOL-EUSMCA
- C301, C310, C311: value 100µ -> 220µ; device rcl:CPOL-EU085CS-1AR -> rcl:CPOL-EUE3.5-10
- C303, C313, C315: device rcl:CPOL-EU085CS-1AR -> rcl:CPOL-EUSMCA
- C305: device rcl:CPOL-EU085CS-1AR -> rcl:CPOL-EUSMCC
- C309: device rcl:CPOL-EU085CS-1AR -> rcl:CPOL-EUSMCD
- Q104: value IXTK102N65X2PADUP- -> IXTK102N65X2PADUP; device transistors:IXTK102N65X2PADUP- -> transistors:IXTK102N65X2PADUP
- R1, R2, R204, R205, R206, R207, R217, R220, R221, R224, R225, R227, R228, R229, R230, R3, R4, R410, R411, R412, R413, R5: device rcl:R-EU_R0805 -> rcl:R-EU_R0603
- R201, R202, R203, R208, R209, R210, R211, R212, R213, R214, R215, R216, R218, R219, R231, R232, R233, R234, R406, R407, R408, R409: device rcl:R-EU_R0805 -> rcl:R-EU_R1206
- R401, R402, R403: device rcl:R-EU_R1206 -> rcl:R-EU_R0603
Connections:
- net +5V: now also C2.+; no longer C2.1
- net DUT_+1: now also PAD3.P
- net GND: now also C2.-; no longer C2.2

Commit message: Updated part list
Parts:
- removed PAD3: PAD-10X4, pads:PAD-10X4
- removed R1: 5k, rcl:R-EU_R0603
- removed R5: 10k, rcl:R-EU_R0603
- added C415, C416: 0.1µ, rcl:C-EUC1206
- added IC305, IC306: LM50, linear:LM50
- added IC401: OPA77P, burr-brown:OPA77P
- added PAD108: PAD-10X4, pads:PAD-10X4
- added R415, R416: 5k, rcl:R-EU_R0603
- added R419, R420, R421, R422: 20k, rcl:R-EU_R0603
- added R423: 20k, rcl:R-TRIMM4G/J
- R404: value 20k -> 10k; device rcl:R-TRIMM4G/J -> rcl:R-EU_R0603
- R406: value 200k -> 20k; device rcl:R-EU_R1206 -> rcl:R-TRIMM4G/J
- R408: value 100R -> 200k
- R410: value 5k -> 100R; device rcl:R-EU_R0603 -> rcl:R-EU_R1206
- renumbered C1 to C413, C2 to C414, C3 to C316, PAD1 to PAD401, PAD2 to PAD402, R2 to R414, R3 to R417, R4 to R418, U1 to U404
Connections:
- removed net N$32 (its old number): R406.2, R408.2, R410.1
- removed net N$33 (its old number): R404.S, R406.1
- new net N$34: R406.S, R408.1
- new net N$35: R408.2, R410.2, R412.1
- new net N$48: IC401.+IN, R420.1, R421.2
- new net N$50: R419.2, R421.1, R422.2
- new net N$51: IC401.TRIM2, R423.E
- new net N$53: IC401.TRIM1, R423.A
- new net N$90: U404.VREF
- new net TEMP1: IC305.VO
- new net TEMP2: IC306.VO
- new net VREF3.0: IC401.-IN, IC401.OUT
- net +15V: now also C415.1, IC401.V+, R423.S
- net +5V: now also IC305.+VS, IC306.+VS, R404.2; no longer R5.2
- net +5V/1: now also R406.E; no longer R404.E
- net -15V: now also C416.1, IC401.V-
- net -5V: now also R406.A; no longer R404.A
- net DAC_FAULT: now also R404.1; no longer R5.1
- net DUT_+1: now also PAD107.P; no longer PAD3.P
- net GND: now also C415.2, C416.2, IC305.GND, IC306.GND, PAD108.P, R410.1, R413.1, R419.1, R422.1; no longer PAD107.P, R1.1, R408.1
- net LOAD_G1: now also R415.2; no longer R412.2
- net LOAD_G2: now also R416.2; no longer R413.2
- net N$28: now also R411.2, R415.1; no longer R410.2, R412.1
- net N$29: now also R412.2, R416.1; no longer R411.2, R413.1
- net N$49: now also R413.2; no longer R1.2
- net VREF: now also R420.2; no longer U404.VREF
Other:
- moved on the sheet: PAD107, R405, R407, R408, R409, R410, R411, R412, R413

Commit message: Changed OPA77 to AD620
Parts:
- added C501, C502, C503, C504, C505, C506, C507, C508, C511, C512: 0.1µ, rcl:C-EUC1206
- added C509, C510: 1µ, rcl:CPOL-EUSMCA
- added IC501, IC502, IC503, IC504: AD620R, analog-devices:AD620R
- added R501, R502, R503, R504: 2k61, rcl:R-EU_R1206
- added U501, U502: LTC1865L, adc_dac:LTC1865L
Connections:
- new net +3V3: C509.+, C510.+, C511.1, C512.1, U501.VCC, U502.VCC
- new net CSENSE_H1_AMP1: IC503.OUT, U502.CH0
- new net CSENSE_H2_AMP1: IC504.OUT, U502.CH1
- new net MISO_ISO: U501.SDO, U502.SDO
- new net MOSI_ISO: U501.SDI, U502.SDI
- new net RG1_H1: IC501.RG@1, R501.2
- new net RG1_H2: IC502.RG@1, R502.2
- new net RG1_L1: IC503.RG@1, R503.2
- new net RG1_L2: IC504.RG@1, R504.2
- new net RG2_H1: IC501.RG@2, R501.1
- new net RG2_H2: IC502.RG@2, R502.1
- new net RG2_L1: IC503.RG@2, R503.1
- new net RG2_L2: IC504.RG@2, R504.1
- new net SCK_ISO: U501.SCK, U502.SCK
- new net SS_CH_ISO: U501.CONV
- new net SS_CL_ISO: U502.CONV
- net +15V: now also C501.1, C502.1, C503.1, C504.1, IC501.+V, IC502.+V, IC503.+V, IC504.+V
- net -15V: now also C505.1, C506.1, C507.1, C508.1, IC501.-V, IC502.-V, IC503.-V, IC504.-V
- net CSENSE_H1: now also IC501.+, IC503.-
- net CSENSE_H1_AMP: now also IC501.OUT, U501.CH0
- net CSENSE_H2: now also IC502.+, IC504.-
- net CSENSE_H2_AMP: now also IC502.OUT, U501.CH1
- net CSENSE_L1: now also IC503.+
- net CSENSE_L2: now also IC504.+
- net GND: now also C501.2, C502.2, C503.2, C504.2, C505.2, C506.2, C507.2, C508.2, C509.-, C510.-, C511.2, C512.2, IC501.-, IC501.REF, IC502.-, IC502.REF, IC503.REF, IC504.REF, U501.GND, U502.GND

Commit message: Added optocouplers
Parts:
- removed C315: 1µ, rcl:CPOL-EUSMCA
- removed C316: 0.1µ, rcl:C-EUC1206
- removed D301, D302: 1N5817-B, diode:1N5817-B
- removed D303, D304: 1N4004, diode:1N4004
- removed IC302, IC303: 7805T, linear:7805T
- removed IC304: 7905, linear:7905T
- removed IC305, IC306: LM50, linear:LM50
- removed IC501, IC502, IC503, IC504: AD620R, analog-devices:AD620R
- removed J301: (no value), con-jack:JACK-PLUG0
- removed L301, L302: 100µ, rcl:L-EU0204/5
- removed PAD401, PAD402: PAD-5X2, pads:PAD-5X2
- removed Q401, Q403: BC817-25SMD, transistor-npn:BC817-25SMD
- removed Q402: BC807-25SMD, transistor-pnp:BC807-25SMD
- removed R201, R202, R203, R208, R209, R210, R211, R212, R213, R214, R215, R216, R218, R219, R231, R232, R233, R234: 200k, rcl:R-EU_R1206
- removed R204, R205, R206, R207, R227, R228, R229, R230, R412, R413, R414, R415, R416: 5k, rcl:R-EU_R0603
- removed R217, R419, R420, R421, R422: 20k, rcl:R-EU_R0603
- removed R220, R221, R224, R225, R417, R418: 10k, rcl:R-EU_R0603
- removed R222, R223, R226, R235, R236, R423: 20k, rcl:R-TRIMM4G/J
- removed U201, U202, U203: LTC1865-MSOP, adc_dac:LTC1865-MSOP
- added C1, C421, C422, C5, C9: 0.1µ, rcl:C-EUC1206
- added C10, C2, C6: 0.01µ, rcl:C-EUC1206
- added C11, C12, C3, C4, C7, C8: 15p, rcl:C-EUC1206
- added C13, C14, C15, C16, C17, C18, C19: 500p, rcl:C-EUC1206
- added C417, C418, C419, C420: 1µ, rcl:CPOL-EUSMCA
- added D201, D202: 1N5817-B, diode:1N5817-B
- added D203, D204: 1N4004, diode:1N4004
- added IC206, IC405, IC406: LM50, linear:LM50
- added IC402, IC403, IC404, IC407: AD620R, analog-devices:AD620R
- added J201: (no value), con-jack:JACK-PLUG0
- added L201, L202: 100µ, rcl:L-EU0204/5
- added Q1, Q2, Q3, Q4, Q5, Q501, Q502, Q503, Q504, Q505, Q506, Q6: BC807-16SMD, transistor-pnp:BC807-16SMD
- added Q301, Q303: BC817-25SMD, transistor-npn:BC817-25SMD
- added Q302: BC807-25SMD, transistor-pnp:BC807-25SMD
- added R1, R10, R11, R12, R2, R3, R4, R5, R505, R506, R507, R508, R509, R510, R511, R512, R6, R7, R8, R9: 350R, rcl:R-EU_R1206
- added R13, R14, R15, R16, R17, R18, R19, R309, R310: 100R, rcl:R-EU_R1206
- added R301, R303: 1k, rcl:R-EU_R0603
- added R302, R304: 10k, rcl:R-EU_R0603
- added R305, R306, R319: 20k, rcl:R-TRIMM4G/J
- added R307, R308: 200k, rcl:R-EU_R1206
- added R311, R312, R313, R314: 5k, rcl:R-EU_R0603
- added R315, R316, R317, R318: 20k, rcl:R-EU_R0603
- added U1, U2, U3, U503: HCPL-063N, isolation:HCPL-063N
- added U301, U302: AD420, adc_dac:AD420
- added U303: LT1014, SparkFun-Retired:LT1014
- C201, C210, C211: value 0.1µ -> 220µ; device rcl:C-EUC1206 -> rcl:CPOL-EUE3.5-10
- C203, C409: value 0.1µ -> 1µ; device rcl:C-EUC1206 -> rcl:CPOL-EUSMCA
- C204, C206: value 0.1µ -> 10n; device rcl:C-EUC1206 -> rcl:C-EUC0805
- C205: value 0.1µ -> 10µ; device rcl:C-EUC1206 -> rcl:CPOL-EUSMCC
- C207: value 1µ -> 0.33µ; device rcl:CPOL-EUSMCA -> rcl:C-EUC1206
- C209: value 1µ -> 22µ; device rcl:CPOL-EUSMCA -> rcl:CPOL-EUSMCD
- C212: value 0.1µ -> 0.33µ
- C213: value 0.1µ -> 2µ2; device rcl:C-EUC1206 -> rcl:CPOL-EUSMCA
- C301, C311: value 220µ -> 0.1µ; device rcl:CPOL-EUE3.5-10 -> rcl:C-EUC1206
- C303, C414: value 1µ -> 0.1µ; device rcl:CPOL-EUSMCA -> rcl:C-EUC1206
- C305: value 10µ -> 10n; device rcl:CPOL-EUSMCC -> rcl:C-EUC0805
- C307: value 0.33µ -> 10n; device rcl:C-EUC1206 -> rcl:C-EUC0805
- C308: value 0.1µ -> 500p
- C309: value 22µ -> 0.1µ; device rcl:CPOL-EUSMCD -> rcl:C-EUC1206
- C310: value 220µ -> 0.1µ; device rcl:CPOL-EUE3.5-10 -> rcl:C-EUC0805
- C312: value 0.33µ -> 0.1µ
- C313: value 2µ2 -> 0.1µ; device rcl:CPOL-EUSMCA -> rcl:C-EUC1206
- C404, C405, C406, C407: value 10n -> 0.1µ; device rcl:C-EUC0805 -> rcl:C-EUC1206
- C408: value 500p -> 0.1µ
- C410: value 0.1µ -> 1µ; device rcl:C-EUC0805 -> rcl:CPOL-EUSMCA
- C504, C505, C506: value 0.1µ -> 0.01µ
- C507, C508, C511, C512: value 0.1µ -> 15p
- C509, C510: value 1µ -> 15p; device rcl:CPOL-EUSMCA -> rcl:C-EUC1206
- IC201: value OPA77P -> MAX743CPE; device burr-brown:OPA77P -> maxim:MAX743CPE
- IC202, IC203: value OPA77P -> 7805T; device burr-brown:OPA77P -> linear:7805T
- IC204: value OPA77P -> 7905; device burr-brown:OPA77P -> linear:7905T
- IC205: value OPA77P -> LM50; device burr-brown:OPA77P -> linear:LM50
- IC301: value MAX743CPE -> OPA77P; device maxim:MAX743CPE -> burr-brown:OPA77P
- IC401: value OPA77P -> AD620R; device burr-brown:OPA77P -> analog-devices:AD620R
- R401, R403: value 1k -> 2k15; device rcl:R-EU_R0603 -> rcl:R-EU_R1206
- R402, R404: value 10k -> 2k15; device rcl:R-EU_R0603 -> rcl:R-EU_R1206
- R405, R406: value 20k -> 2M; device rcl:R-TRIMM4G/J -> rcl:R-EU_R1206
- R407, R408: value 200k -> 2M
- R409: value 100R -> 2M
- R410: value 100R -> 2k15
- R411: value 5k -> 2k15; device rcl:R-EU_R0603 -> rcl:R-EU_R1206
- R501, R502, R503, R504: value 2k61 -> 350R
- U401, U402: value AD420 -> LTC1865L; device adc_dac:AD420 -> adc_dac:LTC1865L
- U403: value LT1014 -> LTC1865L; device SparkFun-Retired:LT1014 -> adc_dac:LTC1865L
- U404: value LTC1865-MSOP -> LTC1865L; device adc_dac:LTC1865-MSOP -> adc_dac:LTC1865L
- U501, U502: value LTC1865L -> HCPL-063N; device adc_dac:LTC1865L -> isolation:HCPL-063N
Connections:
- removed net CLR_DAC1: U401.CLEAR
- removed net CLR_DAC2: U402.CLEAR
- removed net CSENSE_H1_AMP: IC201.OUT, IC501.OUT, R218.2, U201.CH0, U501.CH0
- removed net CSENSE_H1_AMP1: IC503.OUT, U502.CH0
- removed net CSENSE_H2_AMP: IC202.OUT, IC502.OUT, R219.2, U201.CH1, U501.CH1
- removed net CSENSE_H2_AMP1: IC504.OUT, U502.CH1
- removed net CSENSE_L1_AMP: IC204.OUT, R233.2, U203.CH0
- removed net CSENSE_L2_AMP: IC205.OUT, R234.2, U203.CH1
- removed net N$85: R209.1, R210.2
- removed net N$86: R208.1, R209.2
- removed net N$87: R201.2, R208.2
- removed net N$88: R201.1, R202.2
- removed net N$89: R202.1, R203.2
- removed net N$90: U404.VREF
- removed net N$91: IC203.+IN, R220.2, R221.2
- removed net N$92: IC203.-IN, R224.2, R225.1
- removed net SS_ADC_H: U201.CONV
- removed net SS_ADC_L: U203.CONV
- removed net SS_ADC_T: U404.CONV
- removed net SS_ADC_V: U202.CONV
- removed net TEMP1_AMP: R417.2, U403G3.OUT, U404.CH0
- removed net TEMP1_IN: PAD401.P, U403G3.+IN
- removed net TEMP2_AMP: R418.2, U403G4.OUT, U404.CH1
- removed net TEMP2_IN: PAD402.P, U403G4.+IN
- removed net VSENSE: IC203.OUT, R225.2, U202.CH0
- new net BYP_G_ISO: C8.1, Q301.E, Q302.E, R6.1, U2.VO2
- new net DAC_CLR: Q5.B
- new net DAC_CLR_ISO: C11.1, R9.1, U3.VO1
- new net DAC_FAULT_ISO: Q2.B, R304.1, U301.FAULT, U302.FAULT
- new net N$100: R408.1, R409.2
- new net N$101: IC407.+, R409.1, R410.2
- new net N$97: R405.2, R407.1
- new net N$98: R406.1, R407.2
- new net N$99: R406.2, R408.2
- new net RG1_H3: IC407.RG@1, R411.2
- new net RG2_H3: IC407.RG@2, R411.1
- new net SS_CH: Q502.B
- new net SS_CL: Q505.B
- new net SS_DAC_ISO: C7.1, R5.1, U2.VO1
- new net SS_TEMP: Q506.B
- new net SS_TEMP_ISO: C512.1, R512.1, U403.CONV, U503.VO2
- new net SS_V: Q503.B
- new net SS_V_ISO: C509.1, R509.1, U404.CONV, U503.VO1
- new net VSENSE_AMP: IC407.OUT
- net +12V: now also C201.+, C207.1, C304.2, C305.2, C306.2, C307.2, C309.1, C310.1, IC202.VI, J201.3, U301.VCC, U302.VCC; no longer C301.+, C307.1, C404.2, C405.2, C406.2, C407.2, C409.1, C410.1, IC302.VI, J301.3, U401.VCC, U402.VCC
- net +15V: now also C210.+, C311.1, C313.1, C401.1, C402.1, C403.1, C404.1, D201.C, IC201.FB+, IC203.VI, IC301.V+, IC401.+V, IC402.+V, IC403.+V, IC404.+V, IC407.+V, R319.S, U303G1.+V; no longer C201.1, C202.1, C205.1, C211.1, C310.+, C312.1, C411.1, C501.1, C502.1, C503.1, C504.1, D301.C, IC201.V+, IC202.V+, IC203.V+, IC204.V+, IC205.V+, IC301.FB+, IC303.VI, IC401.V+, IC501.+V, IC502.+V, IC503.+V, IC504.+V, R222.S, R223.S, R226.S, R235.S, R236.S, R423.S, U403G1.+V
- net +3V3: now also C409.+, C410.+, C411.1, C412.1, C419.+, C420.+, C421.1, C422.1, U401.VCC, U402.VCC, U403.VCC, U404.VCC; no longer C509.+, C510.+, C511.1, C512.1, U501.VCC, U502.VCC
- net +5V: now also C1.1, C10.1, C2.1, C202.2, C301.1, C302.1, C414.1, C5.1, C501.1, C502.1, C503.1, C504.1, C505.1, C506.1, C6.1, C9.1, IC201.AV+, IC201.V+, IC201.V+@1, IC201.V+@2, IC201.V+@3, IC202.VO, IC205.+VS, IC206.+VS, IC405.+VS, IC406.+VS, L202.1, R1.2, R10.2, R11.2, R12.2, R2.2, R3.2, R304.2, R4.2, R5.2, R501.2, R502.2, R503.2, R504.2, R505.2, R506.2, R507.2, R508.2, R509.2, R510.2, R511.2, R512.2, R6.2, R7.2, R8.2, R9.2, U1.VCC, U2.VCC, U3.VCC, U301.VLL, U302.VLL, U501.VCC, U502.VCC, U503.VCC; no longer C207.+, C210.1, C215.+, C216.1, C302.2, C308.1, C309.+, C401.1, C402.1, C414.+, IC301.AV+, IC301.V+, IC301.V+@1, IC301.V+@2, IC301.V+@3, IC302.VO, IC305.+VS, IC306.+VS, L302.1, R404.2, U201.VCC, U202.VCC, U203.VCC, U401.VLL, U402.VLL, U404.VCC
- net +5V/1: now also C214.1, D203.C, IC203.VO, R305.E, R306.E; no longer C314.1, D303.C, IC303.VO, R405.E, R406.E
- net -15V: now also C211.-, C213.-, C312.1, C314.1, C405.1, C406.1, C407.1, C408.1, D202.A, IC201.FB-, IC204.VI, IC301.V-, IC401.-V, IC402.-V, IC403.-V, IC404.-V, IC407.-V, U303G1.-V; no longer C203.1, C204.1, C206.1, C213.1, C214.1, C311.-, C313.-, C412.1, C505.1, C506.1, C507.1, C508.1, D302.A, IC201.V-, IC202.V-, IC203.V-, IC204.V-, IC205.V-, IC301.FB-, IC304.VI, IC401.V-, IC501.-V, IC502.-V, IC503.-V, IC504.-V, U403G1.-V
- net -5V: now also C215.-, C216.2, D204.A, IC204.VO, R305.A, R306.A; no longer C315.-, C316.2, D304.A, IC304.VO, R405.A, R406.A
- net BYP_CTRL: now also C308.2, R101.1, R303.1; no longer C408.2, R403.1
- net BYP_G: now also Q4.B; no longer Q401.E, Q402.E, R101.1
- net CSENSE_H1: now also IC401.+, IC403.-; no longer IC501.+, IC503.-, R204.1, R228.1
- net CSENSE_H2: now also IC402.+, IC404.-; no longer IC502.+, IC504.-, R206.1, R230.1
- net CSENSE_L1: now also IC403.+; no longer IC503.+, R227.1
- net CSENSE_L2: now also IC404.+; no longer IC504.+, R229.1
- net DAC1_OUT: now also U301.DATA_OUT, U302.DATA_IN; no longer U401.DATA_OUT, U402.DATA_IN
- net DAC2_OUT: now also U302.DATA_OUT; no longer U402.DATA_OUT
- net DAC_FAULT: now also C4.1, R2.1, U1.VO2; no longer R404.1, U401.FAULT, U402.FAULT
- net GND: now also C1.2, C10.2, C11.2, C12.2, C13.2, C14.2, C15.2, C16.2, C17.2, C18.2, C19.2, C2.2, C201.-, C202.1, C203.-, C204.1, C205.-, C210.-, C211.+, C213.+, C215.+, C216.1, C3.2, C301.2, C302.2, C309.2, C310.2, C311.2, C313.2, C4.2, C403.2, C404.2, C405.2, C406.2, C407.2, C408.2, C409.-, C410.-, C414.2, C417.-, C418.-, C419.-, C420.-, C421.2, C422.2, C5.2, C509.2, C510.2, C6.2, C7.2, C8.2, C9.2, D203.A, D204.C, IC201.12/15, IC201.AGND, IC201.GND, IC203.GND, IC204.GND, IC205.GND, IC206.GND, IC401.-, IC401.REF, IC402.-, IC402.REF, IC403.REF, IC404.REF, IC405.GND, IC406.GND, IC407.REF, J201.1, J201.2, L201.2, Q1.C, Q2.C, Q3.C, Q4.C, Q5.C, Q501.C, Q502.C, Q503.C, Q504.C, Q505.C, Q506.C, Q6.C, R309.1, R310.1, R315.1, R318.1, U1.C1, U1.C2, U1.GND, U2.C1, U2.C2, U2.GND, U3.C1, U3.C2, U3.GND, U301.GND, U301.RS1, U301.RS2, U302.GND, U302.RS1, U302.RS2, U403.GND, U404.GND, U501.C1, U501.C2, U502.C1, U502.C2, U503.C1, U503.C2, U503.GND; no longer C201.2, C202.2, C203.2, C204.2, C205.2, C207.-, C208.2, C210.2, C211.2, C213.2, C215.-, C216.2, C301.-, C302.1, C303.-, C304.1, C305.-, C306.2, C309.-, C310.-, C311.+, C313.+, C315.+, C316.1, C409.2, C410.2, C414.-, C509.-, C510.-, D303.A, D304.C, IC301.12/15, IC301.AGND, IC301.GND, IC303.GND, IC304.GND, IC305.GND, IC306.GND, IC501.-, IC501.REF, IC502.-, IC502.REF, IC503.REF, IC504.REF, J301.1, J301.2, L301.2, R205.1, R207.1, R214.1, R215.1, R217.1, R221.1, R231.1, R232.1, R409.1, R413.1, R414.1, R419.1, R422.1, U201.AGND, U201.DGND, U202.AGND, U202.DGND, U203.AGND, U203.DGND, U401.RS1, U401.RS2, U402.RS1, U402.RS2, U404.AGND, U404.DGND
- net LOAD_G1: now also R313.2, U303G1.OUT; no longer R415.2, U403G1.OUT
- net LOAD_G2: now also R314.2, U303G2.OUT; no longer R416.2, U403G2.OUT
- net MISO: now also C3.1, R1.1, U1.VO1; no longer U201.SDO, U202.SDO, U203.SDO, U404.SDO
- net MISO_ISO: now also Q1.B, U401.SDO, U402.SDO, U403.SDO, U404.SDO; no longer U501.SDO, U502.SDO
- net MOSI: now also Q504.B, U301.DATA_IN; no longer U201.SDI, U202.SDI, U203.SDI, U401.DATA_IN, U404.SDI
- net MOSI_ISO: now also C510.1, R510.1, U401.SDI, U402.SDI, U403.SDI, U404.SDI, U501.VO2; no longer U501.SDI, U502.SDI
- net N$24: now also C307.1, U302.CAP2; no longer C407.1, U402.CAP2
- net N$25: now also C304.1, U301.CAP1; no longer C404.1, U401.CAP1
- net N$26: now also C305.1, U302.CAP1; no longer C405.1, U402.CAP1
- net N$27: now also C306.1, U301.CAP2; no longer C406.1, U401.CAP2
- net N$28: now also R311.2, R313.1, U303G1.-IN; no longer R411.2, R415.1, U403G1.-IN
- net N$29: now also R312.2, R314.1, U303G2.-IN; no longer R412.2, R416.1, U403G2.-IN
- net N$32: now also R307.2, R309.2, R311.1; no longer R407.2, R409.2, R411.1
- net N$33: now also R305.S, R307.1; no longer R405.S, R407.1
- net N$34: now also R306.S, R308.1; no longer R406.S, R408.1
- net N$35: now also R308.2, R310.2, R312.1; no longer R408.2, R410.2, R412.1
- net N$36: now also D201.A, IC201.LX+, L202.2; no longer D301.A, IC301.LX+, L302.2
- net N$37: now also C206.1, IC201.CC-; no longer C306.1, IC301.CC-
- net N$38: now also C203.+, IC201.SS; no longer C303.+, IC301.SS
- net N$39: now also D202.C, IC201.LX-, L201.1; no longer D302.C, IC301.LX-, L301.1
- net N$40: now also C204.2, IC201.CC+; no longer C304.2, IC301.CC+
- net N$44: now also C207.2, C208.2, IC202.GND; no longer C307.2, C308.2, IC302.GND
- net N$47: now also Q501.E, R501.1, U501.A1; no longer R414.2, R418.1, U403G4.-IN
- net N$48: now also IC301.+IN, R316.1, R317.2; no longer IC401.+IN, R420.1, R421.2
- net N$49: now also Q502.E, R502.1, U502.A1; no longer R413.2, R417.1, U403G3.-IN
- net N$50: now also R315.2, R317.1, R318.2; no longer R419.2, R421.1, R422.2
- net N$51: now also IC301.TRIM2, R319.E; no longer IC401.TRIM2, R423.E
- net N$53: now also IC301.TRIM1, R319.A; no longer IC401.TRIM1, R423.A
- net N$62: now also Q504.E, R504.1, U501.A2; no longer R216.1, R217.2, R220.1
- net N$63: now also Q505.E, R505.1, U502.A2; no longer IC203.TRIM1, R226.A
- net N$64: now also Q503.E, R503.1, U503.A1; no longer IC204.-IN, R228.2, R233.1
- net N$65: now also Q506.E, R506.1, U503.A2; no longer IC204.+IN, R227.2, R231.2
- net N$66: now also Q1.E, R3.1, U1.A1; no longer IC201.-IN, R205.2, R218.1
- net N$67: now also Q2.E, R4.1, U1.A2; no longer IC201.+IN, R204.2, R214.2
- net N$68: now also Q5.E, R11.1, U3.A1; no longer IC204.TRIM1, R235.A
- net N$69: now also Q6.E, R12.1, U3.A2; no longer IC201.TRIM1, R222.A
- net N$70: now also IC401.OUT, R13.1; no longer IC201.TRIM2, R222.E
- net N$71: now also Q6.B; no longer IC204.TRIM2, R235.E
- net N$72: now also C13.1, R13.2, U401.CH0; no longer IC203.TRIM2, R226.E
- net N$73: now also C12.1, R10.1, U3.VO2; no longer R211.2, R216.2
- net N$74: now also IC402.OUT, R14.1; no longer IC202.-IN, R207.2, R219.1
- net N$75: now also C14.1, R14.2, U401.CH1; no longer IC202.+IN, R206.2, R215.2
- net N$76: now also Q3.E, R7.1, U2.A1; no longer IC202.TRIM1, R223.A
- net N$77: now also Q4.E, R8.1, U2.A2; no longer IC202.TRIM2, R223.E
- net N$78: now also C15.1, R15.2, U402.CH0; no longer R211.1, R212.2
- net N$79: now also C16.1, R16.2, U402.CH1; no longer R212.1, R213.2
- net N$80: now also IC404.OUT, R16.1; no longer IC205.-IN, R230.2, R234.1
- net N$81: now also IC403.OUT, R15.1; no longer IC205.+IN, R229.2, R232.2
- net N$82: now also C17.1, R17.2, U403.CH0; no longer IC205.TRIM1, R236.A
- net N$83: now also C18.1, R18.2, U404.CH0; no longer IC205.TRIM2, R236.E
- net N$84: now also C19.1, R19.2, U403.CH1; no longer R210.1, R213.1
- net N$93: now also Q301.B, Q302.B, Q303.C, R301.1; no longer Q401.B, Q402.B, Q403.C, R401.1
- net N$94: now also C303.1, Q301.C, R301.2, R302.2; no longer C403.1, Q401.C, R401.2, R402.2
- net N$95: now also C303.2, Q302.C, Q303.E; no longer C403.2, Q402.C, Q403.E
- net N$96: now also C308.1, Q303.B, R302.1, R303.2; no longer C408.1, Q403.B, R402.1, R403.2
- net RG1_H1: now also IC401.RG@1, R401.2; no longer IC501.RG@1, R501.2
- net RG1_H2: now also IC402.RG@1, R402.2; no longer IC502.RG@1, R502.2
- net RG1_L1: now also IC403.RG@1, R403.2; no longer IC503.RG@1, R503.2
- net RG1_L2: now also IC404.RG@1, R404.2; no longer IC504.RG@1, R504.2
- net RG2_H1: now also IC401.RG@2, R401.1; no longer IC501.RG@2, R501.1
- net RG2_H2: now also IC402.RG@2, R402.1; no longer IC502.RG@2, R502.1
- net RG2_L1: now also IC403.RG@2, R403.1; no longer IC503.RG@2, R503.1
- net RG2_L2: now also IC404.RG@2, R404.1; no longer IC504.RG@2, R504.1
- net SCK: now also Q501.B, U301.CLOCK, U302.CLOCK; no longer U201.SCK, U202.SCK, U203.SCK, U401.CLOCK, U402.CLOCK, U404.SCK
- net SCK_ISO: now also C507.1, R507.1, U401.SCK, U402.SCK, U403.SCK, U404.SCK, U501.VO1; no longer U501.SCK, U502.SCK
- net SS_CH_ISO: now also C508.1, R508.1, U401.CONV, U502.VO1; no longer U501.CONV
- net SS_CL_ISO: now also C511.1, R511.1, U402.CONV, U502.VO2; no longer U502.CONV
- net SS_DAC: now also Q3.B; no longer U401.LATCH, U402.LATCH
- net TEMP1: now also C417.+, IC205.VO, IC405.VO; no longer IC305.VO
- net TEMP2: now also C418.+, IC206.VO, IC406.VO, R19.1; no longer IC306.VO
- net VGATE_1: now also U301.VOUT, U303G1.+IN; no longer U401.VOUT, U403G1.+IN
- net VGATE_2: now also U302.VOUT, U303G2.+IN; no longer U402.VOUT, U403G2.+IN
- net VREF: now also C205.+, IC201.VREF, R316.2, U301.REF_IN, U301.REF_OUT, U302.REF_IN; no longer C305.+, IC301.VREF, R420.2, U201.VREF, U202.VREF, U203.VREF, U401.REF_IN, U401.REF_OUT, U402.REF_IN
- net VREF3.0: now also IC301.-IN, IC301.OUT; no longer IC401.-IN, IC401.OUT
- net VSENSE+: now also R405.1; no longer R203.1
- net VSENSE-: now also IC407.-; no longer R224.1
Other:
- note added: "Temperature"
- note added: "Voltage sense input (1V-500V) is divided down to 215µV-107mV, which is then amplified to a range of 5.15mV-2.58V and sampled by the ADC with 3V reference. Input voltage step is 8.88mV@16bit, 35.53mV@14-bit. Current range 50mA-50A through a 2mΩ sense resistor has a voltage range of 100µV-100mV, which is then amplified to a range of 2.40mV-2.40V and sampled by the ADC with 3V reference. Current ste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"
- moved on the sheet: C202, C204, C206, C208, C209, C212, C214, C215, C216, C302, C304, C306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
