File: PCB/V1A/Electronic_Load_V1A.sch (EAGLE design)
At the start: 238 parts, among them IC1 MEGA8-AI, IC101 LM50, IC102 LM50, IC301 7805T, IC302 7805T, Q101 SIRC10DP, Q102 SIRC10DP, Q103 BC817-16SMD, Q104 BC817-16SMD, Q105 BC807-16SMD, Q106 SIRC10DP, Q107 IXTK102N65X2R+, Q108 SIRC10DP, Q109 SIRC10DP, Q110 SIRC10DP, Q111 IXTK102N65X2R+, Q601 BC807-16SMD, Q602 BC807-16SMD, Q603 BC807-16SMD, Q604 BC807-16SMD, Q605 BC807-16SMD, Q606 BC807-16SMD, Q607 BC807-16SMD, Q608 BC807-16SMD, Q609 BC807-16SMD, Q610 BC807-16SMD, Q611 BC807-16SMD, Q612 BC807-16SMD, U101 AD420, U102 AD420, U103 LT1014I, U104 LTC1865L, U201 AD620, U202 AD620, U203 AD620, U204 AD620, U205 AD620, U206 LTC1865L, U207 LTC1865L, U208 LTC1865L, U301 MAX743, U302 LT1014, U601 HCPL-063N, U602 HCPL-063N, U603 HCPL-063N, U604 HCPL-063N, U605 HCPL-063N, U606 HCPL-063N

Commit message: Updated schematic
Parts:
- removed IC1: MEGA8-AI, atmel:MEGA8-AI
- removed PAD401: G1, pads:PAD-5X2
- removed PAD402: G2, pads:PAD-5X2
- removed PAD403: VS+, pads:PAD-5X2
- removed PAD404: VS-, pads:PAD-5X2
- removed PAD405: S1, pads:PAD-10X4
- removed PAD406: S2, pads:PAD-10X4
- removed PAD407: UUT-, pads:PAD-10X4
- added IC501: MEGA8-AI, atmel:MEGA8-AI
- added PAD10: UUT-, pads:PAD-10X4
- added PAD11: 12V, pads:PAD-5X2
- added PAD12, PAD16: GND, pads:PAD-5X2
- added PAD13: T1, pads:PAD-5X2
- added PAD14: T2, pads:PAD-5X2
- added PAD15: 5V, pads:PAD-5X2
- C213, C308: value 0.1µ -> 1µ; device passives:C-EU-3216 -> passives:CPOL-3216-A
- C215: value 1µ -> 0.1µ; device passives:CPOL-3216-A -> passives:C-EU-3216
- C216: value 500p -> 0.1µ; device passives:C-EU-1608 -> passives:C-EU-3216
- C218: value 0.1µ -> 500p; device passives:C-EU-3216 -> passives:C-EU-1608
- C301: value 0.1µ -> 0.33µ
- C302: value 1µ -> 0.33µ; device passives:CPOL-3216-A -> passives:C-EU-3216
- C303: value 10n -> 220µ; device passives:C-EU-3216 -> rcl:CPOL-EUE3.5-10
- C304: value 10µ -> 0.1µ; device passives:CPOL-6032-C -> passives:C-EU-3216
- C305: value 10n -> 0.1µ
- C307: value 220µ -> 0.1µ; device rcl:CPOL-EUE3.5-10 -> passives:C-EU-3216
- C309: value 0.33µ -> 0.1µ
- C310: value 22µ -> 10n; device passives:CPOL-6032-C -> passives:C-EU-3216
- C311: value 220µ -> 10µ; device rcl:CPOL-EUE3.5-10 -> passives:CPOL-6032-C
- C312: value 220µ -> 10n; device rcl:CPOL-EUE3.5-10 -> passives:C-EU-3216
- C313: value 0.1µ -> 22µ; device passives:C-EU-3216 -> passives:CPOL-6032-C
- C314: value 0.33µ -> 220µ; device passives:C-EU-3216 -> rcl:CPOL-EUE3.5-10
- C315: value 0.1µ -> 220µ; device passives:C-EU-3216 -> rcl:CPOL-EUE3.5-10
- PAD1: value S1 -> G1; device pads:PAD-10X4 -> pads:PAD-5X2
- PAD2: value S2 -> G2; device pads:PAD-10X4 -> pads:PAD-5X2
- PAD3: value UUT- -> VS+; device pads:PAD-10X4 -> pads:PAD-5X2
- PAD4: value 12V -> VS-
- PAD5: value GND -> S1; device pads:PAD-5X2 -> pads:PAD-10X4
- PAD6: value T1 -> S2; device pads:PAD-5X2 -> pads:PAD-10X4
- PAD7: value T2 -> UUT-; device pads:PAD-5X2 -> pads:PAD-10X4
- PAD8: value 5V -> S1; device pads:PAD-5X2 -> pads:PAD-10X4
- PAD9: value GND -> S2; device pads:PAD-5X2 -> pads:PAD-10X4
- R208, R209: value 2M -> 100R; device passives:R-EU-3216 -> passives:R-EU-2012
- R210, R211: value 2k15 -> 100R
- R212, R213: value 100R -> 2M; device passives:R-EU-2012 -> passives:R-EU-3216
- R214, R215: value 100R -> 2k15
- renumbered MOV1 to MOV201, MOV2 to MOV202, MOV3 to MOV203, MOV4 to MOV204
Connections:
- net +12V: now also C301.1, C302.1, C303.+, PAD11.P; no longer C307.+, C309.1, C314.1, PAD4.P
- net +15V: now also C215.1, C314.+; no longer C213.1, C311.+
- net +3V3: now also C213.+, C216.1, C217.1; no longer C215.+, C218.1, C219.1
- net +5V: now also C304.1, C305.1, C307.2, C313.+, PAD15.P; no longer C301.2, C310.+, C313.1, C315.1, PAD8.P
- net -15V: now also C219.1, C309.1, C315.-; no longer C217.1, C308.1, C312.-
- net CSENSE1_H: now also U201.+, U202.-; no longer U203.+, U204.-
- net CSENSE1_L: now also PAD5.P, PAD8.P, U202.+; no longer PAD1.P, PAD405.P, U204.+
- net CSENSE2_H: now also U203.-, U204.+; no longer U201.-, U202.+
- net CSENSE2_L: now also PAD6.P, PAD9.P, U203.+; no longer PAD2.P, PAD406.P, U201.+
- net GATE1: now also PAD1.P; no longer PAD401.P
- net GATE2: now also PAD2.P; no longer PAD402.P
- net GND: now also C213.-, C215.2, C301.2, C302.2, C303.-, C304.2, C307.1, C308.-, C310.1, C312.2, C313.-, C314.-, C315.+, PAD12.P, PAD16.P, R214.1; no longer C213.2, C215.-, C301.1, C302.-, C303.1, C304.-, C307.-, C308.2, C310.-, C312.+, C313.2, C314.2, C315.2, PAD5.P, PAD9.P, R210.1
- net N$17: now also R210.1, U203.OUT; no longer R212.1, U201.OUT
- net N$18: now also C211.1, R210.2, U207.CH0; no longer C209.1, R212.2, U206.CH0
- net N$19: now also R211.1, U204.OUT; no longer R213.1, U202.OUT
- net N$20: now also C212.1, R211.2, U207.CH1; no longer C210.1, R213.2, U206.CH1
- net N$21: now also C209.1, R208.2, U206.CH0; no longer C211.1, R214.2, U207.CH0
- net N$22: now also C210.1, R209.2, U206.CH1; no longer C212.1, R215.2, U207.CH1
- net N$23: now also R209.1, U202.OUT; no longer R215.1, U204.OUT
- net N$24: now also R208.1, U201.OUT; no longer R214.1, U203.OUT
- net N$25: now also R212.1, R213.2; no longer R208.1, R209.2
- net N$26: now also R212.2; no longer R208.2
- net N$29: now also R213.1, R214.2; no longer R209.1, R210.2
- net N$30: now also C218.1; no longer C216.1
- net N$32: now also C312.1; no longer C305.1
- net N$33: now also C308.+; no longer C302.+
- net N$34: now also C310.2; no longer C303.2
- net RG1_H4: now also R203.2, U203.RG@1; no longer R201.2, U201.RG@1
- net RG1_H5: now also R204.2, U204.RG@1; no longer R202.2, U202.RG@1
- net RG1_H6: now also R215.2; no longer R211.2
- net RG1_L3: now also R201.2, U201.RG@1; no longer R203.2, U203.RG@1
- net RG1_L4: now also R202.2, U202.RG@1; no longer R204.2, U204.RG@1
- net RG2_H4: now also R203.1, U203.RG@2; no longer R201.1, U201.RG@2
- net RG2_H5: now also R204.1, U204.RG@2; no longer R202.1, U202.RG@2
- net RG2_H6: now also R215.1; no longer R211.1
- net RG2_L3: now also R201.1, U201.RG@2; no longer R203.1, U203.RG@2
- net RG2_L4: now also R202.1, U202.RG@2; no longer R204.1, U204.RG@2
- net SS_CH_I: now also U207.CONV; no longer U206.CONV
- net SS_CL_I: now also U206.CONV; no longer U207.CONV
- net T1_OUT: now also PAD13.P; no longer PAD6.P
- net T2_OUT: now also PAD14.P; no longer PAD7.P
- net UUT-: now also PAD10.P, PAD7.P, U201.-, U204.-; no longer PAD3.P, PAD407.P, U202.-, U203.-
- net VREF: now also C311.+; no longer C304.+
- net VSENSE+: now also PAD3.P; no longer PAD403.P
- net VSENSE-: now also PAD4.P; no longer PAD404.P
Other:
- note added: "+/-15V power supply"
- note added: "+12V input"
- note added: "+3V power supply"
- note added: "+5V supply"
- note added: "Load MOSFET 1 current sensing"
- note added: "Load MOSFET 2 current sensing"
- note added: "Test points"
- note removed: "50A range current sense"
- note removed: "50mA range current sense"

Commit message: Removed external parts from PCB, added Front Panel PCB
Parts:
- removed C122: 500p, passives:C-EU-1608
- removed IC101, IC102: LM50, linear:LM50
- removed IC501: MEGA8-AI, atmel:MEGA8-AI
- added PAD317: 12V, pads:PAD-5X2
- added PAD318: FAN_GND, pads:PAD-5X2
- added Q401: BC817-16SMD, transistor-npn:BC817-16SMD
- added Q402: SIRC10DP, transistors:SIRC10DP
- added R401: 1k, passives:R-EU-1608
- added U105: LM50, ic:LM50-NOPCB
- added U106: LTC1865L, ic:LTC1865L
- C116, C118: value 0.1µ -> 1µ; device passives:C-EU-3216 -> passives:CPOL-3216-A
- C117: value 1µ -> 0.1µ; device passives:CPOL-3216-A -> passives:C-EU-3216
- C120: value 1µ -> 500p; device passives:CPOL-3216-A -> passives:C-EU-1608
- Q107, Q111: value IXTK102N65X2R+ -> IXTK102N65X2; device transistors:IXTK102N65X2R+ -> transistors:IXTK102N65X2-NOPCB
- R103, R107: device passives:R-EU-3216 -> passives:R-EU-1608
- U104: value LTC1865L -> LM50; device ic:LTC1865L -> ic:LM50-NOPCB
- renumbered C601 to C501, C602 to C502, C603 to C503, C604 to C504, C605 to C505, C606 to C506, C607 to C507, C608 to C508, C609 to C509, C610 to C510, C611 to C511, C612 to C512, C613 to C513, C614 to C514, C615 to C515, C616 to C516, C617 to C517, C618 to C518, C619 to C519, C620 to C520, C621 to C521, C622 to C522, C623 to C523, C624 to C524, PAD1 to PAD301, PAD10 to PAD316, PAD11 to PAD305, PAD12 to PAD306, PAD13 to PAD307, PAD14 to PAD308, PAD15 to PAD309, PAD16 to PAD310, PAD2 to PAD302, PAD3 to PAD303, PAD4 to PAD304, PAD5 to PAD311, PAD6 to PAD313, PAD7 to PAD315, PAD8 to PAD312, PAD9 to PAD314, Q601 to Q501, Q602 to Q502, Q603 to Q503, Q604 to Q504, Q605 to Q505, Q606 to Q506, Q607 to Q507, Q608 to Q508, Q609 to Q509, Q610 to Q510, Q611 to Q511, Q612 to Q512, R601 to R501, R602 to R502, R603 to R503, R604 to R504, R605 to R505, R606 to R506, R607 to R507, R608 to R508, R609 to R509, R610 to R510, R611 to R511, R612 to R512, R613 to R513, R614 to R514, R615 to R515, R616 to R516, R617 to R517, R618 to R518, R619 to R519, R620 to R520, R621 to R521, R622 to R522, R623 to R523, R624 to R524, U601 to U501, U602 to U502, U603 to U503, U604 to U504, U605 to U505, U606 to U506
Connections:
- new net FAN_GND: PAD318.P, Q402.D
- new net N$42: Q401.C, Q402.G
- new net N$44: Q401.B, R401.2
- new net VREF2: C311.+, U301.VREF
- net +12V: now also PAD317.P
- net +3V3: now also C116.+, C117.1, U106.VCC; no longer C117.+, C118.1, U104.VCC
- net +5V: now also U104.+V, U105.+V; no longer C115.1, IC101.+VS, IC102.+VS
- net -15V: now also C115.1; no longer C116.1
- net GND: now also C116.-, C117.2, C118.-, C120.2, Q401.E, Q402.S, U105.GND, U106.GND; no longer C116.2, C117.-, C118.2, C120.-, C122.2, IC101.GND, IC102.GND
- net MISO_I: now also U106.SDO; no longer U104.SDO
- net MOSI_I: now also U106.SDI; no longer U104.SDI
- net SCK_I: now also U106.SCK; no longer U104.SCK
- net SS_TEMP_I: now also U106.CONV; no longer U104.CONV
- net T1_OUT: now also C118.+, U104.VO; no longer C119.+, IC101.VO
- net T2_OUT: now also C119.+, U105.VO; no longer C120.+, IC102.VO
- net TEMP1: now also C120.1, U106.CH0; no longer C121.1, U104.CH0
- net TEMP2: now also C121.1, U106.CH1; no longer C122.1, U104.CH1
- net VREF: no longer C311.+, U301.VREF
