File: PCB/V1A/Electronic_Load_V1A.brd (EAGLE design)
At the start: 180 x 225 mm, 198 parts, among them IC201 OPA77P, IC202 OPA77P, IC203 OPA77P, IC204 OPA77P, IC205 OPA77P, IC301 MAX743CPE, IC302 7805T, IC303 7805T, IC304 7905, IC305 LM50, IC306 LM50, IC401 OPA77P, IC501 AD620R, IC502 AD620R, IC503 AD620R, IC504 AD620R, J101 +, J102 -, J103 +, J104 -, Q101 SIRC10DP, Q102 SIRC10DP, Q103 SIRC10DP, Q104 IXTK102N65X2PADUP, Q105 SIRC10DP, Q106 SIRC10DP, Q107 SIRC10DP, Q108 IXTK102N65X2PADUP, Q401 BC817-25SMD, Q402 BC807-25SMD, Q403 BC817-25SMD, U201 LTC1865-MSOP, U202 LTC1865-MSOP, U203 LTC1865-MSOP, U401 AD420, U402 AD420, U403 LT1014, U404 LTC1865-MSOP, U501 LTC1865L, U502 LTC1865L

Commit message: Added optocouplers
Parts:
- removed C315: 1µ, rcl:SMC_A
- removed C316: 0.1µ, rcl:C1206
- removed IC302, IC303: 7805T, linear:TO220H
- removed IC304: 7905, linear:TO220H
- removed IC305: LM50, linear:SOT23
- removed IC501: AD620R, analog-devices:SO8
- removed PAD401, PAD402: PAD-5X2, pads:PAD-5X2
- removed R201, R202, R203, R208, R209, R210, R211, R212, R213, R214, R215, R216, R218, R219, R231, R232, R233, R234: 200k, rcl:R1206
- removed R204, R205, R206, R207, R227, R228, R229, R230, R413, R414: 5k, rcl:R0603
- removed R217: 20k, rcl:R0603
- removed R220, R221, R224, R225, R417, R418: 10k, rcl:R0603
- removed R222, R223, R226, R235, R236: 20k, rcl:RTRIM4G/J
- removed U201, U202, U203: LTC1865-MSOP, adc_dac:MSOP-10
- added C1, C421, C422, C5, C9: 0.1µ, rcl:C1206
- added C10, C2, C6: 0.01µ, rcl:C1206
- added C11, C12, C3, C4, C7, C8: 15p, rcl:C1206
- added C13, C14, C15, C16, C17, C18, C19: 500p, rcl:C1206
- added C417, C418, C419, C420: 1µ, rcl:SMC_A
- added IC405, IC406: LM50, linear:SOT23
- added IC407: AD620R, analog-devices:SO8
- added Q1, Q2, Q3, Q4, Q5, Q501, Q502, Q503, Q504, Q505, Q506, Q6: BC807-16SMD, transistor-pnp:SOT23-BEC
- added R1, R10, R11, R12, R2, R3, R4, R5, R505, R506, R507, R508, R509, R510, R511, R512, R6, R7, R8, R9: 350R, rcl:R1206
- added R13, R14, R15, R16, R17, R18, R19, R309, R310: 100R, rcl:R1206
- added R301, R303: 1k, rcl:R0603
- added R302, R304: 10k, rcl:R0603
- added R305, R306: 20k, rcl:RTRIM4G/J
- added R307, R308: 200k, rcl:R1206
- added R311: 5k, rcl:R0603
- added U1, U2, U3, U503: HCPL-063N, isolation:SO8
- added U301, U302: AD420, adc_dac:SO24W
- added U303: LT1014, SparkFun-Retired:SO16L
- C201, C210, C211: value 0.1µ -> 220µ; device rcl:C1206 -> rcl:E3,5-10
- C203, C409: value 0.1µ -> 1µ; device rcl:C1206 -> rcl:SMC_A
- C204, C206: value 0.1µ -> 10n; device rcl:C1206 -> rcl:C0805
- C205: value 0.1µ -> 10µ; device rcl:C1206 -> rcl:SMC_C
- C207: value 1µ -> 0.33µ; device rcl:SMC_A -> rcl:C1206
- C209: value 1µ -> 22µ; device rcl:SMC_A -> rcl:SMC_D
- C212: value 0.1µ -> 0.33µ
- C213: value 0.1µ -> 2µ2; device rcl:C1206 -> rcl:SMC_A
- C301, C311: value 220µ -> 0.1µ; device rcl:E3,5-10 -> rcl:C1206
- C303, C414: value 1µ -> 0.1µ; device rcl:SMC_A -> rcl:C1206
- C305: value 10µ -> 10n; device rcl:SMC_C -> rcl:C0805
- C307: value 0.33µ -> 10n; device rcl:C1206 -> rcl:C0805
- C308: value 0.1µ -> 500p
- C309: value 22µ -> 0.1µ; device rcl:SMC_D -> rcl:C1206
- C310: value 220µ -> 0.1µ; device rcl:E3,5-10 -> rcl:C0805
- C312: value 0.33µ -> 0.1µ
- C313: value 2µ2 -> 0.1µ; device rcl:SMC_A -> rcl:C1206
- C404, C405, C406, C407: value 10n -> 0.1µ; device rcl:C0805 -> rcl:C1206
- C408: value 500p -> 0.1µ
- C410: value 0.1µ -> 1µ; device rcl:C0805 -> rcl:SMC_A
- C504, C505, C506: value 0.1µ -> 0.01µ
- C507, C508, C511, C512: value 0.1µ -> 15p
- C509, C510: value 1µ -> 15p; device rcl:SMC_A -> rcl:C1206
- IC201: value OPA77P -> MAX743CPE; device burr-brown:DIL08 -> maxim:DIL16
- IC202, IC203: value OPA77P -> 7805T; device burr-brown:DIL08 -> linear:TO220H
- IC204: value OPA77P -> 7905; device burr-brown:DIL08 -> linear:TO220H
- IC205: value OPA77P -> LM50; device burr-brown:DIL08 -> linear:SOT23
- IC301: value MAX743CPE -> OPA77P; device maxim:DIL16 -> burr-brown:DIL08
- IC401: value OPA77P -> AD620R; device burr-brown:DIL08 -> analog-devices:SO8
- R401, R403: value 1k -> 2k15; device rcl:R0603 -> rcl:R1206
- R402, R404: value 10k -> 2k15; device rcl:R0603 -> rcl:R1206
- R405, R406: value 20k -> 2M; device rcl:RTRIM4G/J -> rcl:R1206
- R407, R408: value 200k -> 2M
- R409: value 100R -> 2M
- R410: value 100R -> 2k15
- R411: value 5k -> 2k15; device rcl:R0603 -> rcl:R1206
- R501, R502, R503, R504: value 2k61 -> 350R
- U401, U402: value AD420 -> LTC1865L; device adc_dac:SO24W -> adc_dac:SO08
- U403: value LT1014 -> LTC1865L; device SparkFun-Retired:SO16L -> adc_dac:SO08
- U404: value LTC1865-MSOP -> LTC1865L; device adc_dac:MSOP-10 -> adc_dac:SO08
- U501, U502: value LTC1865L -> HCPL-063N; device adc_dac:SO08 -> isolation:SO8
- moved C314 644.8 mm to (-427.0, -340.0)
- moved C313 639.2 mm to (-427.0, -333.0)
- moved IC301 597.1 mm to (-417.0, -318.0)
- moved R405 536.5 mm to (-512.0, -486.0)
- moved R407 522.3 mm to (-512.0, -479.0)
- moved R409 491.4 mm to (-512.0, -451.0)
- moved R408 491.2 mm to (-512.0, -465.0)
- moved R406 484.5 mm to (-512.0, -472.0)
- moved R410 481.6 mm to (-512.0, -458.0)
- moved R411 478.0 mm to (-512.0, -437.0)
- moved C308 441.5 mm to (-170.0, -190.0)
- moved C303 433.2 mm to (-168.0, -198.0)
- moved C307 425.8 mm to (-433.0, 21.0), turned to 180 degrees
- moved C305 423.7 mm to (-433.0, 24.0), turned to 180 degrees
- moved C207 423.2 mm to (-74.9, 251.5), turned to 0 degrees
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- renumbered D301 to D201, D302 to D202, D303 to D203, D304 to D204, IC306 to IC206, IC502 to IC402, IC503 to IC403, IC504 to IC404, J301 to J201, L301 to L201, L302 to L202, Q401 to Q301, Q402 to Q302, Q403 to Q303, R412 to R312, R415 to R313, R416 to R314, R419 to R315, R420 to R316, R421 to R317, R422 to R318, R423 to R319
Connections:
- removed net CLR_DAC1: U401.6
- removed net CLR_DAC2: U402.6
- removed net CSENSE_H1_AMP: IC201.6, IC501.6, R218.2, U201.2, U501.2
- removed net CSENSE_H1_AMP1: IC403.6, U502.2
- removed net CSENSE_H2_AMP: IC202.6, IC402.6, R219.2, U201.3, U501.3
- removed net CSENSE_H2_AMP1: IC404.6, U502.3
- removed net CSENSE_L1_AMP: IC204.6, R233.2, U203.2
- removed net CSENSE_L2_AMP: IC205.6, R234.2, U203.3
- removed net N$85: R209.1, R210.2
- removed net N$86: R208.1, R209.2
- removed net N$87: R201.2, R208.2
- removed net N$88: R201.1, R202.2
- removed net N$89: R202.1, R203.2
- removed net N$90: U404.10
- removed net N$91: IC203.3, R220.2, R221.2
- removed net N$92: IC203.2, R224.2, R225.1
- removed net SS_ADC_H: U201.1
- removed net SS_ADC_L: U203.1
- removed net SS_ADC_T: U404.1
- removed net SS_ADC_V: U202.1
- removed net TEMP1_AMP: R417.2, U403.10, U404.2
- removed net TEMP1_IN: PAD401.1, U403.12
- removed net TEMP2_AMP: R418.2, U403.16, U404.3
- removed net TEMP2_IN: PAD402.1, U403.14
- removed net VSENSE: IC203.6, R225.2, U202.2
- new net +IN: U303.12, U303.14
- new net -IN: U303.11, U303.15
- new net BYP_G_ISO: C8.1, Q301.E, Q302.E, R6.1, U2.6
- new net DAC_CLR: Q5.B
- new net DAC_CLR_ISO: C11.1, R9.1, U3.7
- new net DAC_FAULT_ISO: Q2.B, R304.1, U301.3, U302.3
- new net N$100: R408.1, R409.2
- new net N$101: IC407.3, R409.1, R410.2
- new net N$33: R305.2, R307.1
- new net N$98: R406.1, R407.2
- new net N$99: R406.2, R408.2
- new net OUT: U303.10, U303.16
- new net RG1_H3: IC407.1, R411.2
- new net RG2_H3: IC407.8, R411.1
- new net SS_CH: Q502.B
- new net SS_CL: Q505.B
- new net SS_DAC_ISO: C7.1, R5.1, U2.7
- new net SS_TEMP: Q506.B
- new net SS_TEMP_ISO: C512.1, R512.1, U403.1, U503.6
- new net SS_V: Q503.B
- new net SS_V_ISO: C509.1, R509.1, U404.1, U503.7
- new net VSENSE_AMP: IC407.6
- net +12V: now also C201.+, C207.1, C304.2, C305.2, C306.2, C307.2, C309.1, C310.1, IC202.1, U301.23, U302.23; no longer C301.+, C307.1, C404.2, C405.2, C406.2, C407.2, C409.1, C410.1, IC302.1, U401.23, U402.23
- net +15V: now also C210.+, C311.1, C313.1, C401.1, C402.1, C403.1, C404.1, IC201.16, IC203.1, IC301.7, IC407.7, U303.4; no longer C201.1, C202.1, C205.1, C211.1, C310.+, C312.1, C411.1, C501.1, C502.1, C503.1, C504.1, IC201.7, IC202.7, IC203.7, IC204.7, IC205.7, IC301.16, IC303.1, IC501.7, R222.2, R223.2, R226.2, R235.2, R236.2, U403.4
- net +3V3: now also C409.+, C410.+, C411.1, C412.1, C419.+, C420.+, C421.1, C422.1, U401.8, U402.8, U403.8, U404.8; no longer C509.+, C510.+, C511.1, C512.1, U501.8, U502.8
- net +5V: now also C1.1, C10.1, C2.1, C202.2, C301.1, C302.1, C414.1, C5.1, C501.1, C502.1, C503.1, C504.1, C505.1, C506.1, C6.1, C9.1, IC201.12, IC201.13, IC201.3, IC201.4, IC201.5, IC202.3, IC205.1, IC405.1, IC406.1, R1.2, R10.2, R11.2, R12.2, R2.2, R3.2, R304.2, R4.2, R5.2, R501.2, R502.2, R503.2, R504.2, R505.2, R506.2, R507.2, R508.2, R509.2, R510.2, R511.2, R512.2, R6.2, R7.2, R8.2, R9.2, U1.8, U2.8, U3.8, U301.2, U302.2, U501.8, U502.8, U503.8; no longer C207.+, C210.1, C215.+, C216.1, C302.2, C308.1, C309.+, C401.1, C402.1, C414.+, IC301.12, IC301.13, IC301.3, IC301.4, IC301.5, IC302.3, IC305.1, R404.2, U201.9, U202.9, U203.9, U401.2, U402.2, U404.9
- net +5V/1: now also C214.1, IC203.3, R305.3, R306.3; no longer C314.1, IC303.3, R405.3, R406.3
- net -15V: now also C211.-, C213.-, C312.1, C314.1, C405.1, C406.1, C407.1, C408.1, IC201.9, IC204.2, IC301.4, IC407.4, U303.13; no longer C203.1, C204.1, C206.1, C213.1, C214.1, C311.-, C313.-, C412.1, C505.1, C506.1, C507.1, C508.1, IC201.4, IC202.4, IC203.4, IC204.4, IC205.4, IC301.9, IC304.2, IC501.4, U403.13
- net -5V: now also C215.-, C216.2, IC204.3, R305.1, R306.1; no longer C315.-, C316.2, IC304.3, R405.1, R406.1
- net BOOST: now also U301.19, U302.19; no longer U401.19, U402.19
- net BYP_CTRL: now also C308.2, R101.1, R303.1; no longer C408.2, R403.1
- net BYP_G: now also Q4.B; no longer Q301.E, Q302.E, R101.1
- net CSENSE_H1: now also IC401.3; no longer IC501.3, R204.1, R228.1
- net CSENSE_H2: no longer R206.1, R230.1
- net CSENSE_L1: no longer R227.1
- net CSENSE_L2: no longer R229.1
- net DAC1_OUT: now also U301.10, U302.9; no longer U401.10, U402.9
- net DAC2_OUT: now also U302.10; no longer U402.10
- net DAC_FAULT: now also C4.1, R2.1, U1.6; no longer R404.1, U401.3, U402.3
- net GND: now also C1.2, C10.2, C11.2, C12.2, C13.2, C14.2, C15.2, C16.2, C17.2, C18.2, C19.2, C2.2, C201.-, C202.1, C203.-, C204.1, C205.-, C210.-, C211.+, C213.+, C215.+, C216.1, C3.2, C301.2, C302.2, C309.2, C310.2, C311.2, C313.2, C4.2, C403.2, C404.2, C405.2, C406.2, C407.2, C408.2, C409.-, C410.-, C414.2, C417.-, C418.-, C419.-, C420.-, C421.2, C422.2, C5.2, C509.2, C510.2, C6.2, C7.2, C8.2, C9.2, IC201.11, IC201.14, IC201.2, IC203.2, IC204.1, IC205.3, IC401.2, IC401.5, IC405.3, IC406.3, IC407.5, Q1.C, Q2.C, Q3.C, Q4.C, Q5.C, Q501.C, Q502.C, Q503.C, Q504.C, Q505.C, Q506.C, Q6.C, R309.1, R310.1, U1.2, U1.3, U1.5, U2.2, U2.3, U2.5, U3.2, U3.3, U3.5, U301.11, U301.4, U301.5, U302.11, U302.4, U302.5, U403.4, U501.2, U501.3, U501.5, U502.2, U502.3, U502.5, U503.2, U503.3, U503.5; no longer C201.2, C202.2, C203.2, C204.2, C205.2, C207.-, C208.2, C210.2, C211.2, C213.2, C215.-, C216.2, C301.-, C302.1, C303.-, C304.1, C305.-, C306.2, C309.-, C310.-, C311.+, C313.+, C315.+, C316.1, C409.2, C410.2, C414.-, C509.-, C510.-, IC301.11, IC301.14, IC301.2, IC303.2, IC304.1, IC305.3, IC501.2, IC501.5, R205.1, R207.1, R214.1, R215.1, R217.1, R221.1, R231.1, R232.1, R409.1, R413.1, R414.1, U201.4, U201.5, U202.4, U202.5, U203.4, U203.5, U401.11, U401.5, U402.11, U402.5, U404.5, U501.4, U502.4
- net LOAD_G1: now also U303.1; no longer U403.1
- net LOAD_G2: now also U303.7; no longer U403.7
- net MISO: now also C3.1, R1.1, U1.7; no longer U201.7, U202.7, U203.7, U404.7
- net MISO_ISO: now also Q1.B, U401.6, U402.6, U403.6, U404.6; no longer U501.6, U502.6
- net MOSI: now also Q504.B, U301.9; no longer U201.6, U202.6, U203.6, U401.9, U404.6
- net MOSI_ISO: now also C510.1, R510.1, U401.5, U402.5, U403.5, U404.5, U501.6; no longer U501.5, U502.5
- net N$24: now also C307.1, U302.21; no longer C407.1, U402.21
- net N$25: now also C304.1, U301.20; no longer C404.1, U401.20
- net N$26: now also C305.1, U302.20; no longer C405.1, U402.20
- net N$27: now also C306.1, U301.21; no longer C406.1, U401.21
- net N$28: now also R311.2, U303.2; no longer R411.2, U403.2
- net N$29: now also U303.6; no longer U403.6
- net N$32: now also R307.2, R309.2, R311.1; no longer R407.2, R409.2, R411.1
- net N$34: now also R306.2, R308.1; no longer R406.2, R408.1
- net N$35: now also R308.2, R310.2; no longer R408.2, R410.2
- net N$36: now also IC201.15; no longer IC301.15
- net N$37: now also C206.1, IC201.8; no longer C306.1, IC301.8
- net N$38: now also C203.+, IC201.7; no longer C303.+, IC301.7
- net N$39: now also IC201.10; no longer IC301.10
- net N$40: now also C204.2, IC201.1; no longer C304.2, IC301.1
- net N$44: now also C207.2, C208.2, IC202.2; no longer C307.2, C308.2, IC302.2
- net N$47: now also Q501.E, R501.1, U501.1; no longer R414.2, R418.1, U403.15
- net N$48: now also IC301.3; no longer IC401.3
- net N$49: now also Q502.E, R502.1, U502.1; no longer R413.2, R417.1, U403.11
- net N$51: now also IC301.8; no longer IC401.8
- net N$53: now also IC301.1; no longer IC401.1
- net N$62: now also Q504.E, R504.1, U501.4; no longer R216.1, R217.2, R220.1
- net N$63: now also Q505.E, R505.1, U502.4; no longer IC203.1, R226.1
- net N$64: now also Q503.E, R503.1, U503.1; no longer IC204.2, R228.2, R233.1
- net N$65: now also Q506.E, R506.1, U503.4; no longer IC204.3, R227.2, R231.2
- net N$66: now also Q1.E, R3.1, U1.1; no longer IC201.2, R205.2, R218.1
- net N$67: now also Q2.E, R4.1, U1.4; no longer IC201.3, R204.2, R214.2
- net N$68: now also Q5.E, R11.1, U3.1; no longer IC204.1, R235.1
- net N$69: now also Q6.E, R12.1, U3.4; no longer IC201.1, R222.1
- net N$70: now also IC401.6, R13.1; no longer IC201.8, R222.3
- net N$71: now also Q6.B; no longer IC204.8, R235.3
- net N$72: now also C13.1, R13.2, U401.2; no longer IC203.8, R226.3
- net N$73: now also C12.1, R10.1, U3.6; no longer R211.2, R216.2
- net N$74: now also IC402.6, R14.1; no longer IC202.2, R207.2, R219.1
- net N$75: now also C14.1, R14.2, U401.3; no longer IC202.3, R206.2, R215.2
- net N$76: now also Q3.E, R7.1, U2.1; no longer IC202.1, R223.1
- net N$77: now also Q4.E, R8.1, U2.4; no longer IC202.8, R223.3
- net N$78: now also C15.1, R15.2, U402.2; no longer R211.1, R212.2
- net N$79: now also C16.1, R16.2, U402.3; no longer R212.1, R213.2
- net N$80: now also IC404.6, R16.1; no longer IC205.2, R230.2, R234.1
- net N$81: now also IC403.6, R15.1; no longer IC205.3, R229.2, R232.2
- net N$82: now also C17.1, R17.2, U403.2; no longer IC205.1, R236.1
- net N$83: now also C18.1, R18.2, U404.2; no longer IC205.8, R236.3
- net N$84: now also C19.1, R19.2, U403.3; no longer R210.1, R213.1
- net N$93: now also R301.1; no longer R401.1
- net N$94: now also C303.1, R301.2, R302.2; no longer C403.1, R401.2, R402.2
- net N$95: now also C303.2; no longer C403.2
- net N$96: now also C308.1, R302.1, R303.2; no longer C408.1, R402.1, R403.2
- net RG1_H1: now also IC401.1, R401.2; no longer IC501.1, R501.2
- net RG1_H2: now also R402.2; no longer R502.2
- net RG1_L1: now also R403.2; no longer R503.2
- net RG1_L2: now also R404.2; no longer R504.2
- net RG2_H1: now also IC401.8, R401.1; no longer IC501.8, R501.1
- net RG2_H2: now also R402.1; no longer R502.1
- net RG2_L1: now also R403.1; no longer R503.1
- net RG2_L2: now also R404.1; no longer R504.1
- net SCK: now also Q501.B, U301.8, U302.8; no longer U201.8, U202.8, U203.8, U401.8, U402.8, U404.8
- net SCK_ISO: now also C507.1, R507.1, U401.7, U402.7, U403.7, U404.7; no longer U502.7
- net SS_CH_ISO: now also C508.1, R508.1, U401.1, U502.7; no longer U501.1
- net SS_CL_ISO: now also C511.1, R511.1, U402.1, U502.6; no longer U502.1
- net SS_DAC: now also Q3.B; no longer U401.7, U402.7
- net TEMP1: now also C417.+, IC205.2, IC405.2; no longer IC305.2
- net TEMP2: now also C418.+, IC406.2, R19.1
- net VGATE_1: now also U301.17, U303.3; no longer U401.17, U403.3
- net VGATE_2: now also U302.17, U303.5; no longer U402.17, U403.5
- net VREF: now also C205.+, IC201.6, U301.14, U301.15, U302.15; no longer C305.+, IC301.6, U201.10, U202.10, U203.10, U401.14, U401.15, U402.15
- net VREF3.0: now also IC301.2, IC301.6; no longer IC401.2, IC401.6
- net VSENSE+: now also R405.1; no longer R203.1
- net VSENSE-: now also IC407.2; no longer R224.1
Routing:
- net VSENSE: track 13.6 -> 0.00 mm
- net CSENSE_H1_AMP1: track 13.3 -> 0.00 mm
- net CSENSE_H2_AMP1: track 12.4 -> 0.00 mm
- net CSENSE_H2_AMP: track 12.4 -> 0.00 mm
- net CSENSE_H1_AMP: track 12.3 -> 0.00 mm
- net N$92: track 11.7 -> 0.00 mm
- net +5V: track 16.9 -> 7.05 mm, vias 1 -> 0
- net GND: track 76.9 -> 67.7 mm, vias 13 -> 12
- net N$62: track 7.63 -> 0.00 mm
- net N$91: track 7.24 -> 0.00 mm
- net N$85: track 3.11 -> 0.00 mm
- net N$84: track 3.11 -> 0.00 mm
- net N$89: track 2.66 -> 0.00 mm
- net N$88: track 2.66 -> 0.00 mm
- net N$87: track 2.66 -> 0.00 mm
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