File: PCB/V1A/Electronic_Load_V1A.brd (EAGLE design)
At the start: 160 x 100 mm, 209 parts, among them IC101 LM50, IC102 LM50, IC301 7805T, IC302 OPA77P, Q101 SIRC10DP, Q102 SIRC10DP, Q103 BC817-16SMD, Q104 BC817-16SMD, Q105 BC807-16SMD, Q106 SIRC10DP, Q107 IXTK102N65X2R+, Q108 SIRC10DP, Q109 SIRC10DP, Q110 SIRC10DP, Q111 IXTK102N65X2R+, Q601 BC807-16SMD, Q602 BC807-16SMD, Q603 BC807-16SMD, Q604 BC807-16SMD, Q605 BC807-16SMD, Q606 BC807-16SMD, Q607 BC807-16SMD, Q608 BC807-16SMD, Q609 BC807-16SMD, Q610 BC807-16SMD, Q611 BC807-16SMD, Q612 BC807-16SMD, U101 AD420, U102 AD420, U103 LTC1865L, U104 LT1014I, U201 AD620, U202 AD620, U203 AD620, U204 AD620, U205 AD620, U206 LTC1865L, U207 LTC1865L, U208 LTC1865L, U301 MAX743, U601 HCPL-063N, U602 HCPL-063N, U603 HCPL-063N, U604 HCPL-063N, U605 HCPL-063N, U606 HCPL-063N

Commit message: Added heatsink models, ADC/DAC layout
Parts:
- U103: value LTC1865L -> LT1014I; device ic:SO8 -> ic:SO16W
- U104: value LT1014I -> LTC1865L; device ic:SO16W -> ic:SO8
- moved IC301 247.6 mm to (100.0, 180.0)
- moved U101 247.0 mm to (125.0, 67.5), turned to 90 degrees
- moved Q111 238.2 mm to (125.0, 175.0)
- moved Q107 237.9 mm to (145.0, 175.0)
- moved R123 232.0 mm to (105.5, 129.5)
- moved C122 222.4 mm to (105.5, 123.5), turned to 180 degrees
- moved C118 219.8 mm to (113.0, 125.0), flipped to the bottom, turned to 270 degrees
- moved R121 218.3 mm to (103.0, 78.0), flipped to the bottom
- moved C121 217.4 mm to (105.5, 126.5), turned to 180 degrees
- moved R120 214.2 mm to (103.0, 70.0), flipped to the bottom
- moved R118 214.2 mm to (114.0, 77.0), turned to 90 degrees
- moved U103 212.7 mm to (103.0, 74.0), turned to 90 degrees
- moved C103 211.6 mm to (125.0, 82.5), flipped to the bottom, turned to 90 degrees
- moved C120 208.5 mm to (101.0, 122.0), turned to 90 degrees
- moved C116 207.8 mm to (101.5, 74.0), flipped to the bottom, turned to 90 degrees
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Connections:
- removed net BYP_G_ISO: C610.1, R610.1, U601.6
- removed net CSENSE_H1: U201.3, U203.2
- removed net CSENSE_H2: U202.3, U204.2
- removed net CSENSE_L1: U203.3
- removed net CSENSE_L2: U204.3
- removed net DAC_CLR: Q603.B
- removed net DAC_FAULT_ISO: Q605.B
- removed net SS_DAC_ISO: C607.1, R607.1, U601.7
- net +15V: now also U103.4; no longer U104.4
- net +3V3: now also U104.8; no longer U103.8
- net -15V: now also U103.13; no longer U104.13
- net BYP_I: now also C610.1, R610.1, U601.6
- net CLR_DAC_I: now also Q603.B
- net CSENSE1_H: now also U201.3, U203.2
- net CSENSE1_L: now also U203.3
- net CSENSE2_H: now also U202.3, U204.2
- net CSENSE2_L: now also U204.3
- net FLT_DAC_I: now also Q605.B
- net GND: now also U104.4; no longer U103.4
- net LQ1_G: now also U103.16; no longer U104.1
- net LQ2_G: now also U103.10; no longer U104.7
- net MISO_I: now also U104.6; no longer U103.6
- net MOSI_I: now also U104.5; no longer U103.5
- net N$10: now also U103.14; no longer U104.3
- net N$11: now also U103.12; no longer U104.5
- net N$12: now also U103.15; no longer U104.2
- net N$13: now also U103.1; no longer U104.10
- net N$14: now also U103.2; no longer U104.11
- net N$15: now also U103.6; no longer U104.15
- net N$16: now also U103.7; no longer U104.16
- net N$9: now also U103.11; no longer U104.6
- net SCK_I: now also U104.7; no longer U103.7
- net SS_CH: now also Q610.B; no longer Q607.B
- net SS_CH_I: now also C623.1, R623.1, U605.6; no longer C620.1, R620.1, U605.7
- net SS_CL: now also Q607.B; no longer Q610.B
- net SS_CL_I: now also C620.1, R620.1, U605.7; no longer C623.1, R623.1, U605.6
- net SS_DAC_I: now also C607.1, R607.1, U601.7
- net SS_TEMP: now also Q608.B; no longer Q611.B
- net SS_TEMP_I: now also C621.1, R621.1, U104.1, U606.7; no longer C624.1, R624.1, U103.1, U606.6
- net SS_V: now also Q611.B; no longer Q608.B
- net SS_V_I: now also C624.1, R624.1, U606.6; no longer C621.1, R621.1, U606.7
- net TEMP1: now also U104.2; no longer U103.2
- net TEMP2: now also U104.3; no longer U103.3
- net VSENSE-: now also U103.3, U103.5; no longer U104.12, U104.14
Routing:
- net GND: track 0.00 -> 130.7 mm, vias 0 -> 11
- net +15V: track 0.00 -> 33.3 mm, vias 0 -> 6
- net -15V: track 0.00 -> 32.9 mm, vias 0 -> 6
- net +5V: track 0.00 -> 31.9 mm, vias 0 -> 5
- net +12V: track 0.00 -> 31.4 mm, vias 0 -> 2
- net SS_CL_I: track 0.00 -> 26.9 mm
- net VREF: track 0.00 -> 23.6 mm
- net T1_OUT: track 0.00 -> 21.9 mm
- net SS_CH_I: track 0.00 -> 18.8 mm
- net SS_TEMP_I: track 7.09 -> 23.4 mm
- net T2_OUT: track 0.00 -> 15.2 mm
- net SS_V_I: track 7.09 -> 22.1 mm
- net +3V3: track 0.00 -> 14.0 mm, vias 0 -> 3
- net N$16: track 0.00 -> 13.1 mm, vias 0 -> 1
- net N$13: track 0.00 -> 11.5 mm, vias 0 -> 1
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Other:
- board size 160 x 100 mm -> 200 x 200 mm

Commit message: ADC/DAC board layout
Parts:
- removed IC302: OPA77P, burr-brown:DIL08
- added R306, R307, R308: 100R, passives:R3225W
- added U302: (no value), ic:SO16W
- C306: value 220µ -> 0.1µ; device rcl:E3,5-10 -> passives:C3216
- C307: value 0.33µ -> 220µ; device passives:C3216 -> rcl:E3,5-10
- C308: value 22µ -> 0.1µ; device passives:CT6032 -> passives:C3216
- C309: value 220µ -> 0.33µ; device rcl:E3,5-10 -> passives:C3216
- C310: value 220µ -> 22µ; device rcl:E3,5-10 -> passives:CT6032
- C311, C312: value 0.1µ -> 220µ; device passives:C3216 -> rcl:E3,5-10
- R301, R302, R303, R304: value 20k -> 10k
- R305: value 20k -> 100R; device rcl:RTRIM4G/J -> passives:R3225W
- moved Q601 298.6 mm to (89.5, 15.5), turned to 180 degrees
- moved Q603 298.3 mm to (89.5, 3.50), turned to 180 degrees
- moved Q604 292.7 mm to (89.5, 22.0), turned to 180 degrees
- moved Q606 292.4 mm to (89.5, 10.0), turned to 180 degrees
- moved C612 279.9 mm to (77.0, 11.5)
- moved C601 278.1 mm to (85.5, 19.0), flipped to the bottom, turned to 90 degrees
- moved R612 274.6 mm to (77.0, 8.50)
- moved C610 267.5 mm to (77.0, 23.5)
- moved R610 267.3 mm to (77.0, 20.5)
- moved C609 267.2 mm to (77.0, 2.50)
- moved R609 265.4 mm to (77.0, 5.50)
- moved R606 261.0 mm to (84.0, 11.5), turned to 180 degrees
- moved R607 257.9 mm to (77.0, 17.5)
- moved C606 256.6 mm to (82.5, 7.00), flipped to the bottom, turned to 90 degrees
- moved C607 254.4 mm to (77.0, 14.5)
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Connections:
- removed net BYP_G_LOL: Q604.B
- removed net DAC_CLR_ISO: C609.1, R609.1, U603.7
- removed net N$78: IC302.3, R302.1, R303.2
- removed net N$80: IC302.8, R305.3
- removed net N$81: IC302.1, R305.1
- removed net VREF3.0: IC302.2, IC302.6
- new net BYP: Q603.B
- new net CLR_DAC: Q601.B
- new net N$37: R302.1, R303.2, U302.12, U302.14, U302.3, U302.5
- new net N$38: R306.1, U302.6, U302.7
- new net N$39: R305.1, U302.1, U302.2
- new net N$40: R307.1, U302.10, U302.11
- new net N$43: R308.1, U302.15, U302.16
- net +12V: now also C307.+, C309.1; no longer C306.+, C307.1
- net +15V: now also C306.1, C311.+, U302.4; no longer C309.+, C312.1, IC302.7, R305.2
- net +3V3: now also R305.2, R306.2, R307.2, R308.2
- net +5V: now also C310.+, C313.1; no longer C308.+, C311.1
- net -15V: now also C308.1, C312.-, U302.13; no longer C310.-, C313.1, IC302.4
- net BYP_I: now also C609.1, R609.1, U603.7; no longer C610.1, R610.1, U601.6
- net CLR_DAC_I: now also C607.1, R607.1, U601.7; no longer Q603.B
- net GND: now also C306.2, C307.-, C308.2, C310.-, C311.-, C312.+; no longer C306.-, C308.-, C309.-, C310.+, C312.2, C313.2
- net N$42: now also C309.2, C313.2; no longer C307.2, C311.2
- net SS_DAC: now also Q604.B; no longer Q601.B
- net SS_DAC_I: now also C610.1, R610.1, U601.6; no longer C607.1, R607.1, U601.7
Routing:
- net SCK_I: track 0.00 -> 66.6 mm
- net CLR_DAC_I: track 0.00 -> 43.1 mm
- net +5V: track 31.9 -> 72.3 mm, vias 5 -> 8
- net GND: track 130.7 -> 163.6 mm, vias 11 -> 17
- net SS_DAC_I: track 0.00 -> 30.8 mm
- net N$37: track 0.00 -> 27.0 mm
- net FLT_DAC_I: track 0.00 -> 19.3 mm
- net SS_CL_I: track 26.9 -> 9.42 mm
- net SS_TEMP_I: track 23.4 -> 9.42 mm
- net SS_V_I: track 22.1 -> 9.42 mm
- net +3V3: track 14.0 -> 25.0 mm
- net SS_CH_I: track 18.8 -> 9.42 mm
- net -15V: track 32.9 -> 42.3 mm
- net MOSI_I: track 0.00 -> 9.42 mm
- net MISO: track 0.00 -> 9.42 mm
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- added copper zone on layer 16, net GND
Other:
- board size 200 x 200 mm -> 100 x 100 mm

Commit message: Board layout
Parts:
- moved Q601 79.9 mm to (97.0, 95.0), turned to 270 degrees
- moved R601 76.3 mm to (98.0, 89.5), turned to 270 degrees
- moved Q604 73.0 mm to (90.5, 95.0), turned to 270 degrees
- moved C601 72.4 mm to (93.5, 91.0), turned to 0 degrees
- moved C607 71.2 mm to (98.0, 82.5), turned to 90 degrees
- moved U601 71.1 mm to (93.5, 89.5), turned to 180 degrees
- moved C611 70.2 mm to (86.0, 96.5), turned to 270 degrees
- moved C604 69.9 mm to (93.5, 88.0), turned to 0 degrees
- moved R611 67.5 mm to (83.0, 96.5), turned to 270 degrees
- moved R607 67.4 mm to (95.0, 82.5), turned to 90 degrees
- moved R604 66.2 mm to (89.0, 89.5), turned to 270 degrees
- moved R608 64.9 mm to (80.0, 96.5), turned to 270 degrees
- moved R610 63.8 mm to (92.0, 82.5), turned to 90 degrees
- moved R605 63.0 mm to (86.0, 89.5), turned to 90 degrees
- moved C608 62.6 mm to (77.0, 96.5), turned to 270 degrees
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Routing:
- net GND: track 163.6 -> 227.6 mm
- net SCK_I: track 66.6 -> 9.42 mm
- net +5V: track 72.3 -> 120.4 mm
- net CLR_DAC_I: track 43.1 -> 9.42 mm
- net SS_DAC_I: track 30.8 -> 9.42 mm
- net FLT_DAC_I: track 19.3 -> 0.00 mm
- net SS_TEMP_I: track 9.42 -> 6.37 mm

Commit message: Board layout
Parts:
- added C314: 0.33µ, passives:C3216
- added C315: 0.1µ, passives:C3216
- added IC302: 7805T, linear:TO220H
- added PAD1, PAD405: S1, pads:PAD-10X4
- added PAD2, PAD406: S2, pads:PAD-10X4
- added PAD3, PAD407: UUT-, pads:PAD-10X4
- added PAD401: G1, pads:PAD-5X2
- added PAD402: G2, pads:PAD-5X2
- added PAD403: VS+, pads:PAD-5X2
- added PAD404: VS-, pads:PAD-5X2
- added R133, R217: 10k, passives:R1608
- C107: device rcl:C1206 -> passives:C1608
- C121, C122, C209, C210, C211, C212, C216, C607, C608, C609, C610, C611, C612, C619, C620, C621, C622, C623, C624: device passives:C3216 -> passives:C1608
- R101, R123, R124, R125, R201, R202, R203, R204, R210, R211, R212, R213, R214, R215, R216, R305, R306, R307, R308: device passives:R3225W -> passives:R2012W
- R102: value 1k -> 10k; device passives:R3225W -> passives:R1608
- R103, R107: value 100R -> 1k; device passives:R3225W -> passives:R3216W
- R104, R115, R120, R126: value 10k -> 100R; device passives:R3225W -> passives:R2012W
- R105, R114, R119, R122: value 100R -> 10k; device passives:R3225W -> passives:R1608
- R106: value 1k -> 100R; device passives:R3225W -> passives:R2012W
- R108: value 0R004 -> 100R; device rcl:R6332 -> passives:R2012W
- R109, R129: value 2R -> 0R004; device passives:R3225W -> passives:R6332W
- R110, R130: value 0R004 -> 2R; device rcl:R6332 -> passives:R3216W
- R111, R131: value 10k -> 0R004; device passives:R3225W -> passives:R6332W
- R112, R113, R116, R117, R118, R121, R127, R132, R301, R302, R303, R304, R601, R602, R603, R604, R605, R606, R607, R608, R609, R610, R611, R612, R613, R614, R615, R616, R617, R618, R619, R620, R621, R622, R623, R624: device passives:R3225W -> passives:R1608
- R128: value 0R004 -> 10k; device rcl:R6332 -> passives:R1608
- R205, R206, R207, R208, R209: device passives:R3225W -> passives:R3216W
- U302: value (none) -> LT1014
- moved Q110 167.7 mm to (66.0, 81.0)
- moved Q109 161.0 mm to (66.0, 87.0)
- moved Q108 154.7 mm to (66.0, 93.0)
- moved R115 144.4 mm to (-53.0, 111.0), turned to 0 degrees
- moved R120 141.4 mm to (-53.0, 114.0), flipped to the top
- moved R112 140.9 mm to (-59.0, 90.0), turned to 0 degrees
- moved R126 130.9 mm to (-53.0, 108.0), turned to 0 degrees
- moved R125 126.0 mm to (61.5, 55.5)
- moved R129 110.5 mm to (56.5, 84.0)
- moved Q106 108.6 mm to (29.0, 81.0), turned to 180 degrees
- moved Q601 108.3 mm to (12.2, 27.5), turned to 90 degrees
- moved C611 106.8 mm to (4.50, 27.5), flipped to the bottom, turned to 0 degrees
- moved R611 104.5 mm to (4.50, 27.5), turned to 180 degrees
- moved R601 102.8 mm to (10.5, 35.5), turned to 90 degrees
- moved Q102 102.6 mm to (29.0, 87.0), turned to 180 degrees
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Connections:
- removed net N$1: Q107.3, R105.2
- removed net N$2: Q111.3, R122.2
- removed net N$36: R205.1, S201.15
- new net GATE1: PAD401.1, Q107.3, R106.2
- new net GATE2: PAD402.1, Q111.3, R123.2
- new net N$44: C314.2, C315.2, IC302.2
- new net N$45: R217.2, U208.3
- new net VSENSE+: PAD403.1, R205.1, S201.15
- net +12V: now also C314.1, IC302.1, R105.2, R107.2; no longer R104.2, R106.2
- net +5V: now also C315.1, IC302.3, R102.1
- net BYP_G: now also R104.1, R108.1, R112.2, R115.1, R120.1, R126.1; no longer R103.1, R107.1, R111.2, R114.1, R119.1, R125.1
- net BYP_I: now also R103.1; no longer R102.1
- net CSENSE1_H: now also R109.2, R110.1, R111.2; no longer R108.2, R109.1, R110.2
- net CSENSE1_L: now also PAD1.1, PAD405.1, R110.2, R113.1; no longer R109.2, R112.1
- net CSENSE2_H: now also R129.2, R130.1, R131.2; no longer R128.2, R129.1, R130.2
- net CSENSE2_L: now also PAD2.1, PAD406.1, R114.1, R130.2; no longer R113.1, R129.2
- net FLT_DAC_I: now also R102.2
- net GND: now also R112.1, R133.1, R217.1; no longer R111.1, R131.1
- net LBQ12_G: now also R104.2; no longer R103.2
- net LBQ13_G: now also R108.2; no longer R107.2
- net LBQ21_G: now also R115.2; no longer R114.2
- net LBQ22_G: now also R120.2; no longer R119.2
- net LBQ23_G: now also R126.2; no longer R125.2
- net LQ1_G: now also R106.1, R127.2, R132.2; no longer R105.1, R126.2, R131.2
- net LQ2_G: now also R123.1, R128.2, R133.2; no longer R122.1, R127.2, R132.2
- net N$12: now also R121.2, R127.1; no longer R120.2, R126.1
- net N$13: now also R117.2, R121.1; no longer R115.2, R120.1
- net N$14: now also R113.2, R117.1; no longer R112.2, R115.1
- net N$15: now also R114.2, R119.1; no longer R113.2, R117.1
- net N$16: now also R119.2, R122.1; no longer R117.2, R121.1
- net N$5: now also R107.1; no longer R106.1
- net N$8: now also R103.2, R105.1; no longer R102.2, R104.1
- net N$9: now also R122.2, R128.1; no longer R121.2, R127.1
- net T1_OUT: now also R124.1; no longer R123.1
- net T2_OUT: now also R125.1; no longer R124.1
- net TEMP1: now also R124.2; no longer R123.2
- net TEMP2: now also R125.2; no longer R124.2
- net UUT-: now also PAD3.1, PAD407.1, R109.1, R111.1, R129.1, R131.1; no longer R108.1, R110.1, R128.1, R130.1
- net VSENSE-: now also PAD404.1
Routing:
- net GND: track 227.6 -> 120.0 mm, vias 17 -> 9
- net MISO_I: track 0.00 -> 93.5 mm, vias 0 -> 2
- net SCK_I: track 9.42 -> 96.9 mm, vias 0 -> 1
- net MOSI_I: track 9.67 -> 82.5 mm, vias 0 -> 1
- net SS_V_I: track 9.42 -> 51.4 mm, vias 0 -> 3
- net SS_TEMP_I: track 6.37 -> 45.1 mm, vias 0 -> 3
- net FLT_DAC_I: track 0.00 -> 34.9 mm, vias 0 -> 2
- net SS_CH_I: track 9.42 -> 36.9 mm, vias 0 -> 3
- net N$37: track 27.0 -> 0.00 mm
- net LBQ11_G: track 0.00 -> 24.7 mm, vias 0 -> 1
- net CLR_DAC_I: track 9.42 -> 31.4 mm, vias 0 -> 3
- net SS_DAC_I: track 9.42 -> 31.1 mm, vias 0 -> 3
- net N$11: track 10.7 -> 31.4 mm
- net SDO_DAC1: track 0.00 -> 20.5 mm
- net LBQ21_G: track 0.00 -> 20.4 mm, vias 0 -> 1
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- added copper zone on layer 1, net CSENSE1_H
- added copper zone on layer 16, net CSENSE1_H
- added copper zone on layer 1, net CSENSE1_L
- added copper zone on layer 16, net CSENSE1_L
- added copper zone on layer 1, net CSENSE2_H
- added copper zone on layer 16, net CSENSE2_H
- added copper zone on layer 1, net CSENSE2_L
- added copper zone on layer 16, net CSENSE2_L
- added copper zone on layer 1, net UUT-
- added copper zone on layer 16, net UUT-
Other:
- outline, holes or cut-outs redrawn
