File: PCB/V1A/Electronic_Load_V1A.brd (EAGLE design)
At the start: 100 x 100 mm, 241 parts, among them IC1 MEGA8-AI, IC101 LM50, IC102 LM50, IC301 7805T, IC302 7805T, Q101 SIRC10DP, Q102 SIRC10DP, Q103 BC817-16SMD, Q104 BC817-16SMD, Q105 BC807-16SMD, Q106 SIRC10DP, Q107 IXTK102N65X2R+, Q108 SIRC10DP, Q109 SIRC10DP, Q110 SIRC10DP, Q111 IXTK102N65X2R+, Q601 BC807-16SMD, Q602 BC807-16SMD, Q603 BC807-16SMD, Q604 BC807-16SMD, Q605 BC807-16SMD, Q606 BC807-16SMD, Q607 BC807-16SMD, Q608 BC807-16SMD, Q609 BC807-16SMD, Q610 BC807-16SMD, Q611 BC807-16SMD, Q612 BC807-16SMD, U101 AD420, U102 AD420, U103 LT1014I, U104 LTC1865L, U201 AD620, U202 AD620, U203 AD620, U204 AD620, U205 AD620, U206 LTC1865L, U207 LTC1865L, U208 LTC1865L, U301 MAX743, U302 LT1014, U601 HCPL-063N, U602 HCPL-063N, U603 HCPL-063N, U604 HCPL-063N, U605 HCPL-063N, U606 HCPL-063N

Commit message: Updated schematic
Parts:
- removed PAD401: G1, pads:PAD-5X2
- removed PAD402: G2, pads:PAD-5X2
- removed PAD403: VS+, pads:PAD-5X2
- removed PAD404: VS-, pads:PAD-5X2
- removed PAD405: S1, pads:PAD-10X4
- removed PAD406: S2, pads:PAD-10X4
- added PAD11: 12V, pads:PAD-5X2
- added PAD12, PAD16: GND, pads:PAD-5X2
- added PAD13: T1, pads:PAD-5X2
- added PAD14: T2, pads:PAD-5X2
- added PAD15: 5V, pads:PAD-5X2
- C213, C308: value 0.1µ -> 1µ; device passives:C3216 -> passives:CT3216
- C215: value 1µ -> 0.1µ; device passives:CT3216 -> passives:C3216
- C216: value 500p -> 0.1µ; device passives:C1608 -> passives:C3216
- C218: value 0.1µ -> 500p; device passives:C3216 -> passives:C1608
- C301: value 0.1µ -> 0.33µ
- C302: value 1µ -> 0.33µ; device passives:CT3216 -> passives:C3216
- C303: value 10n -> 220µ; device passives:C3216 -> rcl:E3,5-10
- C304: value 10µ -> 0.1µ; device passives:CT6032 -> passives:C3216
- C305: value 10n -> 0.1µ
- C307: value 220µ -> 0.1µ; device rcl:E3,5-10 -> passives:C3216
- C309: value 0.33µ -> 0.1µ
- C310: value 22µ -> 10n; device passives:CT6032 -> passives:C3216
- C311: value 220µ -> 10µ; device rcl:E3,5-10 -> passives:CT6032
- C312: value 220µ -> 10n; device rcl:E3,5-10 -> passives:C3216
- C313: value 0.1µ -> 22µ; device passives:C3216 -> passives:CT6032
- C314: value 0.33µ -> 220µ; device passives:C3216 -> rcl:E3,5-10
- C315: value 0.1µ -> 220µ; device passives:C3216 -> rcl:E3,5-10
- PAD1: value S1 -> G1; device pads:PAD-10X4 -> pads:PAD-5X2
- PAD2: value S2 -> G2; device pads:PAD-10X4 -> pads:PAD-5X2
- PAD3: value UUT- -> VS+; device pads:PAD-10X4 -> pads:PAD-5X2
- PAD4: value 12V -> VS-
- PAD5: value GND -> S1; device pads:PAD-5X2 -> pads:PAD-10X4
- PAD6: value T1 -> S2; device pads:PAD-5X2 -> pads:PAD-10X4
- PAD7: value T2 -> UUT-; device pads:PAD-5X2 -> pads:PAD-10X4
- PAD8: value 5V -> S1; device pads:PAD-5X2 -> pads:PAD-10X4
- PAD9: value GND -> S2; device pads:PAD-5X2 -> pads:PAD-10X4
- R208, R209: value 2M -> 100R; device passives:R3216W -> passives:R2012W
- R210, R211: value 2k15 -> 100R
- R212, R213: value 100R -> 2M; device passives:R2012W -> passives:R3216W
- R214, R215: value 100R -> 2k15
- moved PAD5 94.1 mm to (23.5, 86.5), turned to 90 degrees
- moved PAD8 77.0 mm to (23.5, 86.5), flipped to the bottom, turned to 90 degrees
- moved PAD4 76.1 mm to (92.0, 89.0), turned to 90 degrees
- moved C309 69.7 mm to (22.0, 71.0), turned to 90 degrees
- moved PAD2 62.5 mm to (14.0, 89.0), flipped to the top, turned to 90 degrees
- moved C308 52.4 mm to (57.5, 32.5), turned to 180 degrees
- moved PAD7 45.0 mm to (50.0, 86.5), turned to 90 degrees
- moved R209 43.8 mm to (37.5, 55.5), turned to 0 degrees
- moved C303 41.1 mm to (83.7, 6.42), turned to 90 degrees
- moved R208 40.1 mm to (44.5, 55.5), turned to 180 degrees
- moved C307 39.2 mm to (58.0, 36.0), turned to 0 degrees
- moved R215 38.6 mm to (74.5, 66.5), turned to 180 degrees
- moved PAD9 36.7 mm to (76.5, 86.5), flipped to the bottom, turned to 270 degrees
- moved PAD3 36.1 mm to (86.0, 89.0), flipped to the top, turned to 90 degrees
- moved C314 35.9 mm to (90.0, 40.0), turned to 0 degrees
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- renumbered IC1 to IC501, MOV1 to MOV201, MOV2 to MOV202, MOV3 to MOV203, MOV4 to MOV204, PAD407 to PAD10
Connections:
- net +12V: now also C301.1, C302.1, C303.+, PAD11.1; no longer C307.+, C309.1, C314.1, PAD4.1
- net +15V: now also C215.1, C314.+; no longer C213.1, C311.+
- net +3V3: now also C213.+, C216.1, C217.1; no longer C215.+, C218.1, C219.1
- net +5V: now also C304.1, C305.1, C307.2, C313.+, PAD15.1; no longer C301.2, C310.+, C313.1, C315.1, PAD8.1
- net -15V: now also C219.1, C309.1, C315.-; no longer C217.1, C308.1, C312.-
- net CSENSE1_H: now also U201.3, U202.2; no longer U203.3, U204.2
- net CSENSE1_L: now also PAD5.1, PAD8.1, U202.3; no longer PAD1.1, PAD405.1, U204.3
- net CSENSE2_H: now also U203.2, U204.3; no longer U201.2, U202.3
- net CSENSE2_L: now also PAD6.1, PAD9.1, U203.3; no longer PAD2.1, PAD406.1, U201.3
- net GATE1: now also PAD1.1; no longer PAD401.1
- net GATE2: now also PAD2.1; no longer PAD402.1
- net GND: now also C213.-, C215.2, C301.2, C302.2, C303.-, C304.2, C307.1, C308.-, C310.1, C312.2, C313.-, C314.-, C315.+, PAD12.1, PAD16.1, R214.1; no longer C213.2, C215.-, C301.1, C302.-, C303.1, C304.-, C307.-, C308.2, C310.-, C312.+, C313.2, C314.2, C315.2, PAD5.1, PAD9.1, R210.1
- net N$17: now also R210.1, U203.6; no longer R212.1, U201.6
- net N$18: now also C211.1, R210.2, U207.2; no longer C209.1, R212.2, U206.2
- net N$19: now also R211.1, U204.6; no longer R213.1, U202.6
- net N$20: now also C212.1, R211.2, U207.3; no longer C210.1, R213.2, U206.3
- net N$21: now also C209.1, R208.2, U206.2; no longer C211.1, R214.2, U207.2
- net N$22: now also C210.1, R209.2, U206.3; no longer C212.1, R215.2, U207.3
- net N$23: now also R209.1, U202.6; no longer R215.1, U204.6
- net N$24: now also R208.1, U201.6; no longer R214.1, U203.6
- net N$25: now also R212.1, R213.2; no longer R208.1, R209.2
- net N$26: now also R212.2; no longer R208.2
- net N$29: now also R213.1, R214.2; no longer R209.1, R210.2
- net N$30: now also C218.1; no longer C216.1
- net N$32: now also C312.1; no longer C305.1
- net N$33: now also C308.+; no longer C302.+
- net N$34: now also C310.2; no longer C303.2
- net RG1_H4: now also R203.2, U203.1; no longer R201.2, U201.1
- net RG1_H5: now also R204.2, U204.1; no longer R202.2, U202.1
- net RG1_H6: now also R215.2; no longer R211.2
- net RG1_L3: now also R201.2, U201.1; no longer R203.2, U203.1
- net RG1_L4: now also R202.2, U202.1; no longer R204.2, U204.1
- net RG2_H4: now also R203.1, U203.8; no longer R201.1, U201.8
- net RG2_H5: now also R204.1, U204.8; no longer R202.1, U202.8
- net RG2_H6: now also R215.1; no longer R211.1
- net RG2_L3: now also R201.1, U201.8; no longer R203.1, U203.8
- net RG2_L4: now also R202.1, U202.8; no longer R204.1, U204.8
- net SS_CH_I: now also U207.1; no longer U206.1
- net SS_CL_I: now also U206.1; no longer U207.1
- net T1_OUT: now also PAD13.1; no longer PAD6.1
- net T2_OUT: now also PAD14.1; no longer PAD7.1
- net UUT-: now also PAD7.1, U201.2, U204.2; no longer PAD3.1, U202.2, U203.2
- net VREF: now also C311.+; no longer C304.+
- net VSENSE+: now also PAD3.1; no longer PAD403.1
- net VSENSE-: now also PAD4.1; no longer PAD404.1
Routing:
- net VSENSE-: track 67.8 -> 58.3 mm
- net T1_OUT: track 28.1 -> 21.6 mm
- net GATE2: track 8.00 -> 2.05 mm
- net GATE1: track 8.85 -> 2.90 mm
- net VSENSE+: track 8.83 -> 4.33 mm
- net +12V: track 53.4 -> 50.3 mm
- net T2_OUT: track 33.7 -> 32.2 mm
- net GND: vias 15 -> 14

Commit message: Removed external parts from PCB, added Front Panel PCB
Parts:
- removed C122: 500p, passives:C1608
- removed IC101, IC102: LM50, linear:SOT23
- removed IC501: MEGA8-AI, atmel:TQFP32-08
- removed PAD10, PAD7: UUT-, pads:PAD-10X4
- removed PAD5, PAD8: S1, pads:PAD-10X4
- removed PAD6, PAD9: S2, pads:PAD-10X4
- removed Q107, Q111: IXTK102N65X2R+, transistors:TO-264P-H-PADUP
- removed U$3: (no value), mechanical:M3
- added PAD311, PAD312: S1, pads:PAD-10X4
- added PAD313, PAD314: S2, pads:PAD-10X4
- added PAD315, PAD316: UUT-, pads:PAD-10X4
- added PAD317: 12V, pads:PAD-5X2
- added PAD318: FAN_GND, pads:PAD-5X2
- added Q401: BC817-16SMD, transistor-npn:SOT23-BEC
- added Q402: SIRC10DP, transistors:POWERPAK-SO-8
- added R401: 1k, passives:R1608
- added U$5: (no value), mechanical:M3
- C116, C118: value 0.1µ -> 1µ; device passives:C3216 -> passives:CT3216
- C117: value 1µ -> 0.1µ; device passives:CT3216 -> passives:C3216
- C120: value 1µ -> 500p; device passives:CT3216 -> passives:C1608
- R103, R107: device passives:R3216W -> passives:R1608
- moved Q105 146.0 mm to (54.0, 74.0), flipped to the bottom, turned to 180 degrees
- moved Q104 134.9 mm to (54.0, 69.5), flipped to the bottom, turned to 180 degrees
- moved R120 121.0 mm to (61.0, 73.5), flipped to the bottom, turned to 180 degrees
- moved R115 120.8 mm to (61.0, 71.0), flipped to the bottom, turned to 180 degrees
- moved R126 118.4 mm to (61.0, 76.0), flipped to the bottom, turned to 180 degrees
- moved R112 117.1 mm to (57.0, 74.0), flipped to the bottom, turned to 90 degrees
- moved C108 116.8 mm to (50.0, 69.0), flipped to the bottom, turned to 90 degrees
- moved Q103 115.5 mm to (50.0, 74.0), flipped to the bottom, turned to 180 degrees
- moved R107 110.4 mm to (46.5, 69.5), flipped to the bottom, turned to 270 degrees
- moved R105 110.0 mm to (44.0, 69.5), flipped to the bottom, turned to 270 degrees
- moved C107 104.7 mm to (44.0, 74.0), flipped to the bottom, turned to 90 degrees
- moved R103 103.4 mm to (46.5, 74.0), flipped to the bottom, turned to 90 degrees
- moved R108 100.0 mm to (39.0, 76.0), flipped to the bottom
- moved R101 98.1 mm to (39.0, 71.0), flipped to the bottom
- moved R104 94.7 mm to (39.0, 73.5), flipped to the bottom
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- renumbered C601 to C501, C602 to C502, C603 to C503, C604 to C504, C605 to C505, C606 to C506, C607 to C507, C608 to C508, C609 to C509, C610 to C510, C611 to C511, C612 to C512, C613 to C513, C614 to C514, C615 to C515, C616 to C516, C617 to C517, C618 to C518, C619 to C519, C620 to C520, C621 to C521, C622 to C522, C623 to C523, C624 to C524, PAD1 to PAD301, PAD11 to PAD305, PAD12 to PAD306, PAD13 to PAD307, PAD14 to PAD308, PAD15 to PAD309, PAD16 to PAD310, PAD2 to PAD302, PAD3 to PAD303, PAD4 to PAD304, Q601 to Q501, Q602 to Q502, Q603 to Q503, Q604 to Q504, Q605 to Q505, Q606 to Q506, Q607 to Q507, Q608 to Q508, Q609 to Q509, Q610 to Q510, Q611 to Q511, Q612 to Q512, R601 to R501, R602 to R502, R603 to R503, R604 to R504, R605 to R505, R606 to R506, R607 to R507, R608 to R508, R609 to R509, R610 to R510, R611 to R511, R612 to R512, R613 to R513, R614 to R514, R615 to R515, R616 to R516, R617 to R517, R618 to R518, R619 to R519, R620 to R520, R621 to R521, R622 to R522, R623 to R523, R624 to R524, U104 to U106, U601 to U501, U602 to U502, U603 to U503, U604 to U504, U605 to U505, U606 to U506
Connections:
- removed net AVCC: IC501.18
- removed net VCC: IC501.4, IC501.6
- new net FAN_GND: PAD318.1, Q402.5
- new net N$42: Q401.C, Q402.4
- new net N$44: Q401.B, R401.2
- new net VREF2: C311.+, U301.6
- net +12V: now also PAD317.1
- net +3V3: now also C116.+, C117.1; no longer C117.+, C118.1
- net +5V: no longer C115.1, IC101.1, IC102.1
- net -15V: now also C115.1; no longer C116.1
- net CSENSE1_L: now also PAD311.1, PAD312.1; no longer PAD5.1, PAD8.1, Q107.1
- net CSENSE2_L: now also PAD313.1, PAD314.1; no longer PAD6.1, PAD9.1, Q111.1
- net GATE1: no longer Q107.3
- net GATE2: no longer Q111.3
- net GND: now also C116.-, C117.2, C118.-, C120.2, Q401.E, Q402.1, Q402.2, Q402.3; no longer C116.2, C117.-, C118.2, C120.-, C122.2, IC101.3, IC102.3, IC501.21, IC501.3, IC501.5
- net T1_OUT: now also C118.+; no longer C119.+, IC101.2
- net T2_OUT: now also C119.+; no longer C120.+, IC102.2
- net TEMP1: now also C120.1; no longer C121.1
- net TEMP2: now also C121.1; no longer C122.1
- net UUT+: no longer Q107.2, Q111.2
- net UUT-: now also PAD315.1, PAD316.1; no longer PAD10.1, PAD7.1
- net VREF: no longer C311.+, U301.6
Routing:
- net BYP_G: track 0.00 -> 35.1 mm
- net GND: track 122.4 -> 139.0 mm, vias 14 -> 24
- net +5V: track 40.7 -> 25.5 mm
- net N$8: track 0.00 -> 12.4 mm
- net N$5: track 0.00 -> 11.8 mm
- net +12V: track 50.3 -> 61.0 mm
- net VREF: track 28.3 -> 20.5 mm
- net VREF2: track 0.00 -> 7.85 mm
- net T1_OUT: track 21.6 -> 28.1 mm
- net LBQ11_G: track 24.7 -> 29.5 mm
- net LBQ12_G: track 17.6 -> 21.6 mm
- net LBQ13_G: track 10.6 -> 13.7 mm
- net LBQ21_G: track 20.4 -> 23.5 mm
- net LBQ22_G: track 12.7 -> 15.6 mm
- net BYP_I: track 5.18 -> 7.68 mm
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Other:
- outline, holes or cut-outs redrawn
- board text added: "Fan Power"
