File: PCB/V1A/MOSFET_Board.brd (EAGLE design)
At the start: 230 x 115 mm, 278 parts, among them IC301 78L05_TO-220AB-3-BR, IC302 78L05_TO-220AB-3-BR, J301 TEMP, J302 +12V, J303 CTRL, J304 FAN_MOLEX4PIN, J305 FAN_MOLEX4PIN, J306 DUT+, J307 DUT-, Q201 SIRC10DP, Q202 SIRC10DP, Q203 BC817, Q204 BC817, Q205 SIRC10DP, Q206 SIRC10DP, Q207 BC817, Q208 BC807, Q209 BC817, Q210 BC807, Q211 IXTK102N65X2, Q212 IXTK102N65X2, Q301 BC817, Q302 BC817, Q401 BC807, Q402 BC807, Q403 BC807, Q404 BC807, Q405 BC807, Q406 BC807, Q407 BC807, Q408 BC807, Q409 BC807, Q410 BC807, Q411 BC807, Q412 BC807, Q413 BC807, Q414 BC807, U201 AD420, U202 AD420, U203 LT1014I, U204 LT1014I, U205 AD620, U206 AD620, U207 AD620, U208 AD620, U209 LTC1865L, U210 LTC1865L, U301 LP2985-3.1, U302 LP2985-3.1, U303 LP2985-3.1, U304 AD620, U305 LTC1865L, U306 LTC1865L, U307 MAX743, U401 HCPL-063N, U402 HCPL-063N, U403 HCPL-063N, U404 HCPL-063N, U405 HCPL-063N, U406 HCPL-063N, U407 HCPL-063N

Commit message: Added power amp for load MOSFET gate
Parts:
- removed R201, R203, R207, R209, R211, R213, R214, R215, R219, R221, R223: 10k, passives:RESC1608
- removed R205: 100k, passives:RESC1608
- added Q1, Q3: BC807, transistors:SOT23
- added Q2, Q4: BC817, transistors:SOT23
- added R1: 10k, passives:RESC1608
- added R2, R5: 1k, passives:RESC1608
- added R3, R4: 2R, passives:RESC3216
Connections:
- removed net N$12: R205.2, R207.2, R211.2, R213.1, R214.1, U203.6
- new net N$67: Q1.1, Q4.1, R229.2
- new net N$68: Q3.1, Q4.2, R5.2
- net CSEN_L1: no longer R201.1
- net DAC_VOUT: now also U203.14; no longer U203.5
- net DUT-: no longer R203.1
- net GND: now also R1.1; no longer R207.1, R209.1, R211.1, R223.1
- net LGATE_1: now also R3.1, R4.2; no longer R229.2
- net N$1: now also Q1.2, Q2.1, R2.1; no longer R203.2, R209.2, U203.12
- net N$11: now also Q3.2, R4.1; no longer R213.2, R214.2, R219.1, U203.7
- net N$13: now also Q2.2, R3.2; no longer R215.2, R221.1, U203.10
- net N$14: now also Q2.3, Q4.3, R2.2; no longer R201.2, R215.1, U203.11
- net N$2: now also R1.2; no longer R221.2
- net N$9: now also Q1.3, Q3.3, R5.1; no longer R219.2, R223.2, U203.14
- net VREF1: no longer R205.1
Routing:
- net N$13: track 22.1 -> 0.00 mm
- net N$1: track 19.9 -> 0.00 mm, vias 3 -> 0
- net N$14: track 19.3 -> 0.00 mm
- net DUT-: track 134.6 -> 115.5 mm
- net N$9: track 16.4 -> 0.00 mm, vias 3 -> 0
- net N$12: track 13.5 -> 0.00 mm
- net N$11: track 10.0 -> 0.00 mm
- net VREF1: track 42.5 -> 33.7 mm
- net GND: track 310.1 -> 303.6 mm, vias 106 -> 103
- net DAC_VOUT: track 12.3 -> 6.29 mm
- net N$2: track 7.74 -> 5.69 mm
- net CSEN_L1: track 35.7 -> 33.9 mm
- net LGATE_1: track 9.02 -> 7.39 mm
- net -15V: track 114.4 -> 115.7 mm
- removed copper zone on layer 1, net +15V
- removed copper zone on layer 1, net -15V

Commit message: Changed load path layout
Parts:
- removed C329, C401, C402, C403, C404, C417, C418, C419: 100n, passives:CAPC1608
- removed C330: 470n, passives:CAPC1608
- removed C331: 10n, passives:CAPC2012
- removed C332: 220µ, passives:CAPPRD500W60D1000H
- removed C405, C406, C407, C408, C420, C421, C422: 10n, passives:CAPC1608
- removed C409, C410, C411, C412, C413, C414, C415, C416, C423, C424, C425, C426, C427, C428: 15p, passives:CAPC1608
- removed D204, D301: BAT54S, diode:SOT23
- removed D302, D303: 1N5817-B, diode:DO41-7.6
- removed IC301, IC302: 78L05_TO-220AB-3-BR, ic:TO-220AB-3-BR
- removed J301: TEMP, mechanical:HEAD_MALE_2X3
- removed J306: DUT+, mechanical:AMPHENOL-12-762_2
- removed J307: DUT-, mechanical:AMPHENOL-12-762_2
- removed MOV301, MOV302: 416NR10D, passives:DISK_9.5MM
- removed Q1, Q208, Q210, Q3, Q401, Q402: BC807, transistors:SOT23
- removed Q2, Q203, Q204, Q207, Q209, Q4: BC817, transistors:SOT23
- removed Q205, Q206: SIRC10DP, transistors:POWERPAK-SO-8
- removed R1, R216, R217, R218, R220, R222, R224, R225, R226: 10k, passives:RESC1608
- removed R2, R231, R233, R237, R239, R5: 1k, passives:RESC1608
- removed R227, R228, R247, R248, R251, R252, R253, R254: 2k15, passives:RESC2012
- removed R229, R230, R255, R256, R257, R258: 100R, passives:RESC1608
- removed R232, R234, R238, R240, R243, R245, R3, R4: 2R, passives:RESC3216
- removed R235, R236: 100k, passives:RESC1608
- removed R241, R242, R244, R246, R249, R250: 0R01, passives:RESC6332
- removed R401, R402, R403, R404, R405, R406, R407, R408, R409, R410, R412, R413: 350R, passives:RESC1608
- removed SJ301: DUT_GND, jumper:SJW
- removed U210: LTC1865L, ic:SO8
- removed U401, U402, U403, U404, U405, U406, U407: HCPL-063N, ic:SO8
- added C101, C102, C133, C134: 4µ7, passives:CAPC3216
- added C103, C104, C105, C106, C111, C112, C113, C114, C119, C120, C121, C122, C123, C124, C125, C126, C127, C128, C135, C136: 100n, passives:CAPC1608
- added C107, C108, C109, C110: 10n, passives:CAPC2012
- added C115, C116, C117, C118: 470n, passives:CAPC1608
- added C129, C130, C131, C132: 470p, passives:CAPC1608
- added D101, D102, D103, D104: BAT54S, diode:SOT23
- added J201: TEMP, mechanical:HEAD_MALE_2X3
- added J206: DUT+, mechanical:AMPHENOL-12-762_2
- added J207: DUT-, mechanical:AMPHENOL-12-762_2
- added MOV201, MOV202: 416NR10D, passives:DISK_9.5MM
- added Q101, Q103, Q106, Q108, Q116, Q118: BC807, transistors:SOT23
- added Q102, Q104, Q105, Q107, Q111, Q112, Q115, Q117: BC817, transistors:SOT23
- added Q109, Q110, Q113, Q114: SIRC10DP, transistors:POWERPAK-SO-8
- added R101, R102: 49k3, passives:RESC1608
- added R103, R104, R105, R106: 5k, passives:RESC1608
- added R107, R108, R109, R110, R112, R114, R118, R120, R123, R125: 2R, passives:RESC3216
- added R111, R113, R117, R119: 1k, passives:RESC1608
- added R115, R116: 100k, passives:RESC1608
- added R121, R122, R124, R126, R129, R130: 0R01, passives:RESC6332
- added R127, R128, R131, R132, R133, R134, R207: 2k15, passives:RESC2012
- added R135, R136, R137, R138, R209: 100R, passives:RESC1608
- added R201, R203, R205: 2M, passives:RESC3216
- added R211: 350R, passives:RESC1608
- added SJ201: DUT_GND, jumper:SJW
- added U101, U102: AD420, ic:SO24W
- added U103, U104, U105, U106, U107, U108: AD620, ic:SO8
- added U109, U110: LTC1865L, ic:SO8
- C201, C202, C203, C217, C224: value 100n -> 4µ7; device passives:CAPC1608 -> passives:CAPC3216
- C208: value 10n -> 4µ7; device passives:CAPC2012 -> passives:CAPC3216
- C211, C212, C213, C215: value 100n -> 470n
- C218: value 100n -> 470p
- C223: value 100n -> 47µ; device passives:CAPC1608 -> passives:CAPCP7343
- C225: value 470p -> 4µ7; device passives:CAPC1608 -> passives:CAPC3216
- C226: value 470p -> 10n; device passives:CAPC1608 -> passives:CAPC2012
- C227: value 470p -> 10µ; device passives:CAPC1608 -> passives:CAPCP6032
- C228, C318: value 470p -> 100n
- C229, C301, C302, C303, C317: value 4µ7 -> 100n; device passives:CAPC3216 -> passives:CAPC1608
- C230: value 4µ7 -> 470n; device passives:CAPC3216 -> passives:CAPC1608
- C231: value 100n -> 10n; device passives:CAPC1608 -> passives:CAPC2012
- C232: value 100n -> 220µ; device passives:CAPC1608 -> passives:CAPPRD500W60D1000H
- C305, C306, C307: device passives:CAPC2012 -> passives:CAPC1608
- C308: value 4µ7 -> 10n; device passives:CAPC3216 -> passives:CAPC1608
- C309, C310, C324, C325: value 4µ7 -> 15p; device passives:CAPC3216 -> passives:CAPC1608
- C311, C312, C313, C315: value 470n -> 15p
- C314, C316, C328: value 100n -> 15p
- C320, C321, C322: value 100n -> 10n
- C323: value 47µ -> 15p; device passives:CAPCP7343 -> passives:CAPC1608
- C326: value 10n -> 15p; device passives:CAPC2012 -> passives:CAPC1608
- C327: value 10µ -> 15p; device passives:CAPCP6032 -> passives:CAPC1608
- D202, D203: value BAT54S -> 1N5817-B; device diode:SOT23 -> diode:DO41-7.6
- Q201, Q202: value SIRC10DP -> BC817; device transistors:POWERPAK-SO-8 -> transistors:SOT23
- Q301, Q302: value BC817 -> BC807
- R202, R208: value 10k -> 2k15; device passives:RESC1608 -> passives:RESC2012
- R204: value 10k -> 2M; device passives:RESC1608 -> passives:RESC3216
- R206: value 100k -> 2M; device passives:RESC1608 -> passives:RESC3216
- R212, R310: value 10k -> 350R
- R301, R303, R304, R305, R306: value 2M -> 350R; device passives:RESC3216 -> passives:RESC1608
- R302, R307, R308: value 2k15 -> 350R; device passives:RESC2012 -> passives:RESC1608
- R309: value 100R -> 350R
- U201, U202: value AD420 -> LP2985-3.1; device ic:SO24W -> ic:SOT23-5L
- U203: value LT1014I -> LP2985-3.1; device ic:SO16W -> ic:SOT23-5L
- U204: value LT1014I -> AD620; device ic:SO16W -> ic:SO8
- U205, U206: value AD620 -> 78L05_TO-220AB-3-BR; device ic:SO8 -> ic:TO-220AB-3-BR
- U207, U208: value AD620 -> LTC1865L
- U209: value LTC1865L -> MAX743; device ic:SO8 -> ic:SO16W
- U301, U302, U303: value LP2985-3.1 -> HCPL-063N; device ic:SOT23-5L -> ic:SO8
- U304: value AD620 -> HCPL-063N
- U305, U306: value LTC1865L -> HCPL-063N
- U307: value MAX743 -> HCPL-063N; device ic:SO16W -> ic:SO8
- moved C213 226.4 mm to (148.0, -61.0), flipped to the bottom, turned to 90 degrees
- moved U206 187.7 mm to (143.0, -61.0), turned to 0 degrees
- moved C222 180.3 mm to (138.0, -61.0), flipped to the bottom, turned to 90 degrees
- moved R306 177.5 mm to (-70.0, -45.5), turned to 0 degrees
- moved C319 175.5 mm to (-77.0, -47.0), flipped to the bottom
- moved R302 174.8 mm to (-65.5, -45.5), turned to 180 degrees
- moved C328 163.1 mm to (-75.0, -49.5), flipped to the bottom, turned to 180 degrees
- moved R301 160.3 mm to (-47.5, -45.5), turned to 180 degrees
- moved R305 158.8 mm to (-52.0, -45.5), turned to 0 degrees
- moved R310 155.7 mm to (-66.0, -28.0), turned to 180 degrees
- moved R307 152.0 mm to (-43.0, -45.5), turned to 0 degrees
- moved C318 149.6 mm to (-59.0, -33.0), turned to 0 degrees
- moved C322 147.3 mm to (-77.0, -45.0), turned to 180 degrees
- moved U306 145.3 mm to (-59.0, -40.0), turned to 0 degrees
- moved C216 145.3 mm to (92.9, -19.6), flipped to the top, turned to 270 degrees
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- renumbered C333 to C233, C334 to C234, C335 to C235, C337 to C236, C338 to C237, C339 to C238, C340 to C239, HS201 to HS101, HS202 to HS102, J302 to J202, J303 to J203, J304 to J204, J305 to J205, L301 to L201, L302 to L202, L303 to L203, PS301 to PS201, Q211 to Q119, Q212 to Q120, Q403 to Q303, Q404 to Q304, Q405 to Q305, Q406 to Q306, Q407 to Q307, Q408 to Q308, Q409 to Q309, Q410 to Q310, Q411 to Q311, Q412 to Q312, Q413 to Q313, Q414 to Q314, R411 to R311, R414 to R314, R415 to R315, R416 to R316, R417 to R317, R418 to R318, R419 to R319, R420 to R320, R421 to R321, R422 to R322, R423 to R323, R424 to R324, R425 to R325, R426 to R326, R427 to R327, R428 to R328
Connections:
- removed net DAC_VOUT: U201.17, U203.14
- removed net DAC_VOUT1: U202.17, U204.5
- removed net N$52: R226.2, R228.2, R230.1, U204.16
- removed net N$53: R220.2, R224.2, U204.14
- removed net N$54: R216.2, R217.2, R220.1, U204.7
- removed net N$55: U204.1, U204.2
- new net N$12: Q103.2, Q107.1, R105.1
- net +12V: now also C105.1, C106.1, C107.1, C108.1, C109.1, C110.1, C119.1, C120.1, C212.1, C232.+, Q115.3, Q117.3, R115.2, R116.2, R117.2, R119.2, U101.23, U102.23, U205.1, U206.1; no longer C205.1, C206.1, C207.1, C208.1, C214.1, C215.1, C216.1, C312.1, C313.1, C332.+, IC301.1, IC302.1, Q207.3, Q209.3, R235.2, R236.2, R237.2, R239.2, U201.23, U202.23
- net +15V: now also C111.1, C113.1, C115.1, C117.1, C121.1, C122.1, C123.1, C124.1, C216.1, Q102.3, Q104.3, Q105.3, Q107.3, Q202.2, R103.2, R105.2, U103.7, U104.7, U105.7, U106.7, U107.7, U108.7, U204.7; no longer C201.1, C202.1, C217.1, C218.1, C219.1, C220.1, C316.1, Q302.2, U203.4, U204.4, U205.7, U206.7, U207.7, U208.7, U304.7
- net +3V3: now also C210.1, R310.2, R312.2, U203.5; no longer C310.1, R410.2, R412.2, U303.5
- net +3V_1: now also C133.1, C135.1, C208.1, C217.1, C220.1, D101.2, D102.2, U109.8, U201.5, U207.8; no longer C229.1, C231.1, C308.1, C317.1, C320.1, D201.2, D202.2, U209.8, U301.5, U305.8
- net +3V_2: now also C134.1, C136.1, C209.1, C224.1, C228.1, D103.2, D104.2, D201.2, U110.8, U202.5, U208.8; no longer C230.1, C232.1, C309.1, C324.1, C328.1, D203.2, D204.2, D301.2, U210.8, U302.5, U306.8
- net +5V: now also C101.1, C102.1, C103.1, C104.1, C203.1, C204.1, C214.1, C221.1, C222.1, C223.+, C225.1, C229.2, C301.1, C302.1, C305.1, C306.1, C307.1, C308.1, C317.1, C318.1, C320.1, J201.3, J201.4, R309.2, R313.2, U101.2, U102.2, U203.1, U203.3, U205.3, U206.3, U209.12, U209.13, U209.3, U209.4, U209.5, U301.8, U302.8, U303.8, U304.8, U305.8, U306.8; no longer C209.1, C210.1, C211.1, C212.1, C314.1, C322.1, C323.+, C325.1, C329.2, C401.1, C402.1, C403.1, C404.1, C405.1, C406.1, C407.1, C408.1, C417.1, C418.1, C420.1, C421.1, IC301.3, IC302.3, J301.3, J301.4, R409.2, R413.2, U201.2, U202.2, U303.1, U303.3, U307.12, U307.13, U307.3, U307.4, U307.5, U401.8, U402.8, U403.8, U404.8, U405.8, U406.8
- net +5V_I: now also C319.1, C322.1, R301.2, R302.2, R303.2, R304.2, R305.2, R306.2, R307.2, R308.2, U307.8; no longer C419.1, C422.1, R401.2, R402.2, R403.2, R404.2, R405.2, R406.2, R407.2, R408.2, U407.8
- net -15V: now also C112.2, C114.2, C116.2, C118.2, C125.1, C126.1, C127.1, C128.1, C219.1, Q101.3, Q103.3, Q106.3, Q108.3, Q201.2, R104.1, R106.1, U103.4, U104.4, U105.4, U106.4, U107.4, U108.4, U204.4; no longer C203.1, C204.1, C221.1, C222.1, C223.1, C224.1, C319.1, Q301.2, U203.13, U204.13, U205.4, U206.4, U207.4, U208.4, U304.4
- net BPY1G1: now also Q109.4, R112.2; no longer Q201.4, R232.2
- net BYP: now also C309.1, R111.1, R113.1, R309.1, U301.7; no longer C409.1, R231.1, R233.1, R409.1, U401.7
- net BYP1: now also Q117.2, Q118.2, R112.1, R118.1, R128.1; no longer Q209.2, Q210.2, R232.1, R238.1, R248.1
- net BYP1G2: now also Q113.4, R118.2; no longer Q205.4, R238.2
- net BYP2: now also Q115.2, Q116.2, R114.1, R120.1, R127.2; no longer Q207.2, Q208.2, R234.1, R240.1, R247.2
- net BYP2G1: now also Q110.4, R114.2; no longer Q202.4, R234.2
- net BYP2G2: now also Q114.4, R120.2; no longer Q206.4, R240.2
- net BYP_I: now also Q301.1; no longer Q401.1
- net CLR_DAC1: now also C324.1, U101.6, U306.7; no longer C424.1, U201.6, U406.7
- net CLR_DAC2: now also C313.1, R313.1, U102.6, U301.6; no longer C413.1, R413.1, U202.6, U401.6
- net CONV_C1: now also C315.1, U109.1, U303.6; no longer C415.1, U209.1, U403.6
- net CONV_C2: now also C316.1, U110.1, U304.6; no longer C416.1, U210.1, U404.6
- net CONV_TEMP: now also C311.1, U207.1, U303.7; no longer C411.1, U305.1, U403.7
- net CONV_V: now also C312.1, R312.1, U208.1, U304.7; no longer C412.1, R412.1, U306.1, U404.7
- net CSEN_H1: now also Q109.1, Q109.2, Q109.3, Q113.1, Q113.2, Q113.3, R121.2, R123.1, R124.2, R128.2, R129.2, U105.3, U106.2; no longer Q201.1, Q201.2, Q201.3, Q205.1, Q205.2, Q205.3, R241.2, R243.1, R244.2, R248.2, R249.2, U205.3, U206.2
- net CSEN_H2: now also Q110.1, Q110.2, Q110.3, Q114.1, Q114.2, Q114.3, R122.2, R125.1, R126.2, R127.1, R130.2, U107.3, U108.2; no longer Q202.1, Q202.2, Q202.3, Q206.1, Q206.2, Q206.3, R242.2, R245.1, R246.2, R247.1, R250.2, U207.3, U208.2
- net CSEN_L1: now also Q109.5, Q109.6, Q109.7, Q109.8, Q113.5, Q113.6, Q113.7, Q113.8, R123.2, U103.5, U106.3; no longer Q201.5, Q201.6, Q201.7, Q201.8, Q205.5, Q205.6, Q205.7, Q205.8, R227.1, R243.2, U206.3
- net CSEN_L2: now also Q110.5, Q110.6, Q110.7, Q110.8, Q114.5, Q114.6, Q114.7, Q114.8, R125.2, U104.5, U108.3; no longer Q202.5, Q202.6, Q202.7, Q202.8, Q206.5, Q206.6, Q206.7, Q206.8, R202.1, R228.1, R245.2, U208.3
- net DUT+: now also J206.2; no longer J306.2
- net DUT-: now also J207.1, R121.1, R122.1, R124.1, R126.1, R129.1, R130.1, SJ201.2, U105.2, U107.2; no longer J307.1, R204.1, R241.1, R242.1, R244.1, R246.1, R249.1, R250.1, SJ301.2, U205.2, U207.2
- net FAN1_PWM: now also C323.1, U305.7; no longer C423.1, U405.7
- net FAN2_PWM: now also C326.1, U305.6; no longer C426.1, U405.6
- net FLT_DAC: now also U101.3, U102.3; no longer U201.3, U202.3
- net FLT_DAC_I: now also C325.1, U307.7; no longer C425.1, U407.7
- net GND: now also C101.2, C102.2, C103.2, C104.2, C105.2, C106.2, C111.2, C112.1, C113.2, C114.1, C115.2, C116.1, C117.2, C118.1, C119.2, C120.2, C121.2, C122.2, C123.2, C124.2, C125.2, C126.2, C127.2, C128.2, C129.2, C130.2, C131.2, C132.2, C133.2, C134.2, C135.2, C136.2, C205.2, C206.2, C207.2, C208.2, C223.-, C226.1, C227.-, C229.1, C232.-, C323.2, C326.2, C327.2, D101.1, D102.1, D103.1, D104.1, J201.1, J201.2, Q111.2, Q112.2, Q116.3, Q118.3, R207.1, SJ201.1, U101.11, U101.4, U101.5, U102.11, U102.4, U102.5, U103.2, U104.2, U105.5, U106.5, U107.5, U108.5, U109.4, U110.4, U201.2, U202.2, U203.2, U204.5, U205.2, U206.2, U207.4, U208.4, U209.11, U209.14, U209.2, U301.5, U302.5, U303.5, U305.5, U306.5, U307.3; no longer C223.2, C226.2, C227.2, C229.2, C232.2, C319.2, C322.2, C323.-, C325.2, C326.1, C327.-, C328.2, C329.1, C330.2, C331.2, C332.-, C401.2, C402.2, C403.2, C404.2, C405.2, C406.2, C407.2, C408.2, C409.2, C410.2, C411.2, C412.2, C413.2, C414.2, C415.2, C416.2, C417.2, C418.2, C420.2, C421.2, C423.2, C424.2, C426.2, C427.2, D202.1, D203.1, D204.1, D301.1, IC301.2, IC302.2, J301.1, J301.2, Q203.2, Q204.2, Q208.3, Q210.3, R1.1, R208.1, R212.1, R224.1, R307.1, R310.1, SJ301.1, U201.11, U201.4, U201.5, U202.11, U202.4, U202.5, U203.3, U204.3, U205.5, U206.5, U207.5, U208.5, U209.4, U210.4, U301.2, U302.2, U303.2, U305.4, U306.4, U307.11, U307.14, U401.5, U402.5, U403.5, U404.5, U405.5, U406.5, U407.2, U407.3
- net GNDI: now also C319.2, C322.2, C325.2, C328.2, Q301.3, Q302.3, U301.2, U301.3, U302.2, U302.3, U303.2, U303.3, U304.2, U304.3, U305.2, U305.3, U306.2, U306.3, U307.5; no longer C419.2, C422.2, C425.2, C428.2, Q401.3, Q402.3, U401.2, U401.3, U402.2, U402.3, U403.2, U403.3, U404.2, U404.3, U405.2, U405.3, U406.2, U406.3, U407.5
- net HIGHC1: now also C129.1, R135.2, U109.2; no longer C225.1, R255.2, U209.2
- net HIGHC2: now also C131.1, R137.2, U110.2; no longer C227.1, R257.2, U210.2
- net LATCH_DAC: now also C327.1, U101.7, U102.7, U306.6; no longer C427.1, U201.7, U202.7, U406.6
- net LGATE_1: now also R107.1, R108.2; no longer R3.1, R4.2
- net LGATE_2: now also R109.1, R110.2; no longer R230.2
- net LOWC1: now also C130.1, R136.2, U109.3; no longer C226.1, R256.2, U209.3
- net LOWC2: now also C132.1, R138.2, U110.3; no longer C228.1, R258.2, U210.3
- net MISO: now also U109.6, U110.6, U207.6, U208.6; no longer U209.6, U210.6, U305.6, U306.6
- net MISO_I: now also C328.1, U307.6; no longer C428.1, U407.6
- net MOSI: now also C310.1, R310.1, U101.9, U109.5, U110.5, U207.5, U208.5, U302.7; no longer C410.1, R410.1, U201.9, U209.5, U210.5, U305.5, U306.5, U402.7
- net MOSI_I: now also Q302.1; no longer Q402.1
- net N$1: now also Q101.2, Q105.1, R103.1; no longer Q1.2, Q2.1, R2.1
- net N$10: now also C205.1, U201.4; no longer C305.1, U301.4
- net N$11: now also Q106.2, R108.1; no longer Q3.2, R4.1
- net N$13: now also Q105.2, R107.2; no longer Q2.2, R3.2
- net N$14: now also Q108.2, R110.1; no longer Q2.3, Q4.3, R2.2
- net N$15: now also Q107.2, R109.2; no longer U203.1, U203.2
- net N$16: now also D102.3, R136.1, U106.6; no longer D202.3, R256.1, U206.6
- net N$17: now also U307.1; no longer U407.1
- net N$18: now also U307.4; no longer U407.4
- net N$19: now also R304.1, U304.1; no longer R404.1, U404.1
- net N$2: now also R101.2, U103.1; no longer R1.2, R225.1, U203.15
- net N$20: now also R308.1, U304.4; no longer R408.1, U404.4
- net N$21: now also Q302.2, R302.1, U302.1; no longer Q402.2, R402.1, U402.1
- net N$22: now also R306.1, U302.4; no longer R406.1, U402.4
- net N$23: now also R209.1, U204.6; no longer R309.1, U304.6
- net N$24: now also R205.1, R206.2; no longer R305.1, R306.2
- net N$25: now also Q111.3, Q115.1, Q116.1, R117.1; no longer Q203.3, Q207.1, Q208.1, R237.1
- net N$26: now also R203.2, R205.2; no longer R303.2, R305.2
- net N$27: now also R203.1, R204.2; no longer R303.1, R304.2
- net N$28: now also MOV201.2, MOV202.1; no longer MOV301.2, MOV302.1
- net N$29: now also R206.1, R207.2, U204.3; no longer R306.1, R307.2, U304.3
- net N$3: now also C107.2, U101.21; no longer C205.2, U201.21
- net N$30: now also C218.1, D201.3, R209.2, U208.2; no longer C318.1, D301.3, R309.2, U306.2
- net N$31: now also Q111.1, R111.2, R115.1; no longer Q203.1, R231.2, R235.1
- net N$32: now also D202.C, Q202.3, R211.1, U209.16; no longer D302.C, Q302.3, R312.1, U307.16
- net N$33: now also R201.2, R204.1; no longer R301.2, R304.1
- net N$34: now also C231.1, U209.8; no longer C331.1, U307.8
- net N$35: now also C230.1, U209.7; no longer C330.1, U307.7
- net N$36: now also R202.2, U204.2; no longer R302.2, U304.2
- net N$37: now also C226.2, U209.1; no longer C326.2, U307.1
- net N$38: now also D202.A, U209.15; no longer D302.A, U307.15
- net N$39: now also D203.C, U209.10; no longer D303.C, U307.10
- net N$4: now also C109.2, U101.20; no longer C207.2, U201.20
- net N$40: now also U305.1; no longer U405.1
- net N$41: now also C108.2, U102.21; no longer C206.2, U202.21
- net N$42: now also C110.2, U102.20; no longer C208.2, U202.20
- net N$43: now also Q103.1, Q104.1, U104.6; no longer R206.2, R208.2, R212.2, R216.1, R217.1, U204.6
- net N$44: now also Q104.2, Q108.1, R106.2; no longer R218.2, R222.1, U204.10
- net N$45: now also R210.2, U208.3; no longer R310.2, U306.3
- net N$46: now also U305.4; no longer U405.4
- net N$47: now also Q301.2, R301.1, U301.1; no longer Q401.2, R401.1, U401.1
- net N$48: now also R305.1, U301.4; no longer R405.1, U401.4
- net N$49: now also R102.2, U104.1; no longer R202.2, R218.1, U204.11
- net N$5: now also Q112.3, Q117.1, Q118.1, R119.1; no longer Q204.3, Q209.1, Q210.1, R239.1
- net N$50: now also R102.1, U104.8; no longer R204.2, R210.2, U204.12
- net N$51: now also U102.17, U104.3; no longer R222.2, R226.1, U204.15
- net N$56: now also D103.3, R137.1, U107.6; no longer D203.3, R257.1, U207.6
- net N$57: now also D104.3, R138.1, U108.6; no longer D204.3, R258.1, U208.6
- net N$58: now also U306.1; no longer U406.1
- net N$59: now also U306.4; no longer U406.4
- net N$6: now also R101.1, U103.8; no longer R225.2, R227.2, R229.1, U203.16
- net N$62: now also C206.1, U202.4; no longer C306.1, U302.4
- net N$63: now also Q202.1, R211.2; no longer Q302.1, R312.2
- net N$64: now also D203.A, Q201.3, R212.1, U209.9; no longer D303.A, Q301.3, R313.1, U307.9
- net N$65: now also Q201.1, R212.2; no longer Q301.1, R313.2
- net N$66: now also C207.1, U203.4; no longer C307.1, U303.4
- net N$67: now also Q101.1, Q102.1, U103.6; no longer Q1.1, Q4.1, R229.2
- net N$68: now also Q102.2, Q106.1, R104.2; no longer Q3.1, Q4.2, R5.2
- net N$7: now also D101.3, R135.1, U105.6; no longer D201.3, R255.1, U205.6
- net N$76: now also R303.1, U303.1; no longer R403.1, U403.1
- net N$77: now also R307.1, U303.4; no longer R407.1, U403.4
- net N$8: now also Q112.1, R113.2, R116.1; no longer Q204.1, R233.2, R236.1
- net N$9: now also U101.17, U103.3; no longer Q1.3, Q3.3, R5.1
- net RG1_H6: now also R208.2, U204.1; no longer R308.2, U304.1
- net RG1_L1: now also R133.2, U107.1; no longer R253.2, U207.1
- net RG1_L2: now also R134.2, U108.1; no longer R254.2, U208.1
- net RG1_L3: now also R131.2, U105.1; no longer R251.2, U205.1
- net RG1_L4: now also R132.2, U106.1; no longer R252.2, U206.1
- net RG2_H6: now also R208.1, U204.8; no longer R308.1, U304.8
- net RG2_L1: now also R133.1, U107.8; no longer R253.1, U207.8
- net RG2_L2: now also R134.1, U108.8; no longer R254.1, U208.8
- net RG2_L3: now also R131.1, U105.8; no longer R251.1, U205.8
- net RG2_L4: now also R132.1, U106.8; no longer R252.1, U206.8
- net SCK: now also C314.1, U101.8, U102.8, U109.7, U110.7, U207.7, U208.7, U302.6; no longer C414.1, U201.8, U202.8, U209.7, U210.7, U305.7, U306.7, U402.6
- net SDO_DAC1: now also U101.10, U102.9; no longer U201.10, U202.9
- net SDO_DAC2: now also U102.10; no longer U202.10
- net TEMP1: now also C211.1, J201.5, U207.2; no longer C311.1, J301.5, U305.2
- net TEMP2: now also C215.1, J201.6, U207.3; no longer C315.1, J301.6, U305.3
- net VREF1: now also C201.1, U101.14, U101.15, U201.1, U201.3; no longer C301.1, U201.14, U201.15, U301.1, U301.3
- net VREF2: now also C202.1, U102.14, U102.15, U202.1, U202.3; no longer C302.1, R206.1, U202.14, U202.15, U302.1, U302.3
- net VREF_MAX743: now also C227.+, U209.6; no longer C327.+, U307.6
- net VSENSE+: now also J206.1, MOV201.1, R201.1; no longer J306.1, MOV301.1, R301.1
- net VSENSE-: now also J207.2, MOV202.2, R202.1; no longer J307.2, MOV302.2, R302.1
Routing:
- net LATCH_DAC: track 184.5 -> 14.7 mm, vias 3 -> 0
- net BYP: track 175.0 -> 34.8 mm, vias 5 -> 2
- net FLT_DAC: track 140.1 -> 0.00 mm, vias 3 -> 0
- net CONV_V: track 144.0 -> 14.7 mm
- net CONV_C2: track 134.8 -> 14.7 mm, vias 2 -> 0
- net SDO_DAC1: track 107.9 -> 0.00 mm
- net MISO: track 188.5 -> 96.2 mm, vias 2 -> 0
- net CLR_DAC2: track 104.0 -> 14.7 mm, vias 2 -> 0
- net VSENSE-: track 61.6 -> 0.20 mm
- net CONV_TEMP: track 69.8 -> 14.7 mm, vias 2 -> 0
- net +12V: track 244.3 -> 293.1 mm
- net CONV_C1: track 47.9 -> 14.7 mm, vias 2 -> 0
- net CLR_DAC1: track 45.6 -> 14.7 mm, vias 3 -> 0
- net +5V: track 298.7 -> 268.7 mm
- net DUT-: track 115.5 -> 85.5 mm, vias 0 -> 124
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- added copper zone on layer 1, net DUT-
- added copper zone on layer 15, net DUT-
- added copper zone on layer 2, net DUT-
Other:
- outline, holes or cut-outs redrawn

Commit message: Cleaned up schematic; PCB layout
Parts:
- added R1: 1k, passives:RESC1608
- R310, R311, R312, R314, R315, R316: value 350R -> 1k
- moved C113 7.62 mm to (25.0, 3.00)
- moved C114 7.62 mm to (25.0, -3.00)
- moved R102 7.62 mm to (29.0, 0.00)
- moved U104 7.62 mm to (25.0, 0.00)
- moved C111 4.12 mm to (-75.0, 3.00)
- moved C112 4.12 mm to (-75.0, -3.00)
- moved R101 4.12 mm to (-71.0, 0.00)
- moved U103 4.12 mm to (-75.0, 0.00)
- moved C110 3.35 mm to (30.5, -4.00)
- moved C108 3.04 mm to (35.0, -4.00)
- moved C101 3.00 mm to (-71.0, -12.8)
- moved C102 3.00 mm to (29.0, -12.8)
- moved C103 3.00 mm to (-71.0, -15.0)
- moved C104 3.00 mm to (29.0, -15.0)
- moved C105 3.00 mm to (-71.0, -10.5)
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Connections:
- net +3V3: no longer R319.2
- net +5V: now also R1.2, R319.2
- net GND: no longer R207.1
- net MISO: now also R1.1
- net VSENSE-: now also R207.1
Routing:
- net FLT_DAC: track 0.00 -> 130.4 mm, vias 0 -> 2
- net CONV_V: track 14.7 -> 139.2 mm
- net CONV_C2: track 14.7 -> 134.3 mm, vias 0 -> 2
- net LATCH_DAC: track 14.7 -> 127.8 mm, vias 0 -> 3
- net SDO_DAC1: track 0.00 -> 105.3 mm
- net BYP: track 34.8 -> 132.4 mm
- net CLR_DAC2: track 14.7 -> 103.4 mm
- net +12V: track 293.1 -> 214.6 mm
- net CONV_TEMP: track 14.7 -> 69.5 mm, vias 0 -> 2
- net MISO: track 96.2 -> 128.2 mm
- net CONV_C1: track 14.7 -> 45.0 mm, vias 0 -> 2
- net CLR_DAC1: track 14.7 -> 37.9 mm, vias 0 -> 2
- net MOSI: track 191.9 -> 210.0 mm, vias 0 -> 2
- net DUT-: track 85.5 -> 68.2 mm
- net SCK: track 190.5 -> 205.4 mm, vias 0 -> 2
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- added copper zone on layer 15, net DUT+
- added copper zone on layer 16, net DUT+
- added copper zone on layer 2, net DUT+

Commit message: Schematic layout
Routing:
- net +12V: track 214.6 -> 205.6 mm
Changed lines of the file:
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@@
 <drawing>
 <settings>
-<setting alwaysvectorfont="yes"/>
+<setting alwaysvectorfont="no"/>
 <setting verticaltext="up"/>
 </settings>
@@
 <contactref element="U101" pad="23"/>
 <contactref element="C109" pad="1"/>
-<contactref element="R117" pad="2"/>
-<contactref element="Q115" pad="3"/>
-<contactref element="R115" pad="2"/>
 <contactref element="C119" pad="1"/>
 <contactref element="C108" pad="1"/>
@@
 <wire x1="35.95" y1="-4" x2="34.7" y2="-2.75" width="0.4064" layer="16"/>
 <wire x1="34.7" y1="-2.75" x2="32.7" y2="-2.75" width="0.4064" layer="16"/>
-<wire x1="46.5" y1="-5.85" x2="44" y2="-5.85" width="0.4064" layer="16"/>
-<wire x1="49" y1="-5.85" x2="46.5" y2="-5.85" width="0.4064" layer="16"/>
 <wire x1="52.75" y1="-5.85" x2="49" y2="-5.85" width="0.4064" layer="16"/>
-<wire x1="53" y1="-6.1" x2="52.75" y2="-5.85" width="0.4064" layer="16"/>
 <via x="49" y="-7" extent="1-16" drill="0.3" diameter="0.6"/>
 <wire x1="49" y1="-5.85" x2="49" y2="-7" width="0.4064" layer="16"/>
-<wire x1="44" y1="-5.85" x2="37.8" y2="-5.85" width="0.4064" layer="16"/>
 <wire x1="37.8" y1="-5.85" x2="35.95" y2="-4" width="0.4064" layer="16"/>
 <via x="-45.75" y="-6" extent="1-16" drill="0.3" diameter="0.6"/>
@@
 <contactref element="R116" pad="2"/>
 <wire x1="-53.25" y1="-5.85" x2="-55.75" y2="-5.85" width="0.4064" layer="16"/>
+<contactref element="R117" pad="2"/>
+<contactref element="Q115" pad="3"/>
+<contactref element="R115" pad="2"/>
+<wire x1="46.5" y1="-5.85" x2="44" y2="-5.85" width="0.4064" layer="16"/>
 <wire x1="110" y1="-45" x2="143.54" y2="-60" width="0" layer="19" extent="1-1"/>
+<wire x1="101.5" y1="-57" x2="110" y2="-45" width="0" layer="19" extent="1-1"/>
+<wire x1="80" y1="-60.85" x2="101.5" y2="-57" width="0" layer="19" extent="16-16"/>
+<wire x1="53" y1="-6.1" x2="77.7432" y2="-45.980071875" width="0" layer="19" extent="1-16"/>
+<wire x1="52.75" y1="-5.85" x2="53" y2="-6.1" width="0" layer="19" extent="16-16"/>
+<wire x1="46.5" y1="-5.85" x2="49" y2="-5.85" width="0" layer="19" extent="16-16"/>
+<wire x1="37.8" y1="-5.85" x2="44" y2="-5.85" width="0" layer="19" extent="16-16"/>
 <wire x1="-47" y1="-6.1" x2="-46.9" y2="-6" width="0" layer="19" extent="16-16"/>
 <wire x1="-47.25" y1="-5.85" x2="-47" y2="-6.1" width="0" layer="19" extent="16-16"/>

Commit message: PCB layout
Parts:
- removed C213: 470n, passives:CAPC1608
- removed C222, C239: 100n, passives:CAPC1608
- removed C233: 10µ, passives:CAPCP6032
- removed C236: 470p, passives:CAPRR1000W80L1300T400H900
- removed L203: 4µ7, inductor-coilcraft:MSS7341
- removed PS201: RFMM-0505S, modules:RECOM-SIP7
- removed U206: 78L05_TO-220AB-3-BR, ic:TO-220AB-3-BR
- moved C219 19.1 mm to (97.0, 0.00), turned to 270 degrees
- moved J204 18.0 mm to (-1.00, -59.0)
- moved J205 18.0 mm to (-1.00, -50.0)
- moved R209 17.9 mm to (98.0, 0.00), turned to 90 degrees
- moved R210 17.0 mm to (96.0, -5.00)
- moved U204 16.0 mm to (94.0, 0.00), turned to 180 degrees
- moved C216 14.6 mm to (94.6, -2.10), turned to 0 degrees
- moved C218 13.3 mm to (92.0, -5.00), turned to 0 degrees
- moved R208 13.0 mm to (90.0, 0.00), turned to 90 degrees
- moved C228 12.5 mm to (94.0, -10.0), turned to 0 degrees
- moved U208 12.5 mm to (94.0, -10.0), turned to 180 degrees
- moved R203 12.1 mm to (106.5, -15.0), turned to 0 degrees
- moved R204 12.0 mm to (112.0, -15.0), turned to 0 degrees
- moved C224 12.0 mm to (94.0, -7.50), turned to 0 degrees
- moved R205 10.5 mm to (105.0, -11.0)
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Connections:
- removed net N$60: C236.1, L203.1, PS201.1
- net +12V: no longer C213.1, U206.1
- net +5V: no longer C222.1, C233.+, L203.2, U206.3
- net +5V_I: no longer C236.2, C239.1, PS201.7
- net GND: no longer C213.2, C222.2, C233.-, PS201.2, U206.2
- net GNDI: no longer C239.2, PS201.5
Routing:
- net MISO: track 128.2 -> 201.6 mm, vias 0 -> 4
- net VSENSE-: track 0.20 -> 37.9 mm
- net DUT-: track 68.2 -> 32.1 mm
- net CSEN_L1: track 9.14 -> 41.2 mm
- net BYP: track 132.4 -> 163.5 mm, vias 2 -> 6
- net CSEN_L2: track 7.14 -> 38.2 mm
- net +3V_2: track 77.7 -> 47.3 mm
- net VSENSE+: track 23.3 -> 53.7 mm
- net GND: track 283.1 -> 307.7 mm, vias 94 -> 98
- net CONV_V: track 139.2 -> 158.1 mm
- net +5V: track 276.8 -> 258.2 mm, vias 38 -> 33
- net -15V: track 113.1 -> 97.9 mm, vias 7 -> 9
- net MOSI: track 210.0 -> 224.4 mm
- net N$36: track 0.44 -> 14.3 mm
- net N$43: track 13.3 -> 24.7 mm
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Other:
- outline, holes or cut-outs redrawn

Commit message: PCB layout
Parts:
- moved C237 32.6 mm to (20.5, -54.0), turned to 270 degrees
- moved R212 29.0 mm to (23.5, -54.0), turned to 90 degrees
- moved C238 28.7 mm to (20.5, -46.0), turned to 270 degrees
- moved Q201 28.2 mm to (22.0, -50.0), turned to 90 degrees
- moved C231 27.5 mm to (59.0, -48.5), turned to 180 degrees
- moved C230 26.6 mm to (59.0, -46.0), turned to 180 degrees
- moved C226 26.2 mm to (59.0, -43.5), turned to 0 degrees
- moved Q202 26.2 mm to (22.0, -42.0), turned to 90 degrees
- moved R211 24.5 mm to (23.5, -46.0), turned to 90 degrees
- moved C235 24.5 mm to (26.0, -52.0), turned to 90 degrees
- moved L202 22.2 mm to (38.0, -58.0), turned to 90 degrees
- moved C227 21.1 mm to (50.0, -54.0), turned to 0 degrees
- moved C234 20.8 mm to (26.0, -40.0), turned to 90 degrees
- moved C229 19.8 mm to (54.5, -43.5), turned to 270 degrees
- moved U209 14.3 mm to (50.0, -46.0), turned to 270 degrees
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Routing:
- net +15V: track 90.6 -> 31.4 mm
- net -15V: track 97.9 -> 58.2 mm
- net +12V: track 202.8 -> 232.8 mm
- net BYP2G1: track 3.87 -> 23.3 mm
- net BPY1G1: track 4.06 -> 22.7 mm
- net BYP2G2: track 2.67 -> 14.7 mm
- net BYP1G2: track 2.77 -> 13.7 mm
- net +5V: track 258.2 -> 252.0 mm
- net RG1_H6: track 0.00 -> 2.74 mm
- net SCK: track 212.8 -> 213.8 mm
- net N$36: track 14.3 -> 13.3 mm
- net N$30: track 18.5 -> 19.5 mm
- net N$29: track 16.4 -> 15.4 mm
- net MOSI: track 224.4 -> 225.4 mm
- net MISO: track 201.6 -> 202.6 mm
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Other:
- outline, holes or cut-outs redrawn
- board text added: "->"
- board text added: "<-"
