File: PCB/V4A/Control_Board.brd (EAGLE design)
At the start: 100 x 100 mm, 53 parts, among them IC301 7805T, U103 LM50, U104 LM50, U205 AD620, U208 LTC1865L, U301 LP2985-3.1, U302 MAX743

Commit message: Added optoisolation to MOSFET board
Parts:
- moved J301 294.5 mm to (44.0, 20.0), turned to 180 degrees
- moved SV1 15.0 mm to (18.0, 10.0)
- moved SV3 15.0 mm to (-18.0, 10.0)
Changed lines of the file:
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@@
 <wire x1="50" y1="100" x2="-50" y2="100" width="0" layer="20"/>
 <wire x1="-50" y1="100" x2="-50" y2="0" width="0" layer="20"/>
+<wire x1="-1" y1="0" x2="-1" y2="-15" width="0.1524" layer="21"/>
+<wire x1="1" y1="0" x2="1" y2="-15" width="0.1524" layer="21"/>
 </plain>
 <attributes>
@@
 <element name="C311" library="passives" package="C3216" value="2µ2" x="-145" y="-200"/>
 <element name="C310" library="passives" package="C3216" value="10n" x="-140" y="-190"/>
-<element name="J301" library="con-jack" library_urn="urn:adsk.eagle:library:154" package="SPC4077" package3d_urn="urn:adsk.eagle:package:7492/1" value="" x="-140" y="-210">
-<attribute name="MF" value="" x="-140" y="-210" size="1.778" layer="27" display="off"/>
-<attribute name="MPN" value="" x="-140" y="-210" size="1.778" layer="27" display="off"/>
-<attribute name="OC_FARNELL" value="unknown" x="-140" y="-210" size="1.778" layer="27" display="off"/>
-<attribute name="OC_NEWARK" value="unknown" x="-140" y="-210" size="1.778" layer="27" display="off"/>
+<element name="J301" library="con-jack" library_urn="urn:adsk.eagle:library:154" package="SPC4077" package3d_urn="urn:adsk.eagle:package:7492/1" value="" x="44" y="20" rot="R180">
+<attribute name="MF" value="" x="44" y="20" size="1.778" layer="27" rot="R180" display="off"/>
+<attribute name="MPN" value="" x="44" y="20" size="1.778" layer="27" rot="R180" display="off"/>
+<attribute name="OC_FARNELL" value="unknown" x="44" y="20" size="1.778" layer="27" rot="R180" display="off"/>
+<attribute name="OC_NEWARK" value="unknown" x="44" y="20" size="1.778" layer="27" rot="R180" display="off"/>
 </element>
-<element name="SV3" library="con-lsta" library_urn="urn:adsk.eagle:library:161" package="FE07-2W" package3d_urn="urn:adsk.eagle:package:8176/1" value="" x="-33" y="10">
-<attribute name="MF" value="" x="-33" y="10" size="1.778" layer="27" display="off"/>
-<attribute name="MPN" value="" x="-33" y="10" size="1.778" layer="27" display="off"/>
-<attribute name="OC_FARNELL" value="unknown" x="-33" y="10" size="1.778" layer="27" display="off"/>
-<attribute name="OC_NEWARK" value="unknown" x="-33" y="10" size="1.778" layer="27" display="off"/>
+<element name="SV3" library="con-lsta" library_urn="urn:adsk.eagle:library:161" package="FE07-2W" package3d_urn="urn:adsk.eagle:package:8176/1" value="" x="-18" y="10">
+<attribute name="MF" value="" x="-18" y="10" size="1.778" layer="27" display="off"/>
+<attribute name="MPN" value="" x="-18" y="10" size="1.778" layer="27" display="off"/>
+<attribute name="OC_FARNELL" value="unknown" x="-18" y="10" size="1.778" layer="27" display="off"/>
+<attribute name="OC_NEWARK" value="unknown" x="-18" y="10" size="1.778" layer="27" display="off"/>
 </element>
-<element name="SV1" library="con-lsta" library_urn="urn:adsk.eagle:library:161" package="FE07-2W" package3d_urn="urn:adsk.eagle:package:8176/1" value="" x="33" y="10">
-<attribute name="MF" value="" x="33" y="10" size="1.778" layer="27" display="off"/>
-<attribute name="MPN" value="" x="33" y="10" size="1.778" layer="27" display="off"/>
-<attribute name="OC_FARNELL" value="unknown" x="33" y="10" size="1.778" layer="27" display="off"/>
-<attribute name="OC_NEWARK" value="unknown" x="33" y="10" size="1.778" layer="27" display="off"/>
+<element name="SV1" library="con-lsta" library_urn="urn:adsk.eagle:library:161" package="FE07-2W" package3d_urn="urn:adsk.eagle:package:8176/1" value="" x="18" y="10">
+<attribute name="MF" value="" x="18" y="10" size="1.778" layer="27" display="off"/>
+<attribute name="MPN" value="" x="18" y="10" size="1.778" layer="27" display="off"/>
+<attribute name="OC_FARNELL" value="unknown" x="18" y="10" size="1.778" layer="27" display="off"/>
+<attribute name="OC_NEWARK" value="unknown" x="18" y="10" size="1.778" layer="27" display="off"/>
 </element>
 </elements>
@@
 <wire x1="-138.6" y1="-190" x2="-143.6" y2="-190" width="0" layer="19" extent="1-1"/>
 <wire x1="-143.6" y1="-200" x2="-143.6" y2="-190" width="0" layer="19" extent="1-1"/>
-<wire x1="-143" y1="-210" x2="-143.6" y2="-200" width="0" layer="19" extent="1-1"/>
-<wire x1="-140" y1="-214.8" x2="-143" y2="-210" width="0" layer="19" extent="1-1"/>
+<wire x1="47" y1="20" x2="-143.6" y2="-200" width="0" layer="19" extent="1-1"/>
+<wire x1="44" y1="24.8" x2="47" y2="20" width="0" layer="19" extent="1-1"/>
 </signal>
 <signal name="+3V3">
@@
 <contactref element="C301" pad="1"/>
 <contactref element="J301" pad="3"/>
-<wire x1="-146.4" y1="-170" x2="-137" y2="-210" width="0" layer="19" extent="1-1"/>
+<wire x1="-146.4" y1="-170" x2="41" y2="20" width="0" layer="19" extent="1-1"/>
 <wire x1="-142.54" y1="-165.16" x2="-146.4" y2="-170" width="0" layer="19" extent="1-1"/>
 </signal>
