File: PCB/V4A/MOSFET_Board.sch (EAGLE design)
At the start: 223 parts, among them IC1 7805T, IC2 7805T, Q101 SIRC10DP, Q102 SIRC10DP, Q103 BC817, Q104 BC817, Q105 SIRC10DP, Q106 SIRC10DP, Q107 BC817, Q108 BC807, Q109 BC817, Q110 BC807, Q111 IXTK102N65X2, Q112 IXTK102N65X2, Q301 BC807, Q302 BC807, Q303 BC807, Q304 BC807, Q305 BC807, Q306 BC807, Q307 BC807, Q308 BC807, U1 LM50, U101 AD420, U102 AD420, U103 LT1014I, U104 LT1014I, U105 AD620, U106 AD620, U107 AD620, U108 AD620, U109 LTC1865L, U110 LTC1865L, U111 LP2985-3.1, U2 LM50, U205 AD620, U208 LTC1865L, U3 LTC1865L, U301 HCPL-063N, U302 HCPL-063N, U303 HCPL-063N, U304 HCPL-063N, U4 MAX743, X1 GMSTBA4

Commit message: PCB layout, cleaned part list
Parts:
- removed C10: 10µ, passives:CPOL-6032-C
- removed C11, C6: 1µ, passives:CPOL-3216-A
- removed C115, C118, C119, C120, C121, C17, C19: 0.1µ, passives:C-EU-1608
- removed C12, C8: 10n, passives:C-EU-3216
- removed C13: 22µ, passives:CPOL-6032-C
- removed C135: 1µ, passives:C-EU-3216
- removed C136: 10n, passives:C-EU-2012
- removed C137: 4µ7, passives:C-EU-3216
- removed C14, C15: 220µ, rcl:CPOL-EUE3.5-10
- removed C16, C18: 0.33µ, passives:C-EU-3216
- removed C4, C5: 500p, passives:C-EU-1608
- removed C7, C9: 0.1µ, passives:C-EU-3216
- removed Q301, Q302, Q303, Q304, Q305, Q306, Q307, Q308: BC807, transistors:BC807
- removed R105, R106: 100k, passives:R-EU-1608
- removed R107, R112, R113, R114, R115, R116, R117: 10k, passives:R-EU-1608
- removed R129, R130: 100R, passives:R-EU-3216
- removed R3, R4: 100R, passives:R-EU-2012
- removed R312, R313, R314, R315, R316: 350R, passives:R-EU-1608
- removed U1, U2: LM50, ic:LM50
- removed U105, U108: AD620, ic:AD620R-8
- removed U111: LP2985-3.1, ic:LP2985-3.1
- removed U3: LTC1865L, ic:LTC1865L
- removed U4: MAX743, ic:MAX743WE
- added C320: 150n, rcl:C-EU050-030X075
- added C321, C326: 1µ, passives:CPOL-3216-A
- added C322, C323, C325, C327: 0.1µ, passives:C-EU-3216
- added C324: 500p, passives:C-EU-1608
- added C401, C402, C403, C404, C417, C418, C419: 0.1µ, passives:C-EU-1608
- added C405, C406, C407, C408, C420, C421, C422: 0.01µ, passives:C-EU-3216
- added C409, C410, C411, C412, C413, C414, C415, C416, C423, C424, C425, C426, C427, C428: 15p, passives:C-EU-1608
- added D303: BAT54S, diode:BAT54S
- added Q401, Q402, Q403, Q404, Q405, Q406, Q407, Q408, Q409, Q410, Q411, Q412, Q413, Q414: BC807, transistors:BC807
- added R229, R230: 100R, passives:R-EU-2012
- added R401, R402, R403, R404, R405, R406, R407, R408, R409, R410, R411, R412, R413, R414, R415, R416, R417, R418, R419, R420, R421, R422, R423, R424, R425, R426, R427, R428: 350R, passives:R-EU-1608
- added U305: AD620, ic:AD620R-8
- added U306, U307: LTC1865L, ic:LTC1865L
- added U401, U402, U403, U404, U405, U406, U407: HCPL-063N, ic:HCPL-063N
- C215, C219, C221: device passives:C-EU-3216 -> passives:C-EU-1608
- C218: value 500p -> 0.1µ
- C220: value 1µ -> 0.1µ; device passives:CPOL-3216-A -> passives:C-EU-1608
- C301, C302: value 0.1µ -> 0.33µ; device passives:C-EU-1608 -> passives:C-EU-3216
- C303: value 0.01µ -> 0.1µ
- C304: value 0.01µ -> 1µ; device passives:C-EU-3216 -> passives:CPOL-3216-A
- C305, C307, C314: value 15p -> 10n; device passives:C-EU-1608 -> passives:C-EU-2012
- C306: value 15p -> 10µ; device passives:C-EU-1608 -> passives:CPOL-6032-C
- C308: value 15p -> 0.1µ
- C310: value 0.1µ -> 22µ; device passives:C-EU-1608 -> passives:CPOL-6032-C
- C311, C312: value 0.01µ -> 220µ; device passives:C-EU-3216 -> rcl:CPOL-EUE3.5-10
- C313: value 15p -> 1µ; device passives:C-EU-1608 -> passives:C-EU-3216
- C315: value 15p -> 4µ7; device passives:C-EU-1608 -> passives:C-EU-3216
- C316: value 15p -> 0.1µ; device passives:C-EU-1608 -> passives:C-EU-3216
- L301, L302: device passives:L-EUSRN1060 -> passives:L-EU_MSS1260
- R205, R206: value 2M -> 100k; device passives:R-EU-3216 -> passives:R-EU-1608
- R207, R212, R213: value 2M -> 10k; device passives:R-EU-3216 -> passives:R-EU-1608
- R214, R215: value 2k15 -> 10k; device passives:R-EU-2012 -> passives:R-EU-1608
- R216: value 100R -> 10k; device passives:R-EU-2012 -> passives:R-EU-1608
- R243, R245: value 3R3 -> 2R
- R301: value 350R -> 0R; device passives:R-EU-1608 -> passives:R-EU-3216
- R302, R304, R305, R306, R307: value 350R -> 2M; device passives:R-EU-1608 -> passives:R-EU-3216
- R303: value 350R -> 16R; device passives:R-EU-1608 -> rcl:R-EU_0204/7
- R308, R309: value 350R -> 2k15; device passives:R-EU-1608 -> passives:R-EU-2012
- R310: value 350R -> 100R; device passives:R-EU-1608 -> passives:R-EU-2012
- R311: value 350R -> 10k
- U208: value LTC1865L -> AD620; device ic:LTC1865L -> ic:AD620R-8
- U301: value HCPL-063N -> MAX743; device ic:HCPL-063N -> ic:MAX743WE
- U302: value HCPL-063N -> LP2985-3.1; device ic:HCPL-063N -> ic:LP2985-3.1
- U303, U304: value HCPL-063N -> LM50; device ic:HCPL-063N -> ic:LM50
- renumbered C1 to C318, C101 to C201, C102 to C202, C103 to C203, C104 to C204, C105 to C205, C106 to C206, C107 to C207, C108 to C208, C109 to C209, C110 to C210, C111 to C211, C112 to C212, C113 to C213, C114 to C214, C116 to C216, C117 to C217, C122 to C222, C123 to C223, C124 to C224, C125 to C225, C126 to C226, C127 to C227, C128 to C228, C129 to C229, C130 to C230, C131 to C231, C132 to C232, C2 to C317, C3 to C319, D101 to D201, D102 to D202, D103 to D203, D104 to D204, HS101 to HS201, HS102 to HS202, IC1 to IC301, IC2 to IC302, J1 to J301, JP1 to JP301, MOV201 to MOV301, MOV202 to MOV302, MOV203 to MOV303, MOV204 to MOV304, PS101 to PS301, Q101 to Q201, Q102 to Q202, Q103 to Q203, Q104 to Q204, Q105 to Q205, Q106 to Q206, Q107 to Q207, Q108 to Q208, Q109 to Q209, Q110 to Q210, Q111 to Q211, Q112 to Q212, R1 to R249, R101 to R201, R102 to R202, R103 to R203, R104 to R204, R108 to R208, R109 to R209, R110 to R210, R111 to R211, R118 to R218, R119 to R219, R120 to R220, R121 to R221, R122 to R222, R123 to R223, R124 to R224, R125 to R225, R126 to R226, R127 to R227, R128 to R228, R131 to R231, R132 to R232, R133 to R233, R134 to R234, R135 to R235, R136 to R236, R137 to R237, R138 to R238, R139 to R239, R140 to R240, R141 to R241, R142 to R242, R143 to R243, R144 to R245, R145 to R247, R146 to R244, R147 to R248, R148 to R246, R149 to R251, R150 to R252, R151 to R253, R152 to R254, R153 to R255, R154 to R256, R155 to R257, R156 to R258, R2 to R250, U$2 to J302, U$3 to J303, U101 to U201, U102 to U202, U103 to U203, U104 to U204, U106 to U206, U107 to U207, U109 to U209, U110 to U210, X1 to X301
Connections:
- removed net BYP_ISO: C306.1, R231.1, R233.1, R306.1, U302.VO1
- removed net CLR_DAC: Q301.B
- removed net CLR_DAC_ISO: C305.1, R305.1, U301.VO1
- removed net FLT_DAC_ISO: Q308.B
- removed net MISO_ISO: Q307.B
- removed net MOSI_ISO: C314.1, R314.1, U303.VO2
- removed net SCK_ISO: C313.1, R313.1, U303.VO1
- removed net SS_C: Q304.B
- removed net SS_C_ISO: C308.1, R308.1, U302.VO2
- removed net SS_DAC: Q303.B
- removed net SS_DAC_ISO: C307.1, R307.1, U301.VO2
- removed net SS_TEMP_I: U3.CONV
- removed net SS_V_I: U208.CONV
- removed net T1_OUT: C318.+, R3.1, U1.VO
- removed net T2_OUT: C319.+, R4.1, U2.VO
- new net BYP_I: Q401.B
- new net CLR_DAC1_I: Q410.B
- new net CLR_DAC2_I: Q413.B
- new net CONV_C1_I: Q403.B
- new net CONV_C2_I: Q407.B
- new net CONV_TEMP: C410.1, R410.1, U306.CONV, U402.VO1
- new net CONV_TEMP_I: Q402.B
- new net CONV_V: C414.1, R414.1, U307.CONV, U402.VO2
- new net CONV_V_I: Q406.B
- new net FAN1_PWM_I: Q409.B
- new net FAN2_PWM_I: Q412.B
- new net FLT_DAC_I: C428.1, R428.1, U407.VO2
- new net LATCH_DAC_I: Q405.B
- new net N$40: Q409.E, R417.1, U405.A1
- new net N$46: Q412.E, R420.1, U405.A2
- new net N$47: Q401.E, R401.1, U401.A1
- new net N$48: Q405.E, R405.1, U401.A2
- new net N$58: Q410.E, R418.1, U406.A1
- new net N$59: Q413.E, R421.1, U406.A2
- new net N$61: C320.1, R303.1
- new net VREF_MAX743: C306.+, U301.VREF
- net +12V: now also C215.1, C301.1, C302.1; no longer C115.1, C16.1, C18.1
- net +15V: now also C218.1, C219.1, C220.1, C311.+, C323.1, U208.+V, U301.FB+, U305.+V; no longer C118.1, C119.1, C120.1, C14.+, C215.1, U105.+V, U108.+V, U4.FB+
- net +3V3: now also C315.1, C321.+, C322.1, C326.+, C327.1, D303.C2, R412.2, R413.2, R414.2, R416.2, R426.2, R427.2, U302.VOUT, U306.VCC, U307.VCC; no longer C137.1, C220.+, C221.1, C6.+, C7.1, R308.2, R313.2, R314.2, U111.VOUT, U208.VCC, U3.VCC
- net +5V: now also C303.2, C308.1, C310.+, C316.1, C401.1, C402.1, C403.1, C404.1, C405.1, C406.1, C407.1, C408.1, C417.1, C418.1, C420.1, C421.1, R409.2, R410.2, R411.2, R415.2, R419.2, R422.2, R423.2, R424.2, U301.AV+, U301.V+, U301.V+@1, U301.V+@2, U301.V+@3, U303.+V, U304.+V, U401.VCC, U402.VCC, U403.VCC, U404.VCC, U405.VCC, U406.VCC; no longer C13.+, C17.1, C19.1, C301.1, C302.1, C303.1, C304.1, C311.1, C9.2, R301.2, R302.2, R303.2, R304.2, R305.2, R306.2, R307.2, R309.2, R310.2, R311.2, R312.2, R315.2, R316.2, U1.+V, U2.+V, U301.VCC, U302.VCC, U303.VCC, U304.VCC, U4.AV+, U4.V+, U4.V+@1, U4.V+@2, U4.V+@3
- net +5V_I: now also C419.1, C422.1, R401.2, R402.2, R403.2, R404.2, R405.2, R406.2, R407.2, R408.2, R417.2, R418.2, R420.2, R421.2, R425.2, R428.2, U407.VCC; no longer C310.1, C312.1
- net -15V: now also C221.1, C312.-, C325.1, U208.-V, U301.FB-, U305.-V; no longer C121.1, C15.-, C219.1, U105.-V, U108.-V, U4.FB-
- net BYP: now also C409.1, R231.1, R233.1, R409.1, U401.VO1; no longer Q302.B
- net CLR_DAC1: now also C424.1, R424.1, U406.VO1
- net CLR_DAC2: now also C427.1, R427.1, U406.VO2
- net CONV_C1: now also C411.1, R411.1, U403.VO1
- net CONV_C2: now also C415.1, R415.1, U403.VO2
- net CSEN_H1: now also U205.+; no longer U105.+
- net CSEN_H2: now also U208.-; no longer U108.-
- net CSEN_L2: now also U208.+; no longer U108.+
- net DUT+: now also R303.2
- net DUT-: now also C320.2, R301.2, U205.-; no longer U105.-
- net FAN1_PWM: now also C423.1, R423.1, U405.VO1
- net FAN2_PWM: now also C426.1, R426.1, U405.VO2
- net FLT_DAC: now also Q414.B; no longer C316.1, R316.1, U304.VO2
- net GND: now also C220.2, C303.1, C304.-, C305.1, C306.-, C310.-, C311.-, C312.+, C315.2, C316.2, C321.-, C322.2, C323.2, C324.2, C325.2, C326.-, C327.2, C401.2, C402.2, C403.2, C404.2, C405.2, C406.2, C407.2, C408.2, C409.2, C410.2, C411.2, C412.2, C413.2, C414.2, C415.2, C416.2, C417.2, C418.2, C420.2, C421.2, C423.2, C424.2, C426.2, C427.2, D303.A1, Q411.C, Q414.C, R207.1, R212.1, R301.1, R308.1, R311.1, U208.REF, U301.12/15, U301.AGND, U304.GND, U305.REF, U306.GND, U307.GND, U401.GND, U402.GND, U403.GND, U404.GND, U405.GND, U406.GND, U407.C1, U407.C2; no longer C10.-, C11.-, C115.2, C118.2, C119.2, C12.2, C120.2, C121.2, C13.-, C135.2, C136.2, C137.2, C14.-, C15.+, C16.2, C17.2, C18.2, C19.2, C220.-, C303.2, C304.2, C305.2, C306.2, C311.2, C4.2, C5.2, C6.-, C7.2, C8.1, C9.1, Q307.C, Q308.C, R107.1, R112.1, R214.1, R217.1, U1.GND, U105.REF, U108.REF, U111.GND, U2.GND, U208.GND, U3.GND, U304.C1, U304.C2, U4.12/15, U4.AGND, U4.GND
- net GNDI: now also C419.2, C422.2, C425.2, C428.2, Q401.C, Q402.C, Q403.C, Q404.C, Q405.C, Q406.C, Q407.C, Q408.C, Q409.C, Q410.C, Q412.C, Q413.C, U401.C1, U401.C2, U402.C1, U402.C2, U403.C1, U403.C2, U404.C1, U404.C2, U405.C1, U405.C2, U406.C1, U406.C2, U407.GND; no longer C310.2, C312.2, C315.2, C316.2, Q301.C, Q302.C, Q303.C, Q304.C, Q305.C, Q306.C, U301.C1, U301.C2, U302.C1, U302.C2, U303.C1, U303.C2, U304.GND
- net LATCH_DAC: now also C413.1, R413.1, U401.VO2
- net LGATE_1: now also R229.2; no longer R129.2
- net LGATE_2: now also R230.2; no longer R130.2
- net MISO: now also Q411.B, U306.SDO, U307.SDO; no longer C315.1, R315.1, U304.VO1
- net MISO_I: now also C425.1, R425.1, U407.VO1; no longer U208.SDO, U3.SDO
- net MOSI: now also C416.1, R416.1, U306.SDI, U307.SDI, U404.VO2; no longer Q306.B
- net MOSI_I: now also Q408.B; no longer U208.SDI, U3.SDI
- net N$10: now also C314.1, U302.BYP; no longer C136.1, U111.BYP
- net N$11: now also R213.2, R214.2; no longer R113.2, R114.2
- net N$12: now also R205.2, R207.2, R213.1, R214.1; no longer R105.2, R107.2, R113.1, R114.1
- net N$13: now also R215.2; no longer R115.2
- net N$14: now also R215.1; no longer R115.1
- net N$17: now also Q411.E, R419.1, U407.A1; no longer Q307.E, R311.1, U304.A1
- net N$18: now also Q414.E, R422.1, U407.A2; no longer Q308.E, R312.1, U304.A2
- net N$19: now also Q404.E, R404.1, U404.A1; no longer Q305.E, R309.1, U303.A1
- net N$20: now also Q408.E, R408.1, U404.A2; no longer Q306.E, R310.1, U303.A2
- net N$21: now also Q402.E, R402.1, U402.A1; no longer Q302.E, R302.1, U302.A1
- net N$22: now also Q406.E, R406.1, U402.A2; no longer Q304.E, R304.1, U302.A2
- net N$23: now also R310.1, U305.OUT; no longer R216.1, U205.OUT
- net N$24: now also R306.1, R307.2; no longer R212.1, R213.2
- net N$26: now also R304.2, R306.2; no longer R206.2, R212.2
- net N$27: now also R304.1, R305.2; no longer R206.1, R207.2
- net N$29: now also R307.1, R308.2, U305.+; no longer R213.1, R214.2, U205.+
- net N$30: now also C324.1, D303.C1A2, R310.2, U307.CH0; no longer C218.1, R216.2, U208.CH0
- net N$33: now also R302.2, R305.1; no longer R205.2, R207.1
- net N$34: now also C307.1, U301.CC-; no longer C12.1, U4.CC-
- net N$35: now also C304.+, U301.SS; no longer C11.+, U4.SS
- net N$37: now also C305.2, U301.CC+; no longer C8.2, U4.CC+
- net N$38: now also U301.LX+; no longer U4.LX+
- net N$39: now also U301.LX-; no longer U4.LX-
- net N$43: now also R206.2, R212.2, R216.1, R217.1; no longer R106.2, R112.2, R116.1, R117.1
- net N$45: now also R311.2, U307.CH1; no longer R217.2, U208.CH1
- net N$52: now also R230.1; no longer R130.1
- net N$54: now also R216.2, R217.2; no longer R116.2, R117.2
- net N$57: now also U208.OUT; no longer U108.OUT
- net N$6: now also R229.1; no longer R129.1
- net N$7: now also U205.OUT; no longer U105.OUT
- net N$76: now also Q403.E, R403.1, U403.A1; no longer Q301.E, R301.1, U301.A1
- net N$77: now also Q407.E, R407.1, U403.A2; no longer Q303.E, R303.1, U301.A2
- net RG1_H6: now also R309.2, U305.RG@1; no longer R215.2, U205.RG@1
- net RG1_L2: now also U208.RG@1; no longer U108.RG@1
- net RG1_L3: now also U205.RG@1; no longer U105.RG@1
- net RG2_H6: now also R309.1, U305.RG@2; no longer R215.1, U205.RG@2
- net RG2_L2: now also U208.RG@2; no longer U108.RG@2
- net RG2_L3: now also U205.RG@2; no longer U105.RG@2
- net SCK: now also C412.1, R412.1, U306.SCK, U307.SCK, U404.VO1; no longer Q305.B
- net SCK_I: now also Q404.B; no longer U208.SCK, U3.SCK
- net TEMP1: now also C318.+, U303.VO, U306.CH0; no longer C4.1, R3.2, U3.CH0
- net TEMP2: now also C319.+, U304.VO, U306.CH1; no longer C5.1, R4.2, U3.CH1
- net VREF1: now also C313.1, R205.1, U302.ON/OFF, U302.VIN; no longer C135.1, R105.1, U111.ON/OFF, U111.VIN
- net VREF2: now also R206.1; no longer C10.+, R106.1, U4.VREF
- net VSENSE+: now also R302.1; no longer R205.1
- net VSENSE-: now also U305.-; no longer U205.-
Other:
- note removed: "Isolation and level shifting"
