File: PCB/V2A/MOSFET_Board.sch (EAGLE design)
At the start: 222 parts, among them J203 CTRL, Q101 BC807, Q102 BC817, Q103 BC807, Q104 BC817, Q105 BC817, Q106 BC807, Q107 BC817, Q108 BC807, Q109 SIRC10DP, Q110 SIRC10DP, Q111 BC817, Q112 BC817, Q113 SIRC10DP, Q114 SIRC10DP, Q115 BC817, Q116 BC807, Q117 BC817, Q118 BC807, Q119 IXTK102N65X2, Q120 IXTK102N65X2, Q301 BC807, Q302 BC807, Q303 BC807, Q304 BC807, Q305 BC807, Q306 BC807, Q307 BC807, Q308 BC807, Q310 BC807, Q311 BC807, Q313 BC807, Q314 BC807, U101 AD420, U102 AD420, U103 AD620, U104 AD620, U105 AD620, U106 AD620, U107 AD620, U108 AD620, U109 LTC1865_S8, U110 LTC1865_S8, U201 LP2985, U202 LP2985, U203 LP2985, U204 AD620, U208 LTC1865_S8, U301 HCPL-063N, U302 HCPL-063N, U303 HCPL-063N, U304 HCPL-063N, U306 HCPL-063N, U307 HCPL-063N

Commit message: V2A fully routed
Parts:
- removed C122, C123, C124, C125, C126, C127, C128, C135, C136, C228: 100n, custom_capacitors:CAP-1608
- removed C129, C130, C131, C132: 470p, custom_capacitors:CAP-1608
- removed C133, C134, C224: 4µ7, custom_capacitors:CAP-3216
- removed C324, C325, C327, C328: 15p, custom_capacitors:CAP-1608
- removed D103, D104: BAT54S, custom_semiconductors_discrete:BAT54S
- removed J203: CTRL, mechanical:HEAD_1X16_MALE
- removed PAD1, PAD2, PAD3, PAD4, PAD5, PAD6: WIREPADSMD5-2,5, wirepad:WIREPADSMD5-2,5
- removed Q111, Q112, Q115, Q117: BC817, custom_semiconductors_discrete:BC817
- removed Q113, Q114: SIRC10DP, custom_semiconductors_discrete:SIRC10DP
- removed Q116, Q118, Q303, Q304, Q305, Q306, Q307, Q308, Q310, Q311, Q313, Q314: BC807, custom_semiconductors_discrete:BC807
- removed Q119, Q120: IXTK102N65X2, custom_semiconductors_discrete:IXTK102N65X2
- removed R1, R315, R316: 1k, custom_resistors:R-EU-1608
- removed R10, R11, R12, R13, R6, R7, R8, R9: 5k, custom_resistors:R-EU-1608
- removed R125: 2R, custom_resistors:R-EU-3216
- removed R127, R128, R131, R132, R133, R134: 2k15, custom_resistors:R-EU-2012
- removed R135, R136, R137, R138: 100R, custom_resistors:R-EU-1608
- removed R14, R15, R16: (no value), custom_resistors:MOV-14X7.4
- removed R2, R3, R4, R5: 0R003, custom_resistors:WSL3637_0.01
- removed R318, R319, R321, R322, R324, R325, R327, R328: 350R, custom_resistors:R-EU-1608
- removed SJ201: DUT_GND, jumper:SJW
- removed U107, U108: AD620, custom_semiconductors:AD620R-8
- removed U109, U110, U208: LTC1865_S8, custom_semiconductors:LTC1865_S8
- removed U306, U307: HCPL-063N, custom_semiconductors:HCPL-063N
- added C204: 470n, custom_capacitors:CAP-1608
- added C211, C214: 4µ7, custom_capacitors:CAP-3216
- added C212, C402, C404, C410, C414, C416: 10n, custom_capacitors:CAP-1608
- added C213, C215, C217, C220, C320, C401, C403, C409, C413, C415: 100n, custom_capacitors:CAP-1608
- added C221, C323: 470p, custom_capacitors:CAP-1608
- added C317: 100µ 10V, custom_capacitors:CAP-POL7343
- added C405, C406, C407, C408, C411, C412, C417, C418, C419: 15p, custom_capacitors:CAP-1608
- added D202, D304: BAT54S, custom_semiconductors_discrete:BAT54S
- added D301, D302, D303: SK12, custom_semiconductors_discrete:SK12
- added J301: (no value), custom_mechanical:JACK-PLUG-2.5
- added JP301: (no value), pinhead:PINHD-1X12
- added L301, L302: 100µ, custom_inductors:SRN5040
- added L303: 47µ, custom_inductors:SRN5040
- added MOV101: 680V, custom_resistors:MOV-14X7.4
- added MOV201: (no value), custom_resistors:MOV-14X7.4
- added PAD301, PAD302: WIREPADSMD5-2,5, wirepad:WIREPADSMD5-2,5
- added Q201, Q203, Q208, Q209: BC817, custom_semiconductors_discrete:BC817
- added Q202, Q204, Q210, Q401, Q402, Q403, Q404, Q405, Q406, Q407, Q408, Q409: BC807, custom_semiconductors_discrete:BC807
- added Q205: IXTK102N65X2, custom_semiconductors_discrete:IXTK102N65X2
- added Q206, Q207: SIRC10DP, custom_semiconductors_discrete:SIRC10DP
- added R121, R221, R223: 100R, custom_resistors:R-EU-1608
- added R122, R217, R220, R222: 2k15, custom_resistors:R-EU-2012
- added R211, R218, R219: 5k, custom_resistors:R-EU-1608
- added R212: 100k, custom_resistors:R-EU-1608
- added R213, R216, R411, R412, R415, R416, R417: 1k, custom_resistors:R-EU-1608
- added R214, R215: 0R003, custom_resistors:WSL3637_0.01
- added R401, R402, R403, R404, R405, R406, R407, R408, R409, R410, R413, R414, R418, R419: 350R, custom_resistors:R-EU-1608
- added SJ301: DUT_GND, jumper:SJW
- added U205, U305: LTC1865_S8, custom_semiconductors:LTC1865_S8
- added U206: AD620, custom_semiconductors:AD620R-8
- added U401, U402, U403, U404, U405: HCPL-063N, custom_semiconductors:HCPL-063N
- C102, C203, C208: value 4µ7 -> 100n; device custom_capacitors:CAP-3216 -> custom_capacitors:CAP-1608
- C103, C104, C112, C304: value 100n -> 10n
- C107, C306: value 10n -> 470n; device custom_capacitors:CAP-2012 -> custom_capacitors:CAP-1608
- C108, C109, C205, C308: value 10n -> 4µ7; device custom_capacitors:CAP-2012 -> custom_capacitors:CAP-3216
- C110, C206, C207, C305, C321, C322: value 10n -> 100n; device custom_capacitors:CAP-2012 -> custom_capacitors:CAP-1608
- C111, C302: value 100n -> 470n
- C114, C303, C318, C319: value 100n -> 4µ7; device custom_capacitors:CAP-1608 -> custom_capacitors:CAP-3216
- C115, C116, C117: value 470n -> 100n
- C118: value 470n -> 470p
- C121: value 100n -> 470p
- C201, C202: value 4µ7 -> 10n; device custom_capacitors:CAP-3216 -> custom_capacitors:CAP-1608
- C209: value 4µ7 -> 470n; device custom_capacitors:CAP-3216 -> custom_capacitors:CAP-1608
- C301: value 100n -> 15µ 25V; device custom_capacitors:CAP-1608 -> custom_capacitors:CAP-POL7343
- C307: value 10n -> 15µ 25V; device custom_capacitors:CAP-2012 -> custom_capacitors:CAP-POL7343
- C309: value 15p -> 470n
- C310, C311, C314: value 15p -> 10n
- C312, C313: value 15p -> 4µ7; device custom_capacitors:CAP-1608 -> custom_capacitors:CAP-3216
- C315: value 15p -> 15µ 25V; device custom_capacitors:CAP-1608 -> custom_capacitors:CAP-POL7343
- C316: value 15p -> 100n
- Q101, Q103, Q106, Q301, Q302: value BC807 -> BC817; device custom_semiconductors_discrete:BC807 -> custom_semiconductors_discrete:BC817
- Q102, Q104: value BC817 -> BC807; device custom_semiconductors_discrete:BC817 -> custom_semiconductors_discrete:BC807
- Q105: value BC817 -> IXTK102N65X2; device custom_semiconductors_discrete:BC817 -> custom_semiconductors_discrete:IXTK102N65X2
- Q107: value BC817 -> SIRC10DP; device custom_semiconductors_discrete:BC817 -> custom_semiconductors_discrete:SIRC10DP
- Q108: value BC807 -> SIRC10DP; device custom_semiconductors_discrete:BC807 -> custom_semiconductors_discrete:SIRC10DP
- Q109: value SIRC10DP -> BC817; device custom_semiconductors_discrete:SIRC10DP -> custom_semiconductors_discrete:BC817
- Q110: value SIRC10DP -> BC807; device custom_semiconductors_discrete:SIRC10DP -> custom_semiconductors_discrete:BC807
- R101: value 49k3 -> 5k
- R102: value 49k3 -> 2R; device custom_resistors:R-EU-1608 -> custom_resistors:R-EU-3216
- R104: value 5k -> 49k3
- R105: value 5k -> 2R; device custom_resistors:R-EU-1608 -> custom_resistors:R-EU-3216
- R107: value 2R -> 100k; device custom_resistors:R-EU-3216 -> custom_resistors:R-EU-1608
- R108: value 2R -> 1k; device custom_resistors:R-EU-3216 -> custom_resistors:R-EU-1608
- R113, R310, R311: value 1k -> 2k15; device custom_resistors:R-EU-1608 -> custom_resistors:R-EU-2012
- R114, R118: value 2R -> 5k; device custom_resistors:R-EU-3216 -> custom_resistors:R-EU-1608
- R115: value 100k -> 5k
- R116: value 100k -> 0R003; device custom_resistors:R-EU-1608 -> custom_resistors:WSL3637_0.01
- R117: value 1k -> 0R003; device custom_resistors:R-EU-1608 -> custom_resistors:WSL3637_0.01
- R119: value 1k -> 5k
- R120: value 2R -> 2k15; device custom_resistors:R-EU-3216 -> custom_resistors:R-EU-2012
- R123: value 2R -> 100R; device custom_resistors:R-EU-3216 -> custom_resistors:R-EU-1608
- R201, R206: value 2M -> 5k; device custom_resistors:R-EU-2012 -> custom_resistors:R-EU-1608
- R202: value 2k15 -> 5k; device custom_resistors:R-EU-2012 -> custom_resistors:R-EU-1608
- R203, R205: value 2M -> 2R; device custom_resistors:R-EU-2012 -> custom_resistors:R-EU-3216
- R204: value 2M -> 49k3; device custom_resistors:R-EU-2012 -> custom_resistors:R-EU-1608
- R207, R208: value 2k15 -> 2R; device custom_resistors:R-EU-2012 -> custom_resistors:R-EU-3216
- R209: value 100R -> 2R; device custom_resistors:R-EU-1608 -> custom_resistors:R-EU-3216
- R210: value 10k -> 5k
- R303, R304: value 350R -> 10k
- R305, R306, R307, R308, R309: value 350R -> 2M; device custom_resistors:R-EU-1608 -> custom_resistors:R-EU-3216
- R312: value 1k -> 100R
- R313: value 350R -> 2k15; device custom_resistors:R-EU-1608 -> custom_resistors:R-EU-2012
- R314: value 1k -> 10k
- U102: value AD420 -> AD620; device custom_semiconductors:AD420AR -> custom_semiconductors:AD620R-8
- U103: value AD620 -> LP2985; device custom_semiconductors:AD620R-8 -> custom_semiconductors:LP2985
- U105: value AD620 -> LTC1865_S8; device custom_semiconductors:AD620R-8 -> custom_semiconductors:LTC1865_S8
- U201: value LP2985 -> AD420; device custom_semiconductors:LP2985 -> custom_semiconductors:AD420AR
- U202: value LP2985 -> AD620; device custom_semiconductors:LP2985 -> custom_semiconductors:AD620R-8
- U301: value HCPL-063N -> MAX743; device custom_semiconductors:HCPL-063N -> custom_semiconductors:MAX743W
- U302: value HCPL-063N -> LP2985; device custom_semiconductors:HCPL-063N -> custom_semiconductors:LP2985
- U303: value HCPL-063N -> LM2671M; device custom_semiconductors:HCPL-063N -> custom_semiconductors:LM2671M
- U304: value HCPL-063N -> AD620; device custom_semiconductors:HCPL-063N -> custom_semiconductors:AD620R-8
Connections:
- removed net CLR_DAC1: C324.1, R324.1, U101.CLR, U306.VO1
- removed net CLR_DAC1_I: J203.6, Q310.B
- removed net CLR_DAC2: C313.1, R313.1, U102.CLR, U301.VO2
- removed net CLR_DAC2_I: J203.7
- removed net CONV_TEMP: C311.1, R311.1, U303.VO1
- removed net CONV_TEMP_I: J203.10
- removed net FAN1_PWM_I: J203.14
- removed net FAN2_PWM_I: J203.13
- removed net FLT_DAC: Q311.B, U101.FLT, U102.FLT
- removed net FLT_DAC_I: C325.1, J203.1, R325.1, U307.VO1
- removed net SDO_DAC1: U101.SDO, U102.SDI
- new net CLR_DAC: C407.1, R407.1, U101.CLR, U201.CLR, U402.VO1
- new net CLR_DAC_I: JP301.5, Q403.B
- new net N$28: R314.2, U305.CH0
- new net N$55: C310.1, U301.CC-
- new net N$60: R103.1, U101.FLT
- new net N$61: C309.1, U301.SS
- new net N$64: C304.2, U301.CC+
- new net N$65: D301.A, L301.2, U301.LX+
- new net N$69: D302.C, L302.1, U301.LX-
- new net N$70: C301.+, D301.C, Q301.C, R301.1, U301.FB+
- new net N$71: C302.1, Q301.B, R301.2
- new net N$72: C307.-, D302.A, Q302.C, R302.1, U301.FB-
- new net N$73: C306.1, Q302.B, R302.2
- new net VREF_MAX743: C308.1, U301.VREF
- net +12V: now also C103.1, C104.1, C113.1, C201.1, C202.1, C207.1, C213.1, C315.+, C316.1, J301.3, Q106.C, Q208.C, R107.2, R108.2, R212.2, R213.2, U201.VCC, U303.VIN; no longer C106.1, C107.1, C108.1, C109.1, C110.1, C119.1, C120.1, Q115.C, Q117.C, R115.2, R116.2, R117.2, R119.2, U102.VCC
- net +15V: now also C106.1, C107.1, C116.1, C119.1, C203.1, C204.1, C219.1, C321.1, Q101.C, Q103.C, Q201.C, Q203.C, Q301.E, R101.2, R201.2, U102.+V, U202.+V, U206.+V, U304.+V; no longer C111.1, C113.1, C115.1, C117.1, C121.1, C122.1, C123.1, C124.1, Q102.C, Q104.C, Q105.C, Q107.C, R103.2, R105.2, U103.+V, U105.+V, U107.+V, U108.+V
- net +3V3: now also C313.1, R411.2, R412.2, R415.2, R416.2, U302.VOUT; no longer C210.1, R310.2, R311.2, R312.2, R314.2, R315.2, R316.2, U203.VOUT
- net +3V_1: now also C109.1, C114.1, C115.1, C319.1, C320.1, D304.C2, U103.VOUT, U105.VCC, U305.VCC; no longer C133.1, C135.1, C208.1, U109.VCC, U201.VOUT
- net +3V_2: now also C211.1, C214.1, C215.1, D202.C2, U203.VOUT, U205.VCC; no longer C134.1, C136.1, C209.1, C224.1, C228.1, D103.C2, D104.C2, U110.VCC, U202.VOUT, U208.VCC
- net +5V: now also C205.1, C206.1, C305.2, C312.1, C317.+, C401.1, C402.1, C403.1, C404.1, C409.1, C410.1, C413.1, C414.1, L301.1, L303.2, R103.2, R202.2, R304.1, R403.2, R404.2, R407.2, R408.2, R417.2, R418.2, U201.VLL, U301.AV+, U301.V+, U301.V+@1, U301.V+@2, U301.V+@3, U302.ON/OFF, U302.VIN, U401.VCC, U402.VCC, U403.VCC, U404.VCC; no longer C103.1, C104.1, C203.1, C301.1, C302.1, C304.1, C305.1, C306.1, C307.1, C308.1, C321.1, R1.2, R309.2, R313.2, R319.2, R322.2, R324.2, R327.2, U102.VLL, U203.ON/OFF, U203.VIN, U301.VCC, U302.VCC, U303.VCC, U304.VCC, U306.VCC
- net +5V_I: now also C415.1, C416.1, JP301.12, R401.2, R402.2, R405.2, R406.2, R409.2, R410.2, R413.2, R414.2, R419.2, U405.VCC; no longer C319.1, C322.1, J203.16, R301.2, R302.2, R303.2, R304.2, R305.2, R306.2, R307.2, R308.2, R318.2, R321.2, R325.2, R328.2, U307.VCC
- net -15V: now also C110.2, C111.2, C117.1, C120.1, C208.2, C209.2, C217.1, C220.1, C322.1, Q102.C, Q104.C, Q202.C, Q204.C, Q302.E, R206.1, U102.-V, U202.-V, U206.-V, U304.-V; no longer C112.2, C114.2, C116.2, C118.2, C125.1, C126.1, C127.1, C128.1, C219.1, Q101.C, Q103.C, Q106.C, Q108.C, R104.1, U103.-V, U105.-V, U107.-V, U108.-V
- net BPY1G1: now also Q107.G, R110.2; no longer Q109.G, R112.2
- net BYP: now also C406.1, R216.1, R404.1, U401.VO2; no longer C309.1, R113.1, R309.1, U301.VO1
- net BYP1: now also Q106.E, Q110.E, R110.1, R113.1; no longer Q117.E, Q118.E, R118.1, R128.1
- net BYP1G2: now also Q108.G, R112.2; no longer Q113.G, R118.2
- net BYP2: now also Q208.E, Q210.E, R208.1, R209.1, R217.2; no longer Q115.E, Q116.E, R114.1, R120.1, R127.2
- net BYP2G1: now also Q206.G, R208.2; no longer Q110.G, R114.2
- net BYP2G2: now also Q207.G, R209.2; no longer Q114.G, R120.2
- net BYP_I: now also JP301.6, Q402.B; no longer J203.8, Q301.B
- net CONV_C1: now also C418.1, R416.1, U105.CONV, U404.VO2; no longer C315.1, R315.1, U109.CONV, U303.VO2
- net CONV_C1_I: now also JP301.8, Q408.B; no longer J203.9, Q307.B
- net CONV_C2: now also C405.1, R403.1, U205.CONV, U401.VO1; no longer C316.1, R316.1, U110.CONV, U304.VO2
- net CONV_C2_I: now also JP301.7, Q401.B; no longer J203.11, Q308.B
- net CONV_V: now also C417.1, R415.1, U305.CONV, U404.VO1; no longer C312.1, R312.1, U208.CONV, U304.VO1
- net CONV_V_I: now also JP301.9, Q407.B; no longer J203.12, Q304.B
- net CSEN_H1: now also Q107.S, Q108.S, R109.1, R113.2, R116.I1, R117.I2, U104.-; no longer Q109.S, Q113.S, R123.1, R128.2, R2.I1, R3.I2, U106.-
- net CSEN_H2: now also Q206.S, Q207.S, R207.1, R214.I1, R215.I2, R217.1, U204.-; no longer Q110.S, Q114.S, R125.1, R127.1, R4.I1, R5.I2, U108.-
- net CSEN_L1: now also Q105.S, Q107.D, Q108.D, R109.2, U102.REF, U104.+; no longer Q109.D, Q113.D, Q119.S, R123.2, U103.REF, U106.+
- net CSEN_L2: now also Q205.S, Q206.D, Q207.D, R207.2, U202.REF, U204.+; no longer Q110.D, Q114.D, Q120.S, R125.2, U104.REF, U108.+
- net DUT+: now also MOV101.2, MOV201.2, Q105.D, Q205.D; no longer PAD1.P, PAD3.P, Q119.D, Q120.D, R15.2, R16.2
- net DUT-: now also MOV101.1, MOV201.1, R116.I2, R117.I1, R214.I2, R215.I1, SJ301.2; no longer PAD2.P, PAD4.P, R15.1, R16.1, R2.I2, R3.I1, R4.I2, R5.I1, SJ201.2
- net GND: now also C107.2, C108.2, C109.2, C110.1, C111.1, C112.2, C114.2, C116.2, C118.2, C204.2, C208.1, C209.1, C211.2, C212.2, C213.2, C214.2, C215.2, C217.2, C220.2, C221.2, C301.-, C304.1, C305.1, C307.+, C315.-, C317.-, C319.2, C320.2, C322.2, C323.2, C401.2, C402.2, C403.2, C404.2, C405.2, C406.2, C407.2, C408.2, C409.2, C410.2, C411.2, C412.2, C413.2, C414.2, C417.2, C418.2, D202.A1, D303.A, D304.A1, J301.1, L302.2, Q109.E, Q110.C, Q209.E, Q210.C, Q409.C, R303.2, R314.1, SJ301.1, U102.-, U103.GND, U104.REF, U105.GND, U201.RS1, U201.RS2, U202.-, U205.GND, U206.REF, U301.12/15, U301.AGND, U304.REF, U305.GND, U401.GND, U402.GND, U403.GND, U404.GND, U405.A1, U405.C1, U405.C2; no longer C103.2, C104.2, C111.2, C112.1, C114.1, C116.1, C118.1, C122.2, C123.2, C124.2, C125.2, C126.2, C127.2, C128.2, C129.2, C130.2, C131.2, C132.2, C133.2, C134.2, C135.2, C136.2, C201.2, C202.2, C208.2, C209.2, C224.2, C228.2, C301.2, C304.2, C305.2, C307.2, C311.2, C315.2, C324.2, C327.2, D103.A1, D104.A1, Q111.E, Q112.E, Q116.C, Q118.C, Q311.C, Q314.C, R210.1, SJ201.1, U102.GND, U102.RS1, U102.RS2, U103.-, U104.-, U105.REF, U107.REF, U108.REF, U109.GND, U110.GND, U202.GND, U208.GND, U304.GND, U306.GND, U307.C1, U307.C2
- net GNDI: now also C415.2, C416.2, C419.2, JP301.10, JP301.11, Q401.C, Q402.C, Q403.C, Q404.C, Q405.C, Q406.C, Q407.C, Q408.C, U401.C1, U401.C2, U402.C1, U402.C2, U403.C1, U403.C2, U404.C1, U404.C2, U405.GND, U405.VO1; no longer C319.2, C322.2, C325.2, C328.2, J203.15, Q301.C, Q302.C, Q303.C, Q304.C, Q305.C, Q306.C, Q307.C, Q308.C, Q310.C, Q313.C, U301.C1, U301.C2, U302.C1, U302.C2, U303.C1, U303.C2, U304.C1, U304.C2, U306.C1, U306.C2, U307.GND
- net HIGHC1: now also C121.1, R123.2, U105.CH0; no longer C129.1, R135.2, U109.CH0
- net HIGHC2: now also C221.1, R223.2, U205.CH0; no longer C131.1, R137.2, U110.CH0
- net LATCH_DAC: now also C408.1, R408.1, U201.LATCH, U402.VO2; no longer C327.1, R327.1, U102.LATCH, U306.VO2
- net LATCH_DAC_I: now also JP301.4, Q404.B; no longer J203.5, Q313.B
- net LGATE_1: now also Q105.G, R102.1, R105.2; no longer Q119.G, R107.1, R108.2
- net LGATE_2: now also Q205.G, R203.1, R205.2; no longer Q120.G, R109.1, R110.2
- net LOWC1: now also C118.1, R121.2, U105.CH1; no longer C130.1, R136.2, U109.CH1
- net LOWC2: now also C218.1, R221.2, U205.CH1; no longer C132.1, R138.2, U110.CH1
- net MISO: now also Q409.B, R417.1, U105.SDO, U205.SDO, U305.SDO; no longer Q314.B, R1.1, U109.SDO, U110.SDO, U208.SDO
- net MISO_I: now also C419.1, JP301.1, R419.1, U405.VO2; no longer C328.1, J203.2, R328.1, U307.VO2
- net MOSI: now also C412.1, R412.1, U105.SDI, U201.SDI, U205.SDI, U305.SDI, U403.VO2; no longer C310.1, R310.1, U101.SDI, U109.SDI, U110.SDI, U208.SDI, U302.VO1
- net MOSI_I: now also JP301.2, Q406.B; no longer J203.4, Q302.B
- net N$1: now also Q101.B, Q102.E, R101.1; no longer Q101.E, Q105.B, R103.1
- net N$10: now also C112.1, U103.BYP; no longer C205.1, U201.BYP
- net N$11: now also Q104.E, R105.1; no longer Q106.E, R108.1
- net N$12: now also Q201.B, Q202.E, R201.1; no longer Q103.E, Q107.B, R105.1
- net N$13: now also Q101.E, R102.2; no longer Q105.E, R107.2
- net N$14: now also Q204.E, R205.1; no longer Q108.E, R110.1
- net N$15: now also Q201.E, R203.2; no longer Q107.E, R109.2
- net N$16: now also D101.C1A2, R121.1, U104.OUT; no longer D102.C1A2, R136.1, U106.OUT
- net N$17: now also C311.1, U303.CB; no longer Q311.E, R319.1, U307.A1
- net N$18: now also Q409.E, R418.1, U405.A2; no longer Q314.E, R322.1, U307.A2
- net N$19: now also C311.2, D303.C, L303.1, U303.VSW; no longer Q304.E, R304.1, U304.A1
- net N$2: now also R104.2, U102.RG@1; no longer R101.2, U103.RG@1
- net N$20: now also R303.1, R304.2, U303.FB; no longer Q308.E, R308.1, U304.A2
- net N$21: now also Q405.E, R409.1, U403.A1; no longer Q302.E, R302.1, U302.A1
- net N$22: now also Q406.E, R410.1, U403.A2; no longer Q306.E, R306.1, U302.A2
- net N$23: now also D304.C1A2, R312.1, U304.OUT; no longer R209.1, U204.OUT
- net N$24: now also R306.1, R308.2; no longer R205.1, R206.2
- net N$25: now also Q208.B, Q209.C, Q210.B, R213.1; no longer Q111.C, Q115.B, Q116.B, R117.1
- net N$26: now also R305.2, R306.2; no longer R203.2, R205.2
- net N$27: now also R305.1, R307.2; no longer R203.1, R204.2
- net N$29: now also R308.1, R310.2, U304.+; no longer R206.1, R207.2, U204.+
- net N$3: now also C103.2; no longer C107.2
- net N$30: now also C323.1, R312.2, U305.CH1; no longer C218.1, D201.C1A2, R209.2, U208.CH0
- net N$31: now also Q209.B, R212.1, R216.2; no longer Q111.B, R111.2, R115.1
- net N$32: now also R115.2, R117.E2; no longer R3.E2, R7.2
- net N$33: now also R307.1, R309.2; no longer R201.2, R204.1
- net N$34: now also R114.1, R115.1, U106.+; no longer R6.1, R7.1, U105.+
- net N$35: now also R116.E2, R118.1; no longer R2.E2, R8.1
- net N$36: now also R313.2, U304.-; no longer R202.2, U204.-
- net N$37: now also R118.2, R119.2, U106.-; no longer R8.2, R9.2, U105.-
- net N$38: now also R117.E1, R119.1; no longer R3.E1, R9.1
- net N$39: now also R210.1, R214.E1; no longer R10.1, R4.E1
- net N$4: now also C104.2; no longer C109.2
- net N$40: now also R114.2, R116.E1; no longer R2.E1, R6.2
- net N$41: now also C201.2, U201.C2; no longer C108.2, U102.C2
- net N$42: now also C202.2, U201.C1; no longer C110.2, U102.C1
- net N$43: now also Q202.B, Q203.B, U202.OUT; no longer Q103.B, Q104.B, U104.OUT
- net N$44: now also Q203.E, Q204.B, R206.2; no longer Q104.E, Q108.B, R106.2
- net N$45: now also R202.1, U201.FLT; no longer R210.2, U208.CH1
- net N$46: now also R211.1, R215.E2; no longer R11.1, R5.E2
- net N$47: now also Q401.E, R401.1, U401.A1; no longer Q301.E, R301.1, U301.A1
- net N$48: now also Q402.E, R402.1, U401.A2; no longer Q305.E, R305.1, U301.A2
- net N$49: now also R204.2, U202.RG@1; no longer R102.2, U104.RG@1
- net N$5: now also Q106.B, Q109.C, Q110.B, R108.1; no longer Q112.C, Q117.B, Q118.B, R119.1
- net N$50: now also R204.1, U202.RG@2; no longer R102.1, U104.RG@2
- net N$51: now also U201.VOUT, U202.+; no longer U102.VOUT, U104.+
- net N$52: now also R215.E1, R218.2; no longer R12.2, R5.E1
- net N$53: now also R214.E2, R219.2; no longer R13.2, R4.E2
- net N$54: now also R210.2, R211.2, U206.+; no longer R10.2, R11.2, U107.+
- net N$56: now also D202.C1A2, R223.1, U206.OUT; no longer D103.C1A2, R137.1, U107.OUT
- net N$57: now also D201.C1A2, R221.1, U204.OUT; no longer D104.C1A2, R138.1, U108.OUT
- net N$58: now also Q403.E, R405.1, U402.A1; no longer Q310.E, R318.1, U306.A1
- net N$59: now also Q404.E, R406.1, U402.A2; no longer Q313.E, R321.1, U306.A2
- net N$6: now also R104.1, U102.RG@2; no longer R101.1, U103.RG@2
- net N$62: now also C212.1, U203.BYP; no longer C206.1, U202.BYP
- net N$63: now also R218.1, R219.1, U206.-; no longer R12.1, R13.1, U107.-
- net N$66: now also C314.1, U302.BYP; no longer C207.1, U203.BYP
- net N$67: now also Q103.B, U102.OUT; no longer Q101.B, U103.OUT
- net N$68: now also Q103.E, Q104.B, R106.2; no longer Q102.E, Q106.B, R104.2
- net N$7: now also D102.C1A2, R123.1, U106.OUT; no longer D101.C1A2, R135.1, U105.OUT
- net N$76: now also Q407.E, R413.1, U404.A1; no longer Q303.E, R303.1, U303.A1
- net N$77: now also Q408.E, R414.1, U404.A2; no longer Q307.E, R307.1, U303.A2
- net N$8: now also Q109.B, R107.1, R111.2; no longer Q112.B, R113.2, R116.1
- net N$9: now also U102.+; no longer U103.+
- net RG1_H6: now also R311.2, U304.RG@1; no longer R208.2, U204.RG@1
- net RG1_L1: now also R222.2, U206.RG@1; no longer R133.2, U107.RG@1
- net RG1_L2: now also R220.2, U204.RG@1; no longer R134.2, U108.RG@1
- net RG1_L3: now also R122.2, U106.RG@1; no longer R131.2, U105.RG@1
- net RG1_L4: now also R120.2, U104.RG@1; no longer R132.2, U106.RG@1
- net RG2_H6: now also R311.1, U304.RG@2; no longer R208.1, U204.RG@2
- net RG2_L1: now also R222.1, U206.RG@2; no longer R133.1, U107.RG@2
- net RG2_L2: now also R220.1, U204.RG@2; no longer R134.1, U108.RG@2
- net RG2_L3: now also R122.1, U106.RG@2; no longer R131.1, U105.RG@2
- net RG2_L4: now also R120.1, U104.RG@2; no longer R132.1, U106.RG@2
- net SCK: now also C411.1, R411.1, U105.SCK, U201.SCK, U205.SCK, U305.SCK, U403.VO1; no longer C314.1, R314.1, U102.SCK, U109.SCK, U110.SCK, U208.SCK, U302.VO2
- net SCK_I: now also JP301.3, Q405.B; no longer J203.3, Q306.B
- net SDO_DAC2: now also U101.SDI, U201.SDO; no longer U102.SDO
- net VREF1: now also C108.1, U103.ON/OFF, U103.VIN; no longer C201.1, U201.ON/OFF, U201.VIN
- net VREF2: now also C210.1, U201.REF_IN, U201.REF_OUT, U203.ON/OFF, U203.VIN; no longer C202.1, U102.REF_IN, U102.REF_OUT, U202.ON/OFF, U202.VIN
- net VSENSE+: now also PAD301.P, R309.1; no longer PAD5.P, R14.2, R201.1
- net VSENSE-: now also PAD302.P, R310.1, R313.1; no longer PAD6.P, R14.1, R202.1, R207.1
Other:
- note removed: "+12V -> +5V"
- note removed: "+3V for CSEN1 and TEMP ADCs"
- note removed: "+5V -> +/-15V"
